Commit message: Update bounds, positions, axis in urdf

File: urdf/arm.urdf.xacro (robot description, xacro)
@@ -33,6 +33,6 @@
     </link>
     <joint name="shoulder_pan_joint" type="revolute">
-        <axis xyz="0 -1 0"/>
-        <limit lower="-${pi/2}" upper="${pi/2}" effort="1000.0" velocity="0.5"/>
+        <axis xyz="0 1 0"/>
+        <limit lower="${0.43 - (330./2.)*pi/180.}" upper="0.43" effort="1000.0" velocity="0.5"/>
         <parent link="base_link"/>
         <child link="shoulder_pan_link"/>
@@ -49,9 +49,9 @@
     </link>
     <joint name="shoulder_lift_joint" type="revolute">
-        <axis xyz="1 0 0"/>
-        <limit lower="-${pi/2}" upper="${pi/2}" effort="1000.0" velocity="0.5"/>
+        <axis xyz="-1 0 0"/>
+        <limit lower="-0.82" upper="${-0.82 + (330./2.)*pi/180.}" effort="1000.0" velocity="0.5"/>
         <parent link="shoulder_pan_link"/>
         <child link="shoulder_lift_link"/>
-        <origin xyz="0 -${pan_to_lift} 0" rpy="-${pi/20} 0 0" />
+        <origin xyz="0 -${pan_to_lift} 0" rpy="0 0 0" />
     </joint>
     <link name="elbow_link">
@@ -66,8 +66,8 @@
     <joint name="elbow_joint" type="revolute">
         <axis xyz="1 0 0"/>
-        <limit lower="-${pi/2}" upper="${pi/2}" effort="1000.0" velocity="0.5"/>
+        <limit lower="-2.1" upper="2.1" effort="1000.0" velocity="0.5"/>
         <parent link="shoulder_lift_link"/>
         <child link="elbow_link"/>
-        <origin xyz="0 0 -${lift_to_elbow}" rpy="${pi/10} 0 0"/>
+        <origin xyz="0 0 -${lift_to_elbow}" rpy="0 0 0"/>
     </joint>
     <link name="wrist_link">
@@ -81,9 +81,9 @@
     </link>
     <joint name="wrist_joint" type="revolute">
-        <axis xyz="1 0 0"/>
+        <axis xyz="-1 0 0"/>
         <limit lower="-${pi/2}" upper="${pi/2}" effort="1000.0" velocity="0.5"/>
         <parent link="elbow_link"/>
         <child link="wrist_link"/>
-        <origin xyz="0 0 -${elbow_to_wrist}" rpy="${pi/10} 0 0"/>
+        <origin xyz="0 0 -${elbow_to_wrist}" rpy="0 0 0"/>
     </joint>
     <link name="wrist_twist_link">
@@ -97,5 +97,5 @@
     </link>
     <joint name="wrist_twist_joint" type="revolute">
-        <axis xyz="0 0 1"/>
+        <axis xyz="0 0 -1"/>
         <limit lower="-${pi/2}" upper="${pi/2}" effort="1000.0" velocity="0.5"/>
         <parent link="wrist_link"/>
@@ -115,5 +115,5 @@
 	<joint name="left_gripper_joint" type="revolute">
 		<axis xyz="1 0 0"/>
-		<limit effort="1000.0" lower="0.0" upper="0.548" velocity="0.5"/>
+		<limit effort="1000.0" lower="0.0" upper="1.2" velocity="0.5"/>
 		<origin rpy="0 0 0" xyz="0 ${radius/2} -${twist_to_gripper}"/>
 		<parent link="wrist_twist_link"/>
@@ -142,5 +142,5 @@
 	<joint name="right_gripper_joint" type="revolute">
 		<axis xyz="-1 0 0"/>
-		<limit effort="1000.0" lower="0.0" upper="0.548" velocity="0.5"/>
+		<limit effort="1000.0" lower="0.0" upper="1.2" velocity="0.5"/>
 		<origin rpy="0 0 0" xyz="0 -${radius/2} -${twist_to_gripper}"/>
 		<parent link="wrist_twist_link"/>
