Commit message: Tilt kinect

File: robot/urdf/base_kinect.urdf.xacro (robot description, xacro)
@@ -2,5 +2,6 @@
 <robot xmlns:xacro="http://www.ros.org/wiki/xacro" name="arm">
     <xacro:property name="pi" value="3.14159" />
-    <xacro:property name="kinect_angle_rad" value="0.71" />
+    <xacro:property name="kinect_angle_rad" value="0.40" />
+	<!-- 0.71 -->
     <link name="base_link" />
     <link name="base_footprint" />
