Commit message: Fix packages after recent name changes

File: roomac_arm/urdf/arm.urdf.xacro (robot description, xacro)
@@ -124,5 +124,5 @@
 			<origin rpy="0.0 ${pi/2} 0" xyz="0 0 0"/>
 			<geometry>
-				<mesh filename="package://robot_arm/meshes/l_finger.dae" scale="${scale} ${scale} ${scale}"/>
+				<mesh filename="package://roomac_arm/meshes/l_finger.dae" scale="${scale} ${scale} ${scale}"/>
 			</geometry>
 		</visual>
@@ -139,5 +139,5 @@
 			<origin rpy="0.0 ${pi/2} 0" xyz="0 ${scale*0.00495} ${scale * -0.09137}"/>
 			<geometry>
-				<mesh filename="package://robot_arm/meshes/l_finger_tip.dae" scale="${scale} ${scale} ${scale}"/>
+				<mesh filename="package://roomac_arm/meshes/l_finger_tip.dae" scale="${scale} ${scale} ${scale}"/>
 			</geometry>
 		</visual>
@@ -151,5 +151,5 @@
 			<origin rpy="-3.1415 ${pi/2} 0" xyz="0 0 0"/>
 			<geometry>
-				<mesh filename="package://robot_arm/meshes/l_finger.dae" scale="${scale} ${scale} ${scale}"/>
+				<mesh filename="package://roomac_arm/meshes/l_finger.dae" scale="${scale} ${scale} ${scale}"/>
 			</geometry>
 		</visual>
@@ -167,5 +167,5 @@
 			<origin rpy="-3.1415 ${pi/2} 0" xyz="0 ${scale*0.00495} ${scale*-0.09137}"/>
 			<geometry>
-				<mesh filename="package://robot_arm/meshes/l_finger_tip.dae" scale="${scale} ${scale} ${scale}" />
+				<mesh filename="package://roomac_arm/meshes/l_finger_tip.dae" scale="${scale} ${scale} ${scale}" />
 			</geometry>
 		</visual>

File: roomac_arm/urdf/test2.urdf (robot description, URDF)
Before this commit: robot visual, 16 links, 15 joints
Links:
- link left_gripper: geometry visual mesh filename=package://roomac_arm/meshes/l_finger.dae

Commit message: Combine arm with upper kinect

File: roomac_arm/urdf/arm.urdf.xacro (robot description, xacro)
@@ -14,5 +14,12 @@
         <color rgba="0 0 0 1"/>
     </material>
-    <link name="base_link">
+    <link name="base_link"/>
+    <joint name="robot_to_arm" type="fixed">
+        <axis xyz="0 0 0"/>
+        <parent link="base_link"/>
+        <child link="arm_base_link"/>
+        <origin xyz="-0.1135 -0.153521 0.9465"/>
+    </joint>
+    <link name="arm_base_link">
         <visual>
             <geometry>
@@ -35,5 +42,5 @@
         <axis xyz="0 1 0"/>
         <limit lower="${0.43 - (330./2.)*pi/180.}" upper="0.43" effort="1000.0" velocity="0.5"/>
-        <parent link="base_link"/>
+        <parent link="arm_base_link"/>
         <child link="shoulder_pan_link"/>
         <origin xyz="0 0 0"/>

File: roomac_kinect/urdf/upper_kinect.urdf.xacro (robot description, xacro)
@@ -10,5 +10,5 @@
   <link name="camera_link" />
   <joint name="kinect_joint" type="fixed">
-		<origin rpy="0.0103379679904 0.424522933365 0.876123018686" xyz="-0.15252797763 -0.129919622053 0.930481065395"/>
+		<origin rpy="0.0103379679904 0.424522933365 ${0.876123018686-pi/2}" xyz="-0.15252797763 0.129919622053 0.930481065395"/>
 		<parent link="base_link"/>
 		<child link="camera_link"/>
