Commit message: Move simulation gripper_right_grip link

File: roomac_description/urdf/roomac_gripper_simulation.xacro (robot description, xacro)
@@ -3,5 +3,5 @@
   <link name="gripper_right_grip"/>
   <joint name="right_grip" type="fixed">
-    <origin rpy="0 0 0" xyz="0.0 0.0 -0.085"/>
+    <origin rpy="0 0 0" xyz="0.0 0.0 -0.04"/>
     <parent link="gripper_right_1"/>
     <child link="gripper_right_grip"/>

Commit message: Decrease size of fingers in simulated gripper
they were in collision in new home position

File: roomac_description/urdf/roomac_gripper_simulation.xacro (robot description, xacro)
@@ -40,5 +40,5 @@
       <origin xyz="0 0 -0.03" rpy="0 0 0"/>
       <geometry>
-        <box size="0.02 0.02 0.06" />
+        <box size="0.02 0.01 0.06" />
       </geometry>
     </collision>
@@ -46,5 +46,5 @@
       <origin xyz="0 0 -0.03" rpy="0 0 0"/>
       <geometry>
-        <box size="0.02 0.02 0.06" />
+        <box size="0.02 0.01 0.06" />
       </geometry>
     </visual>
@@ -69,5 +69,5 @@
       <origin xyz="0 0 -0.03" rpy="0 0 0"/>
       <geometry>
-        <box size="0.02 0.02 0.06" />
+        <box size="0.02 0.01 0.06" />
       </geometry>
     </collision>
@@ -75,5 +75,5 @@
       <origin xyz="0 0 -0.03" rpy="0 0 0"/>
       <geometry>
-        <box size="0.02 0.02 0.06" />
+        <box size="0.02 0.01 0.06" />
       </geometry>
     </visual>
