Commit message: Change body colors

File: roomac_description/urdf/materials.xacro (robot description, xacro)
@@ -2,5 +2,11 @@
 <robot name="roomac" xmlns:xacro="http://www.ros.org/wiki/xacro" >
 <material name="silver">
-  <color rgba="0.700 0.700 0.700 1.000"/>
+  <color rgba="0.7 0.7 0.7 1.0"/>
+</material>
+<material name="white">
+  <color rgba="1.0 1.0 1.0 1.0"/>
+</material>
+<material name="black">
+  <color rgba="0.15 0.15 0.15 1.0"/>
 </material>
 </robot>

File: roomac_description/urdf/roomac_body.xacro (robot description, xacro)
@@ -19,5 +19,5 @@
       <mesh filename="package://roomac_description/meshes/base_link.stl" scale="0.001 0.001 0.001"/>
     </geometry>
-    <material name="silver"/>
+    <material name="black"/>
   </visual>
   <collision>
@@ -79,5 +79,5 @@
       <mesh filename="package://roomac_description/meshes/hub_right_1.stl" scale="0.001 0.001 0.001"/>
     </geometry>
-    <material name="silver"/>
+    <material name="black"/>
   </visual>
   <collision>
@@ -99,5 +99,5 @@
       <mesh filename="package://roomac_description/meshes/hub_left_1.stl" scale="0.001 0.001 0.001"/>
     </geometry>
-    <material name="silver"/>
+    <material name="black"/>
   </visual>
   <collision>
@@ -179,5 +179,5 @@
       <mesh filename="package://roomac_description/meshes/eye_left_1.stl" scale="0.001 0.001 0.001"/>
     </geometry>
-    <material name="silver"/>
+    <material name="white"/>
   </visual>
   <collision>
@@ -199,5 +199,5 @@
       <mesh filename="package://roomac_description/meshes/elbow_right_1.stl" scale="0.001 0.001 0.001"/>
     </geometry>
-    <material name="silver"/>
+    <material name="black"/>
   </visual>
   <collision>
@@ -219,5 +219,5 @@
       <mesh filename="package://roomac_description/meshes/elbow_wrist_right_1.stl" scale="0.001 0.001 0.001"/>
     </geometry>
-    <material name="silver"/>
+    <material name="black"/>
   </visual>
   <collision>
@@ -239,5 +239,5 @@
       <mesh filename="package://roomac_description/meshes/caster_tire_right_1.stl" scale="0.001 0.001 0.001"/>
     </geometry>
-    <material name="silver"/>
+    <material name="black"/>
   </visual>
   <collision>
@@ -259,5 +259,5 @@
       <mesh filename="package://roomac_description/meshes/caster_tire_left_1.stl" scale="0.001 0.001 0.001"/>
     </geometry>
-    <material name="silver"/>
+    <material name="black"/>
   </visual>
   <collision>
@@ -279,5 +279,5 @@
       <mesh filename="package://roomac_description/meshes/wheel_tire_right_1.stl" scale="0.001 0.001 0.001"/>
     </geometry>
-    <material name="silver"/>
+    <material name="black"/>
   </visual>
   <collision>
@@ -299,5 +299,5 @@
       <mesh filename="package://roomac_description/meshes/wheel_tire_left_1.stl" scale="0.001 0.001 0.001"/>
     </geometry>
-    <material name="silver"/>
+    <material name="black"/>
   </visual>
   <collision>
@@ -319,5 +319,5 @@
       <mesh filename="package://roomac_description/meshes/base_link_frames_1.stl" scale="0.001 0.001 0.001"/>
     </geometry>
-    <material name="silver"/>
+    <material name="white"/>
   </visual>
   <collision>
@@ -339,5 +339,5 @@
       <mesh filename="package://roomac_description/meshes/shoulder_elbow_gear_right_1.stl" scale="0.001 0.001 0.001"/>
     </geometry>
-    <material name="silver"/>
+    <material name="black"/>
   </visual>
   <collision>
@@ -359,5 +359,5 @@
       <mesh filename="package://roomac_description/meshes/wrist_right_1.stl" scale="0.001 0.001 0.001"/>
     </geometry>
-    <material name="silver"/>
+    <material name="black"/>
   </visual>
   <collision>
@@ -399,5 +399,5 @@
       <mesh filename="package://roomac_description/meshes/shoulder_right_1.stl" scale="0.001 0.001 0.001"/>
     </geometry>
-    <material name="silver"/>
+    <material name="black"/>
   </visual>
   <collision>
@@ -419,5 +419,5 @@
       <mesh filename="package://roomac_description/meshes/shoulder_base_right_1.stl" scale="0.001 0.001 0.001"/>
     </geometry>
-    <material name="silver"/>
+    <material name="black"/>
   </visual>
   <collision>
@@ -439,5 +439,5 @@
       <mesh filename="package://roomac_description/meshes/head_1.stl" scale="0.001 0.001 0.001"/>
     </geometry>
-    <material name="silver"/>
+    <material name="black"/>
   </visual>
   <collision>
@@ -459,5 +459,5 @@
       <mesh filename="package://roomac_description/meshes/eye_right_1.stl" scale="0.001 0.001 0.001"/>
     </geometry>
-    <material name="silver"/>
+    <material name="white"/>
   </visual>
   <collision>
@@ -479,5 +479,5 @@
       <mesh filename="package://roomac_description/meshes/shoulder_base_left_1.stl" scale="0.001 0.001 0.001"/>
     </geometry>
-    <material name="silver"/>
+    <material name="black"/>
   </visual>
   <collision>
@@ -499,5 +499,5 @@
       <mesh filename="package://roomac_description/meshes/shoulder_left_1.stl" scale="0.001 0.001 0.001"/>
     </geometry>
-    <material name="silver"/>
+    <material name="black"/>
   </visual>
   <collision>
@@ -519,5 +519,5 @@
       <mesh filename="package://roomac_description/meshes/gripper_finger_2_left_1.stl" scale="0.001 0.001 0.001"/>
     </geometry>
-    <material name="silver"/>
+    <material name="black"/>
   </visual>
   <collision>
@@ -539,5 +539,5 @@
       <mesh filename="package://roomac_description/meshes/gripper_finger_1_left_1.stl" scale="0.001 0.001 0.001"/>
     </geometry>
-    <material name="silver"/>
+    <material name="black"/>
   </visual>
   <collision>
@@ -559,5 +559,5 @@
       <mesh filename="package://roomac_description/meshes/gripper_left_1.stl" scale="0.001 0.001 0.001"/>
     </geometry>
-    <material name="silver"/>
+    <material name="black"/>
   </visual>
   <collision>
@@ -579,5 +579,5 @@
       <mesh filename="package://roomac_description/meshes/wrist_left_1.stl" scale="0.001 0.001 0.001"/>
     </geometry>
-    <material name="silver"/>
+    <material name="black"/>
   </visual>
   <collision>
@@ -599,5 +599,5 @@
       <mesh filename="package://roomac_description/meshes/elbow_wrist_left_1.stl" scale="0.001 0.001 0.001"/>
     </geometry>
-    <material name="silver"/>
+    <material name="black"/>
   </visual>
   <collision>
@@ -619,5 +619,5 @@
       <mesh filename="package://roomac_description/meshes/elbow_left_1.stl" scale="0.001 0.001 0.001"/>
     </geometry>
-    <material name="silver"/>
+    <material name="black"/>
   </visual>
   <collision>
@@ -659,5 +659,5 @@
       <mesh filename="package://roomac_description/meshes/shoulder_elbow_gear_left_1.stl" scale="0.001 0.001 0.001"/>
     </geometry>
-    <material name="silver"/>
+    <material name="black"/>
   </visual>
   <collision>

File: roomac_description/urdf/roomac_gripper_real.xacro (robot description, xacro)
@@ -18,5 +18,5 @@
       <mesh filename="package://roomac_description/meshes/gripper_right_1.stl" scale="0.001 0.001 0.001"/>
     </geometry>
-    <material name="silver"/>
+    <material name="black"/>
   </visual>
   <collision>
@@ -38,5 +38,5 @@
       <mesh filename="package://roomac_description/meshes/gripper_finger_1_right_1.stl" scale="0.001 0.001 0.001"/>
     </geometry>
-    <material name="silver"/>
+    <material name="black"/>
   </visual>
   <collision>
@@ -58,5 +58,5 @@
       <mesh filename="package://roomac_description/meshes/gripper_finger_2_right_1.stl" scale="0.001 0.001 0.001"/>
     </geometry>
-    <material name="silver"/>
+    <material name="black"/>
   </visual>
   <collision>
