Commit message: Improve detecting artag on robot in gazebo simulation

File: roomac_description/urdf/roomac_body.xacro (robot description, xacro)
@@ -494,5 +494,5 @@
         <origin rpy="0 0 0" xyz="0.0 0.0 0.0"/>
         <geometry>
-            <mesh filename="package://roomac_description/materials/aruco_cube_5cm.dae" scale="1 1 0.001"/>
+            <mesh filename="package://roomac_description/materials/aruco_cube_5cm.dae" scale="1.2 1.2 0.001"/>
         </geometry>
         <material name="artag"/>
@@ -501,5 +501,5 @@
         <origin rpy="0 0 0" xyz="0.0 0.0 0.0"/>
         <geometry>
-            <mesh filename="package://roomac_description/materials/aruco_cube_5cm.dae" scale="1 1 0.001"/>
+            <mesh filename="package://roomac_description/materials/aruco_cube_5cm.dae" scale="1.2 1.2 0.001"/>
         </geometry>
     </collision>

Commit message: Change default left arm position

File: roomac_description/urdf/roomac_body.xacro (robot description, xacro)
@@ -438,5 +438,5 @@
 </joint>
 <joint name="left_shoulder_lift" type="continuous">
-  <origin rpy="0 0 0" xyz="-0.0265 0.0995 0.0"/>
+  <origin rpy="0.32 0 0" xyz="-0.0265 0.0995 0.0"/>
   <parent link="shoulder_left_1"/>
   <child link="shoulder_elbow_left_1"/>
@@ -444,5 +444,5 @@
 </joint>
 <joint name="left_elbow" type="continuous">
-  <origin rpy="0 0 0" xyz="0.0425 0.0 -0.201075"/>
+  <origin rpy="-0.64 0 0" xyz="0.0425 0.0 -0.201075"/>
   <parent link="shoulder_elbow_left_1"/>
   <child link="elbow_wrist_left_1"/>

Commit message: Switch to bundle detection

File: roomac_description/urdf/roomac_body.xacro (robot description, xacro)
@@ -512,5 +512,5 @@
 </joint>
 <joint name="artag_joint_2" type="fixed">
-    <origin rpy="0 0 ${pi/2}" xyz="0 0 0"/>
+    <origin rpy="0 0 ${pi/2}" xyz="0.0595 -0.004 0"/>
     <parent link="artag_link"/>
     <child link="artag_link_2"/>

Commit message: Add robot_base link so that base_link won't have inertia to fix KDL moveit warning

File: roomac_description/urdf/roomac_body.xacro (robot description, xacro)
@@ -1,5 +1,12 @@
 <?xml version="1.0" ?>
 <robot name="roomac" xmlns:xacro="http://www.ros.org/wiki/xacro">
-<link name="base_link">
+<link name="base_link" />
+<joint name="robot_base" type="fixed">
+  <parent link="base_link"/>
+  <child link="robot_base_1"/>
+</joint>
+<!-- Additional link needed to solve moveit warning (as far as I know it shouldn't cause any issue as I'm not using KDL, but still better to solve it): -->
+<!-- The root link base_link has an inertia specified in the URDF, but KDL does not support a root link with an inertia.  As a workaround, you can add an extra dummy link to your URDF. -->
+<link name="robot_base_1">
   <inertial>
     <origin rpy="0 0 0" xyz="-0.13060699359614247 -1.269142483394603e-05 0.10737373059306837"/>

Commit message: Update xacro files

File: roomac_description/urdf/roomac_body.xacro (robot description, xacro)
@@ -10,10 +10,10 @@
 <link name="robot_base_1">
   <inertial>
-    <origin rpy="0 0 0" xyz="-0.13060699359614247 -1.269142483394603e-05 0.10737373059306837"/>
-    <mass value="3.353734949059196"/>
-    <inertia ixx="0.139756" ixy="-3e-06" ixz="0.003607" iyy="0.140028" iyz="1.7e-05" izz="0.11189"/>
-  </inertial>
-  <visual>
-    <origin rpy="0 0 0" xyz="0 0 0"/>
+    <origin xyz="-0.18736789633381332 0.0015304678388801296 0.2632175316600572" rpy="0 0 0"/>
+    <mass value="31.013883468506926"/>
+    <inertia ixx="2.674027" iyy="2.737864" izz="0.665771" ixy="-0.003283" iyz="-0.013126" ixz="-0.310987"/>
+  </inertial>
+  <visual>
+    <origin xyz="0 0 0" rpy="0 0 0"/>
     <geometry>
       <mesh filename="package://roomac_description/meshes/base_link.stl" scale="0.001 0.001 0.001"/>
@@ -22,5 +22,5 @@
   </visual>
   <collision>
-    <origin rpy="0 0 0" xyz="0 0 0"/>
+    <origin xyz="0 0 0" rpy="0 0 0"/>
     <geometry>
       <mesh filename="package://roomac_description/meshes/base_link.stl" scale="0.001 0.001 0.001"/>
@@ -28,41 +28,361 @@
   </collision>
 </link>
-<link name="right_wheel_hub_1">
-  <inertial>
-    <origin rpy="0 0 0" xyz="-1.789765202460103e-06 0.012712108125801563 3.1361035185462073e-06"/>
-    <mass value="0.09451094240372128"/>
-    <inertia ixx="5e-05" ixy="0.0" ixz="0.0" iyy="8.5e-05" iyz="-0.0" izz="5e-05"/>
-  </inertial>
-  <visual>
-    <origin rpy="0 0 0" xyz="-0.0 0.2429 0.0"/>
-    <geometry>
-      <mesh filename="package://roomac_description/meshes/right_wheel_hub_1.stl" scale="0.001 0.001 0.001"/>
-    </geometry>
-    <material name="silver"/>
-  </visual>
-  <collision>
-    <origin rpy="0 0 0" xyz="-0.0 0.2429 0.0"/>
-    <geometry>
-      <mesh filename="package://roomac_description/meshes/right_wheel_hub_1.stl" scale="0.001 0.001 0.001"/>
-    </geometry>
-  </collision>
-</link>
-<link name="right_caster_1">
-  <inertial>
-    <origin rpy="0 0 0" xyz="-0.020793104918766903 -0.0009180067931599534 -0.11995837555497461"/>
-    <mass value="1.2807118618501256"/>
-    <inertia ixx="0.001622" ixy="-2e-06" ixz="-0.000322" iyy="0.002002" iyz="-8e-06" izz="0.000685"/>
-  </inertial>
-  <visual>
-    <origin rpy="0 0 0" xyz="0.2985 0.16 -0.0275"/>
-    <geometry>
-      <mesh filename="package://roomac_description/meshes/right_caster_1.stl" scale="0.001 0.001 0.001"/>
-    </geometry>
-    <material name="silver"/>
-  </visual>
-  <collision>
-    <origin rpy="0 0 0" xyz="0.2985 0.16 -0.0275"/>
-    <geometry>
-      <mesh filename="package://roomac_description/meshes/right_caster_1.stl" scale="0.001 0.001 0.001"/>
+<link name="caster_right_1">
+  <inertial>
+    <origin xyz="0.0037004833856989494 -0.027923972873388603 -0.08822047192631874" rpy="0 0 0"/>
+    <mass value="0.9867038593578229"/>
+    <inertia ixx="0.000947" iyy="0.001166" izz="0.000456" ixy="-2e-06" iyz="-5e-06" ixz="-0.000231"/>
+  </inertial>
+  <visual>
+    <origin xyz="0.324 0.133 0.00465" rpy="0 0 0"/>
+    <geometry>
+      <mesh filename="package://roomac_description/meshes/caster_right_1.stl" scale="0.001 0.001 0.001"/>
+    </geometry>
+    <material name="silver"/>
+  </visual>
+  <collision>
+    <origin xyz="0.324 0.133 0.00465" rpy="0 0 0"/>
+    <geometry>
+      <mesh filename="package://roomac_description/meshes/caster_right_1.stl" scale="0.001 0.001 0.001"/>
+    </geometry>
+  </collision>
+</link>
+<link name="caster_left_1">
+  <inertial>
+    <origin xyz="0.0037004833856989494 0.021923972873387293 -0.0882204719263213" rpy="0 0 0"/>
+    <mass value="0.9867038593578229"/>
+    <inertia ixx="0.000947" iyy="0.001166" izz="0.000456" ixy="2e-06" iyz="5e-06" ixz="-0.000231"/>
+  </inertial>
+  <visual>
+    <origin xyz="0.324 -0.139 0.00465" rpy="0 0 0"/>
+    <geometry>
+      <mesh filename="package://roomac_description/meshes/caster_left_1.stl" scale="0.001 0.001 0.001"/>
+    </geometry>
+    <material name="silver"/>
+  </visual>
+  <collision>
+    <origin xyz="0.324 -0.139 0.00465" rpy="0 0 0"/>
+    <geometry>
+      <mesh filename="package://roomac_description/meshes/caster_left_1.stl" scale="0.001 0.001 0.001"/>
+    </geometry>
+  </collision>
+</link>
+<link name="hub_right_1">
+  <inertial>
+    <origin xyz="-1.789765220804318e-06 0.012712108125801869 3.1361035183559637e-06" rpy="0 0 0"/>
+    <mass value="0.09451094240372103"/>
+    <inertia ixx="5e-05" iyy="8.5e-05" izz="5e-05" ixy="0.0" iyz="-0.0" ixz="0.0"/>
+  </inertial>
+  <visual>
+    <origin xyz="0.0 0.246 0.0" rpy="0 0 0"/>
+    <geometry>
+      <mesh filename="package://roomac_description/meshes/hub_right_1.stl" scale="0.001 0.001 0.001"/>
+    </geometry>
+    <material name="silver"/>
+  </visual>
+  <collision>
+    <origin xyz="0.0 0.246 0.0" rpy="0 0 0"/>
+    <geometry>
+      <mesh filename="package://roomac_description/meshes/hub_right_1.stl" scale="0.001 0.001 0.001"/>
+    </geometry>
+  </collision>
+</link>
+<link name="hub_left_1">
+  <inertial>
+    <origin xyz="-1.7897652210308038e-06 -0.012712108125801591 3.1361035183086937e-06" rpy="0 0 0"/>
+    <mass value="0.09451094240372113"/>
+    <inertia ixx="5e-05" iyy="8.5e-05" izz="5e-05" ixy="-0.0" iyz="0.0" ixz="0.0"/>
+  </inertial>
+  <visual>
+    <origin xyz="0.0 -0.246 0.0" rpy="0 0 0"/>
+    <geometry>
+      <mesh filename="package://roomac_description/meshes/hub_left_1.stl" scale="0.001 0.001 0.001"/>
+    </geometry>
+    <material name="silver"/>
+  </visual>
+  <collision>
+    <origin xyz="0.0 -0.246 0.0" rpy="0 0 0"/>
+    <geometry>
+      <mesh filename="package://roomac_description/meshes/hub_left_1.stl" scale="0.001 0.001 0.001"/>
+    </geometry>
+  </collision>
+</link>
+<link name="wheel_right_1">
+  <inertial>
+    <origin xyz="-4.446890699227879e-08 -0.046359989716390604 2.8955374773431687e-08" rpy="0 0 0"/>
+    <mass value="1.4792126361607076"/>
+    <inertia ixx="0.006728" iyy="0.012762" izz="0.006728" ixy="0.0" iyz="-0.0" ixz="0.0"/>
+  </inertial>
+  <visual>
+    <origin xyz="-0.0 0.21064 0.0" rpy="0 0 0"/>
+    <geometry>
+      <mesh filename="package://roomac_description/meshes/wheel_right_1.stl" scale="0.001 0.001 0.001"/>
+    </geometry>
+    <material name="silver"/>
+  </visual>
+  <collision>
+    <origin xyz="-0.0 0.21064 0.0" rpy="0 0 0"/>
+    <geometry>
+      <mesh filename="package://roomac_description/meshes/wheel_right_1.stl" scale="0.001 0.001 0.001"/>
+    </geometry>
+  </collision>
+</link>
+<link name="wheel_left_1">
+  <inertial>
+    <origin xyz="-3.1796540813644466e-08 0.04035998903806015 1.6110734861740638e-08" rpy="0 0 0"/>
+    <mass value="1.4792124768984427"/>
+    <inertia ixx="0.006728" iyy="0.012762" izz="0.006728" ixy="0.0" iyz="0.0" ixz="0.0"/>
+  </inertial>
+  <visual>
+    <origin xyz="0.0 -0.21664 0.0" rpy="0 0 0"/>
+    <geometry>
+      <mesh filename="package://roomac_description/meshes/wheel_left_1.stl" scale="0.001 0.001 0.001"/>
+    </geometry>
+    <material name="silver"/>
+  </visual>
+  <collision>
+    <origin xyz="0.0 -0.21664 0.0" rpy="0 0 0"/>
+    <geometry>
+      <mesh filename="package://roomac_description/meshes/wheel_left_1.stl" scale="0.001 0.001 0.001"/>
+    </geometry>
+  </collision>
+</link>
+<link name="frame_1">
+  <inertial>
+    <origin xyz="-0.06363233755923882 -0.10316506754069626 -0.18305645699853168" rpy="0 0 0"/>
+    <mass value="4.866480003493675"/>
+    <inertia ixx="0.611797" iyy="0.597598" izz="0.154569" ixy="-7e-06" iyz="5e-06" ixz="0.016258"/>
+  </inertial>
+  <visual>
+    <origin xyz="0.06485 -0.10315 -0.52765" rpy="0 0 0"/>
+    <geometry>
+      <mesh filename="package://roomac_description/meshes/frame_1.stl" scale="0.001 0.001 0.001"/>
+    </geometry>
+    <material name="silver"/>
+  </visual>
+  <collision>
+    <origin xyz="0.06485 -0.10315 -0.52765" rpy="0 0 0"/>
+    <geometry>
+      <mesh filename="package://roomac_description/meshes/frame_1.stl" scale="0.001 0.001 0.001"/>
+    </geometry>
+  </collision>
+</link>
+<link name="eye_left_1">
+  <inertial>
+    <origin xyz="0.006260241058239718 3.517735615299333e-08 -3.5598063252706424e-07" rpy="0 0 0"/>
+    <mass value="0.12003246414388502"/>
+    <inertia ixx="0.000115" iyy="5.8e-05" izz="5.8e-05" ixy="-0.0" iyz="0.0" ixz="-0.0"/>
+  </inertial>
+  <visual>
+    <origin xyz="0.0825 -0.056021 -1.083347" rpy="0 0 0"/>
+    <geometry>
+      <mesh filename="package://roomac_description/meshes/eye_left_1.stl" scale="0.001 0.001 0.001"/>
+    </geometry>
+    <material name="silver"/>
+  </visual>
+  <collision>
+    <origin xyz="0.0825 -0.056021 -1.083347" rpy="0 0 0"/>
+    <geometry>
+      <mesh filename="package://roomac_description/meshes/eye_left_1.stl" scale="0.001 0.001 0.001"/>
+    </geometry>
+  </collision>
+</link>
+<link name="elbow_right_1">
+  <inertial>
+    <origin xyz="0.0005136115276251074 3.101290486640096e-07 -0.023818498356463658" rpy="0 0 0"/>
+    <mass value="0.4245429501284504"/>
+    <inertia ixx="0.000153" iyy="0.00017" izz="7.8e-05" ixy="0.0" iyz="-0.0" ixz="4e-06"/>
+  </inertial>
+  <visual>
+    <origin xyz="0.1135 0.243979 -0.774925" rpy="0 0 0"/>
+    <geometry>
+      <mesh filename="package://roomac_description/meshes/elbow_right_1.stl" scale="0.001 0.001 0.001"/>
+    </geometry>
+    <material name="silver"/>
+  </visual>
+  <collision>
+    <origin xyz="0.1135 0.243979 -0.774925" rpy="0 0 0"/>
+    <geometry>
+      <mesh filename="package://roomac_description/meshes/elbow_right_1.stl" scale="0.001 0.001 0.001"/>
+    </geometry>
+  </collision>
+</link>
+<link name="elbow_wrist_right_1">
+  <inertial>
+    <origin xyz="-0.019371175261057166 -0.0012025990213214988 -0.09242894014376357" rpy="0 0 0"/>
+    <mass value="0.6102002908923237"/>
+    <inertia ixx="0.00103" iyy="0.001092" izz="0.000114" ixy="0.0" iyz="-1.8e-05" ixz="-1e-05"/>
+  </inertial>
+  <visual>
+    <origin xyz="0.0925 0.243979 -0.733443" rpy="0 0 0"/>
+    <geometry>
+      <mesh filename="package://roomac_description/meshes/elbow_wrist_right_1.stl" scale="0.001 0.001 0.001"/>
+    </geometry>
+    <material name="silver"/>
+  </visual>
+  <collision>
+    <origin xyz="0.0925 0.243979 -0.733443" rpy="0 0 0"/>
+    <geometry>
+      <mesh filename="package://roomac_description/meshes/elbow_wrist_right_1.stl" scale="0.001 0.001 0.001"/>
+    </geometry>
+  </collision>
+</link>
+<link name="caster_tire_right_1">
+  <inertial>
+    <origin xyz="-2.3869795029440866e-15 -2.498001805406602e-16 5.398459457239824e-15" rpy="0 0 0"/>
+    <mass value="0.030691695984031726"/>
+    <inertia ixx="2.1e-05" iyy="3.7e-05" izz="2.1e-05" ixy="-0.0" iyz="-0.0" ixz="-0.0"/>
+  </inertial>
+  <visual>
+    <origin xyz="0.325 0.161 0.105" rpy="0 0 0"/>
+    <geometry>
+      <mesh filename="package://roomac_description/meshes/caster_tire_right_1.stl" scale="0.001 0.001 0.001"/>
+    </geometry>
+    <material name="silver"/>
+  </visual>
+  <collision>
+    <origin xyz="0.325 0.161 0.105" rpy="0 0 0"/>
+    <geometry>
+      <mesh filename="package://roomac_description/meshes/caster_tire_right_1.stl" scale="0.001 0.001 0.001"/>
+    </geometry>
+  </collision>
+</link>
+<link name="caster_tire_left_1">
+  <inertial>
+    <origin xyz="-2.55351295663786e-15 -7.494005416219807e-16 3.969047313034935e-15" rpy="0 0 0"/>
+    <mass value="0.03069169598403176"/>
+    <inertia ixx="2.1e-05" iyy="3.7e-05" izz="2.1e-05" ixy="-0.0" iyz="-0.0" ixz="-0.0"/>
+  </inertial>
+  <visual>
+    <origin xyz="0.325 -0.161 0.105" rpy="0 0 0"/>
+    <geometry>
+      <mesh filename="package://roomac_description/meshes/caster_tire_left_1.stl" scale="0.001 0.001 0.001"/>
+    </geometry>
+    <material name="silver"/>
+  </visual>
+  <collision>
+    <origin xyz="0.325 -0.161 0.105" rpy="0 0 0"/>
+    <geometry>
+      <mesh filename="package://roomac_description/meshes/caster_tire_left_1.stl" scale="0.001 0.001 0.001"/>
+    </geometry>
+  </collision>
+</link>
+<link name="wheel_tire_right_1">
+  <inertial>
+    <origin xyz="-1.0835776720341528e-15 -2.220446049250313e-16 1.4210854715202004e-16" rpy="0 0 0"/>
+    <mass value="1.1787904912381322"/>
+    <inertia ixx="0.009661" iyy="0.018749" izz="0.009661" ixy="-0.0" iyz="-0.0" ixz="-0.0"/>
+  </inertial>
+  <visual>
+    <origin xyz="0.0 0.257 -0.0" rpy="0 0 0"/>
+    <geometry>
+      <mesh filename="package://roomac_description/meshes/wheel_tire_right_1.stl" scale="0.001 0.001 0.001"/>
+    </geometry>
+    <material name="silver"/>
+  </visual>
+  <collision>
+    <origin xyz="0.0 0.257 -0.0" rpy="0 0 0"/>
+    <geometry>
+      <mesh filename="package://roomac_description/meshes/wheel_tire_right_1.stl" scale="0.001 0.001 0.001"/>
+    </geometry>
+  </collision>
+</link>
+<link name="wheel_tire_left_1">
+  <inertial>
+    <origin xyz="-1.3677947663381929e-15 -6.106226635438361e-16 1.4210854715202004e-16" rpy="0 0 0"/>
+    <mass value="1.178790491238132"/>
+    <inertia ixx="0.009661" iyy="0.018749" izz="0.009661" ixy="-0.0" iyz="-0.0" ixz="-0.0"/>
+  </inertial>
+  <visual>
+    <origin xyz="0.0 -0.257 0.0" rpy="0 0 0"/>
+    <geometry>
+      <mesh filename="package://roomac_description/meshes/wheel_tire_left_1.stl" scale="0.001 0.001 0.001"/>
+    </geometry>
+    <material name="silver"/>
+  </visual>
+  <collision>
+    <origin xyz="0.0 -0.257 0.0" rpy="0 0 0"/>
+    <geometry>
+      <mesh filename="package://roomac_description/meshes/wheel_tire_left_1.stl" scale="0.001 0.001 0.001"/>
+    </geometry>
+  </collision>
+</link>
+<link name="base_link_frames_1">
+  <inertial>
+    <origin xyz="0.05219682070735798 0.09908927488444497 0.4776891193965433" rpy="0 0 0"/>
+    <mass value="2.6725201136516104"/>
+    <inertia ixx="0.264075" iyy="0.253077" izz="0.065833" ixy="1e-06" iyz="-8e-06" ixz="-0.022361"/>
+  </inertial>
+  <visual>
+    <origin xyz="0.223282 0.099058 0.0075" rpy="0 0 0"/>
+    <geometry>
+      <mesh filename="package://roomac_description/meshes/base_link_frames_1.stl" scale="0.001 0.001 0.001"/>
+    </geometry>
+    <material name="silver"/>
+  </visual>
+  <collision>
+    <origin xyz="0.223282 0.099058 0.0075" rpy="0 0 0"/>
+    <geometry>
+      <mesh filename="package://roomac_description/meshes/base_link_frames_1.stl" scale="0.001 0.001 0.001"/>
+    </geometry>
+  </collision>
+</link>
+<link name="shoulder_elbow_gear_right_1">
+  <inertial>
+    <origin xyz="4.458388786428291e-05 -3.227258993376836e-08 0.001208993450583895" rpy="0 0 0"/>
+    <mass value="0.48507719135410154"/>
+    <inertia ixx="0.000258" iyy="0.000141" izz="0.000153" ixy="-0.0" iyz="0.0" ixz="0.0"/>
+  </inertial>
+  <visual>
+    <origin xyz="0.113 0.243979 -0.9345" rpy="0 0 0"/>
+    <geometry>
+      <mesh filename="package://roomac_description/meshes/shoulder_elbow_gear_right_1.stl" scale="0.001 0.001 0.001"/>
+    </geometry>
+    <material name="silver"/>
+  </visual>
+  <collision>
+    <origin xyz="0.113 0.243979 -0.9345" rpy="0 0 0"/>
+    <geometry>
+      <mesh filename="package://roomac_description/meshes/shoulder_elbow_gear_right_1.stl" scale="0.001 0.001 0.001"/>
+    </geometry>
+  </collision>
+</link>
+<link name="wrist_right_1">
+  <inertial>
+    <origin xyz="0.02427263159088615 -0.0008946909413816428 -0.023520440866137693" rpy="0 0 0"/>
+    <mass value="0.15933052176631626"/>
+    <inertia ixx="6.4e-05" iyy="0.000118" izz="6.6e-05" ixy="0.0" iyz="-2e-06" ixz="1.5e-05"/>
+  </inertial>
+  <visual>
+    <origin xyz="0.139354 0.243979 -0.603601" rpy="0 0 0"/>
+    <geometry>
+      <mesh filename="package://roomac_description/meshes/wrist_right_1.stl" scale="0.001 0.001 0.001"/>
+    </geometry>
+    <material name="silver"/>
+  </visual>
+  <collision>
+    <origin xyz="0.139354 0.243979 -0.603601" rpy="0 0 0"/>
+    <geometry>
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
File: roomac_description/urdf/roomac_gripper_real.xacro (robot description, xacro)
@@ -7,23 +7,73 @@
     <child link="gripper_right_grip"/>
   </joint>
-  <link name="gripper_right_1">
-    <inertial>
-      <origin rpy="0 0 0" xyz="0.0003095175801113986 0.0006959817920443867 -0.037223762933811466"/>
-      <mass value="0.2826112434389509"/>
-      <inertia ixx="0.000262" ixy="4e-06" ixz="7e-06" iyy="0.000181" iyz="-4e-06" izz="0.000107"/>
-    </inertial>
-    <visual>
-      <origin rpy="0 0 0" xyz="0.111135 0.244052 -0.558565"/>
-      <geometry>
-        <mesh filename="package://roomac_description/meshes/gripper_right_1.stl" scale="0.001 0.001 0.001"/>
-      </geometry>
-      <material name="silver"/>
-    </visual>
-    <collision>
-      <origin rpy="0 0 0" xyz="0.111135 0.244052 -0.558565"/>
-      <geometry>
-        <mesh filename="package://roomac_description/meshes/gripper_right_1.stl" scale="0.001 0.001 0.001"/>
-      </geometry>
-    </collision>
-  </link>
+<link name="gripper_right_1">
+  <inertial>
+    <origin xyz="-0.00024163561260628907 0.001034172528649041 -0.024005885240587554" rpy="0 0 0"/>
+    <mass value="0.20788263258389922"/>
+    <inertia ixx="8.7e-05" iyy="5.3e-05" izz="5.8e-05" ixy="4e-06" iyz="-1e-06" ixz="3e-06"/>
+  </inertial>
+  <visual>
+    <origin xyz="0.114635 0.244052 -0.544809" rpy="0 0 0"/>
+    <geometry>
+      <mesh filename="package://roomac_description/meshes/gripper_right_1.stl" scale="0.001 0.001 0.001"/>
+    </geometry>
+    <material name="silver"/>
+  </visual>
+  <collision>
+    <origin xyz="0.114635 0.244052 -0.544809" rpy="0 0 0"/>
+    <geometry>
+      <mesh filename="package://roomac_description/meshes/gripper_right_1.stl" scale="0.001 0.001 0.001"/>
+    </geometry>
+  </collision>
+</link>
+<link name="gripper_finger_1_right_1">
+  <inertial>
+    <origin xyz="0.004500248654849631 0.005686730533079498 -0.01101605906930514" rpy="0 0 0"/>
+    <mass value="0.03746064390067365"/>
+    <inertia ixx="1.2e-05" iyy="1e-05" izz="2e-06" ixy="-0.0" iyz="4e-06" ixz="-0.0"/>
+  </inertial>
+  <visual>
+    <origin xyz="0.117385 0.274314 -0.487702" rpy="0 0 0"/>
+    <geometry>
+      <mesh filename="package://roomac_description/meshes/gripper_finger_1_right_1.stl" scale="0.001 0.001 0.001"/>
+    </geometry>
+    <material name="silver"/>
+  </visual>
+  <collision>
+    <origin xyz="0.117385 0.274314 -0.487702" rpy="0 0 0"/>
+    <geometry>
+      <mesh filename="package://roomac_description/meshes/gripper_finger_1_right_1.stl" scale="0.001 0.001 0.001"/>
+    </geometry>
+  </collision>
+</link>
+<link name="gripper_finger_2_right_1">
+  <inertial>
+    <origin xyz="0.00450024860853869 -0.005494466336699089 -0.011113636952014339" rpy="0 0 0"/>
+    <mass value="0.037460643900623564"/>
+    <inertia ixx="1.2e-05" iyy="1e-05" izz="2e-06" ixy="-0.0" iyz="-4e-06" ixz="-0.0"/>
+  </inertial>
+  <visual>
+    <origin xyz="0.117385 0.214585 -0.487702" rpy="0 0 0"/>
+    <geometry>
+      <mesh filename="package://roomac_description/meshes/gripper_finger_2_right_1.stl" scale="0.001 0.001 0.001"/>
+    </geometry>
+    <material name="silver"/>
+  </visual>
+  <collision>
+    <origin xyz="0.117385 0.214585 -0.487702" rpy="0 0 0"/>
+    <geometry>
+      <mesh filename="package://roomac_description/meshes/gripper_finger_2_right_1.stl" scale="0.001 0.001 0.001"/>
+    </geometry>
+  </collision>
+</link>
+<joint name="gripper_finger_r_right" type="fixed">
+  <origin xyz="-0.00275 -0.030262 -0.057107" rpy="0 0 0"/>
+  <parent link="gripper_right_1"/>
+  <child link="gripper_finger_1_right_1"/>
+</joint>
+<joint name="gripper_finger_l_right" type="fixed">
+  <origin xyz="-0.00275 0.029467 -0.057107" rpy="0 0 0"/>
+  <parent link="gripper_right_1"/>
+  <child link="gripper_finger_2_right_1"/>
+</joint>
 </robot>

Commit message: Update artag position

File: roomac_description/urdf/roomac_body.xacro (robot description, xacro)
@@ -856,4 +856,5 @@
 </joint>
 <joint name="kinect_joint" type="fixed">
+  <!-- todo: update kinect position -->
 		<origin rpy="0 ${(31.513/180.)*pi} 0" xyz="-0.108561 0.039543 0.479024"/>
 		<parent link="base_link"/>
@@ -870,6 +871,5 @@
 </link>
 <joint name="artag_joint" type="fixed">
-    <!-- Real z position is 0.972, but I had to add 12mm (height of plywood) - this urdf is older - pre base rework -->
-    <origin rpy="0 0 0" xyz="-0.149 -0.125 0.984"/>
+    <origin rpy="0 0 0" xyz="-0.149 -0.125 0.972"/>
     <parent link="base_link"/>
     <child link="artag_link"/>
