Commit message: Fix wheel direction of revolute

File: roomac_description/urdf/roomac_body.xacro (robot description, xacro)
@@ -692,5 +692,5 @@
   <parent link="base_link"/>
   <child link="wheel_right_1"/>
-  <axis xyz="0.0 -1.0 -0.0"/>
+  <axis xyz="0.0 1.0 -0.0"/>
 </joint>
 <joint name="wheel_left" type="continuous">

Commit message: Cleanup xacro

File: roomac_description/urdf/roomac_body.xacro (robot description, xacro)
@@ -1,31 +1,130 @@
 <?xml version="1.0" ?>
 <robot name="roomac" xmlns:xacro="http://www.ros.org/wiki/xacro">
+<!-- BODY -->
 <link name="base_link" />
+<!-- Additional link needed to solve moveit warning (as far as I know it shouldn't cause any issue as I'm not using KDL, but still better to solve it): -->
+<!-- The root link base_link has an inertia specified in the URDF, but KDL does not support a root link with an inertia.  As a workaround, you can add an extra dummy link to your URDF. -->
+<link name="robot_base_1">
+  <inertial>
+    <origin xyz="-0.18736789633381332 0.0015304678388801296 0.2632175316600572" rpy="0 0 0"/>
+    <mass value="31.013883468506926"/>
+    <inertia ixx="2.674027" iyy="2.737864" izz="0.665771" ixy="-0.003283" iyz="-0.013126" ixz="-0.310987"/>
+  </inertial>
+  <visual>
+    <origin xyz="0 0 0" rpy="0 0 0"/>
+    <geometry>
+      <mesh filename="package://roomac_description/meshes/base_link.stl" scale="0.001 0.001 0.001"/>
+    </geometry>
+    <material name="black"/>
+  </visual>
+  <collision>
+    <origin xyz="0 0 0" rpy="0 0 0"/>
+    <geometry>
+      <mesh filename="package://roomac_description/meshes/base_link.stl" scale="0.001 0.001 0.001"/>
+    </geometry>
+  </collision>
+</link>
+<link name="base_link_frames_1">
+  <inertial>
+    <origin xyz="0.05219682070735798 0.09908927488444497 0.4776891193965433" rpy="0 0 0"/>
+    <mass value="2.6725201136516104"/>
+    <inertia ixx="0.264075" iyy="0.253077" izz="0.065833" ixy="1e-06" iyz="-8e-06" ixz="-0.022361"/>
+  </inertial>
+  <visual>
+    <origin xyz="0.223282 0.099058 0.0075" rpy="0 0 0"/>
+    <geometry>
+      <mesh filename="package://roomac_description/meshes/base_link_frames_1.stl" scale="0.001 0.001 0.001"/>
+    </geometry>
+    <material name="white"/>
+  </visual>
+  <collision>
+    <origin xyz="0.223282 0.099058 0.0075" rpy="0 0 0"/>
+    <geometry>
+      <mesh filename="package://roomac_description/meshes/base_link_frames_1.stl" scale="0.001 0.001 0.001"/>
+    </geometry>
+  </collision>
+</link>
+<link name="frame_1">
+  <inertial>
+    <origin xyz="-0.06363233755923882 -0.10316506754069626 -0.18305645699853168" rpy="0 0 0"/>
+    <mass value="4.866480003493675"/>
+    <inertia ixx="0.611797" iyy="0.597598" izz="0.154569" ixy="-7e-06" iyz="5e-06" ixz="0.016258"/>
+  </inertial>
+  <visual>
+    <origin xyz="0.06485 -0.10315 -0.52765" rpy="0 0 0"/>
+    <geometry>
+      <mesh filename="package://roomac_description/meshes/frame_1.stl" scale="0.001 0.001 0.001"/>
+    </geometry>
+    <material name="silver"/>
+  </visual>
+  <collision>
+    <origin xyz="0.06485 -0.10315 -0.52765" rpy="0 0 0"/>
+    <geometry>
+      <mesh filename="package://roomac_description/meshes/frame_1.stl" scale="0.001 0.001 0.001"/>
+    </geometry>
+  </collision>
+</link>
 <joint name="robot_base" type="fixed">
   <parent link="base_link"/>
   <child link="robot_base_1"/>
 </joint>
-<!-- Additional link needed to solve moveit warning (as far as I know it shouldn't cause any issue as I'm not using KDL, but still better to solve it): -->
-<!-- The root link base_link has an inertia specified in the URDF, but KDL does not support a root link with an inertia.  As a workaround, you can add an extra dummy link to your URDF. -->
-<link name="robot_base_1">
-  <inertial>
-    <origin xyz="-0.18736789633381332 0.0015304678388801296 0.2632175316600572" rpy="0 0 0"/>
-    <mass value="31.013883468506926"/>
-    <inertia ixx="2.674027" iyy="2.737864" izz="0.665771" ixy="-0.003283" iyz="-0.013126" ixz="-0.310987"/>
-  </inertial>
-  <visual>
-    <origin xyz="0 0 0" rpy="0 0 0"/>
-    <geometry>
-      <mesh filename="package://roomac_description/meshes/base_link.stl" scale="0.001 0.001 0.001"/>
-    </geometry>
-    <material name="black"/>
-  </visual>
-  <collision>
-    <origin xyz="0 0 0" rpy="0 0 0"/>
-    <geometry>
-      <mesh filename="package://roomac_description/meshes/base_link.stl" scale="0.001 0.001 0.001"/>
-    </geometry>
-  </collision>
-</link>
+<joint name="base_link_frames" type="fixed">
+  <origin xyz="-0.223282 -0.099058 -0.0075" rpy="0 0 0"/>
+  <parent link="base_link"/>
+  <child link="base_link_frames_1"/>
+</joint>
+<joint name="frame" type="fixed">
+  <origin xyz="-0.06485 0.10315 0.52765" rpy="0 0 0"/>
+  <parent link="base_link"/>
+  <child link="frame_1"/>
+</joint>
+<!-- KINECT -->
+<link name="camera_link" />
+<joint name="kinect_joint" type="fixed">
+  <!-- todo: update kinect position -->
+  <origin rpy="0 ${(31.513/180.)*pi} 0" xyz="-0.108561 0.039543 0.479024"/>
+  <parent link="base_link"/>
+  <child link="camera_link"/>
+</joint>
+<!-- IMU -->
+<link name="imu" />
+<joint name="imu_joint" type="fixed">
+  <origin rpy="0 0 0" xyz="-0.09873 -0.0375 0.0305"/>
+  <parent link="base_link"/>
+  <child link="imu"/>
+</joint>
+<!-- ARTAG -->
+<link name="artag_link" />
+<link name="artag_link_bundle_visual">
+  <inertial>
+    <origin rpy="0 0 0" xyz="0 0 0"/>
+    <mass value="0.1"/>
+    <inertia ixx="0" ixy="-0.0" ixz="0.0" iyy="0" iyz="0.0" izz="0"/>
+  </inertial>
+  <visual name="visual">
+    <origin rpy="0 0 0" xyz="0.0 0.0 0.0"/>
+    <geometry>
+      <mesh filename="package://roomac_description/materials/artag_bundle.dae" scale="3.142857143 1.2 0.001"/>
+    </geometry>
+    <material name="artag"/>
+  </visual>
+  <collision>
+    <origin rpy="0 0 0" xyz="0.0 0.0 0.0"/>
+    <geometry>
+      <mesh filename="package://roomac_description/materials/artag_bundle.dae" scale="3.142857143 1.2 0.001"/>
+    </geometry>
+  </collision>
+</link>
+<joint name="artag_joint" type="fixed">
+  <origin rpy="0 0 0" xyz="-0.149 -0.125 0.972"/>
+  <parent link="base_link"/>
+  <child link="artag_link"/>
+</joint>
+<joint name="artag_joint_bundle_visual" type="fixed">
+  <origin rpy="0 0 0" xyz="0.01 0.0 0"/>
+  <parent link="artag_link"/>
+  <child link="artag_link_bundle_visual"/>
+</joint>
+<!-- CASTERS -->
 <link name="caster_right_1">
   <inertial>
@@ -68,164 +167,4 @@
   </collision>
 </link>
-<link name="hub_right_1">
-  <inertial>
-    <origin xyz="-1.789765220804318e-06 0.012712108125801869 3.1361035183559637e-06" rpy="0 0 0"/>
-    <mass value="0.09451094240372103"/>
-    <inertia ixx="5e-05" iyy="8.5e-05" izz="5e-05" ixy="0.0" iyz="-0.0" ixz="0.0"/>
-  </inertial>
-  <visual>
-    <origin xyz="0.0 0.246 0.0" rpy="0 0 0"/>
-    <geometry>
-      <mesh filename="package://roomac_description/meshes/hub_right_1.stl" scale="0.001 0.001 0.001"/>
-    </geometry>
-    <material name="black"/>
-  </visual>
-  <collision>
-    <origin xyz="0.0 0.246 0.0" rpy="0 0 0"/>
-    <geometry>
-      <mesh filename="package://roomac_description/meshes/hub_right_1.stl" scale="0.001 0.001 0.001"/>
-    </geometry>
-  </collision>
-</link>
-<link name="hub_left_1">
-  <inertial>
-    <origin xyz="-1.7897652210308038e-06 -0.012712108125801591 3.1361035183086937e-06" rpy="0 0 0"/>
-    <mass value="0.09451094240372113"/>
-    <inertia ixx="5e-05" iyy="8.5e-05" izz="5e-05" ixy="-0.0" iyz="0.0" ixz="0.0"/>
-  </inertial>
-  <visual>
-    <origin xyz="0.0 -0.246 0.0" rpy="0 0 0"/>
-    <geometry>
-      <mesh filename="package://roomac_description/meshes/hub_left_1.stl" scale="0.001 0.001 0.001"/>
-    </geometry>
-    <material name="black"/>
-  </visual>
-  <collision>
-    <origin xyz="0.0 -0.246 0.0" rpy="0 0 0"/>
-    <geometry>
-      <mesh filename="package://roomac_description/meshes/hub_left_1.stl" scale="0.001 0.001 0.001"/>
-    </geometry>
-  </collision>
-</link>
-<link name="wheel_right_1">
-  <inertial>
-    <origin xyz="-4.446890699227879e-08 -0.046359989716390604 2.8955374773431687e-08" rpy="0 0 0"/>
-    <mass value="1.4792126361607076"/>
-    <inertia ixx="0.006728" iyy="0.012762" izz="0.006728" ixy="0.0" iyz="-0.0" ixz="0.0"/>
-  </inertial>
-  <visual>
-    <origin xyz="-0.0 0.21064 0.0" rpy="0 0 0"/>
-    <geometry>
-      <mesh filename="package://roomac_description/meshes/wheel_right_1.stl" scale="0.001 0.001 0.001"/>
-    </geometry>
-    <material name="silver"/>
-  </visual>
-  <collision>
-    <origin xyz="-0.0 0.21064 0.0" rpy="0 0 0"/>
-    <geometry>
-      <mesh filename="package://roomac_description/meshes/wheel_right_1.stl" scale="0.001 0.001 0.001"/>
-    </geometry>
-  </collision>
-</link>
-<link name="wheel_left_1">
-  <inertial>
-    <origin xyz="-3.1796540813644466e-08 0.04035998903806015 1.6110734861740638e-08" rpy="0 0 0"/>
-    <mass value="1.4792124768984427"/>
-    <inertia ixx="0.006728" iyy="0.012762" izz="0.006728" ixy="0.0" iyz="0.0" ixz="0.0"/>
-  </inertial>
-  <visual>
-    <origin xyz="0.0 -0.21664 0.0" rpy="0 0 0"/>
-    <geometry>
-      <mesh filename="package://roomac_description/meshes/wheel_left_1.stl" scale="0.001 0.001 0.001"/>
-    </geometry>
-    <material name="silver"/>
-  </visual>
-  <collision>
-    <origin xyz="0.0 -0.21664 0.0" rpy="0 0 0"/>
-    <geometry>
-      <mesh filename="package://roomac_description/meshes/wheel_left_1.stl" scale="0.001 0.001 0.001"/>
-    </geometry>
-  </collision>
-</link>
-<link name="frame_1">
-  <inertial>
-    <origin xyz="-0.06363233755923882 -0.10316506754069626 -0.18305645699853168" rpy="0 0 0"/>
-    <mass value="4.866480003493675"/>
-    <inertia ixx="0.611797" iyy="0.597598" izz="0.154569" ixy="-7e-06" iyz="5e-06" ixz="0.016258"/>
-  </inertial>
-  <visual>
-    <origin xyz="0.06485 -0.10315 -0.52765" rpy="0 0 0"/>
-    <geometry>
-      <mesh filename="package://roomac_description/meshes/frame_1.stl" scale="0.001 0.001 0.001"/>
-    </geometry>
-    <material name="silver"/>
-  </visual>
-  <collision>
-    <origin xyz="0.06485 -0.10315 -0.52765" rpy="0 0 0"/>
-    <geometry>
-      <mesh filename="package://roomac_description/meshes/frame_1.stl" scale="0.001 0.001 0.001"/>
-    </geometry>
-  </collision>
-</link>
-<link name="eye_left_1">
-  <inertial>
-    <origin xyz="0.006260241058239718 3.517735615299333e-08 -3.5598063252706424e-07" rpy="0 0 0"/>
-    <mass value="0.12003246414388502"/>
-    <inertia ixx="0.000115" iyy="5.8e-05" izz="5.8e-05" ixy="-0.0" iyz="0.0" ixz="-0.0"/>
-  </inertial>
-  <visual>
-    <origin xyz="0.0825 -0.056021 -1.083347" rpy="0 0 0"/>
-    <geometry>
-      <mesh filename="package://roomac_description/meshes/eye_left_1.stl" scale="0.001 0.001 0.001"/>
-    </geometry>
-    <material name="white"/>
-  </visual>
-  <collision>
-    <origin xyz="0.0825 -0.056021 -1.083347" rpy="0 0 0"/>
-    <geometry>
-      <mesh filename="package://roomac_description/meshes/eye_left_1.stl" scale="0.001 0.001 0.001"/>
-    </geometry>
-  </collision>
-</link>
-<link name="elbow_right_1">
-  <inertial>
-    <origin xyz="0.0005136115276251074 3.101290486640096e-07 -0.023818498356463658" rpy="0 0 0"/>
-    <mass value="0.4245429501284504"/>
-    <inertia ixx="0.000153" iyy="0.00017" izz="7.8e-05" ixy="0.0" iyz="-0.0" ixz="4e-06"/>
-  </inertial>
-  <visual>
-    <origin xyz="0.1135 0.243979 -0.774925" rpy="0 0 0"/>
-    <geometry>
-      <mesh filename="package://roomac_description/meshes/elbow_right_1.stl" scale="0.001 0.001 0.001"/>
-    </geometry>
-    <material name="black"/>
-  </visual>
-  <collision>
-    <origin xyz="0.1135 0.243979 -0.774925" rpy="0 0 0"/>
-    <geometry>
-      <mesh filename="package://roomac_description/meshes/elbow_right_1.stl" scale="0.001 0.001 0.001"/>
-    </geometry>
-  </collision>
-</link>
-<link name="elbow_wrist_right_1">
-  <inertial>
-    <origin xyz="-0.019371175261057166 -0.0012025990213214988 -0.09242894014376357" rpy="0 0 0"/>
-    <mass value="0.6102002908923237"/>
-    <inertia ixx="0.00103" iyy="0.001092" izz="0.000114" ixy="0.0" iyz="-1.8e-05" ixz="-1e-05"/>
-  </inertial>
-  <visual>
-    <origin xyz="0.0925 0.243979 -0.733443" rpy="0 0 0"/>
-    <geometry>
-      <mesh filename="package://roomac_description/meshes/elbow_wrist_right_1.stl" scale="0.001 0.001 0.001"/>
-    </geometry>
-    <material name="black"/>
-  </visual>
-  <collision>
-    <origin xyz="0.0925 0.243979 -0.733443" rpy="0 0 0"/>
-    <geometry>
-      <mesh filename="package://roomac_description/meshes/elbow_wrist_right_1.stl" scale="0.001 0.001 0.001"/>
-    </geometry>
-  </collision>
-</link>
 <link name="caster_tire_right_1">
   <inertial>
@@ -265,404 +204,4 @@
     <geometry>
       <mesh filename="package://roomac_description/meshes/caster_tire_left_1.stl" scale="0.001 0.001 0.001"/>
-    </geometry>
-  </collision>
-</link>
-<link name="wheel_tire_right_1">
-  <inertial>
-    <origin xyz="-1.0835776720341528e-15 -2.220446049250313e-16 1.4210854715202004e-16" rpy="0 0 0"/>
-    <mass value="1.1787904912381322"/>
-    <inertia ixx="0.009661" iyy="0.018749" izz="0.009661" ixy="-0.0" iyz="-0.0" ixz="-0.0"/>
-  </inertial>
-  <visual>
-    <origin xyz="0.0 0.257 -0.0" rpy="0 0 0"/>
-    <geometry>
-      <mesh filename="package://roomac_description/meshes/wheel_tire_right_1.stl" scale="0.001 0.001 0.001"/>
-    </geometry>
-    <material name="black"/>
-  </visual>
-  <collision>
-    <origin xyz="0.0 0.257 -0.0" rpy="0 0 0"/>
-    <geometry>
-      <mesh filename="package://roomac_description/meshes/wheel_tire_right_1.stl" scale="0.001 0.001 0.001"/>
-    </geometry>
-  </collision>
-</link>
-<link name="wheel_tire_left_1">
-  <inertial>
-    <origin xyz="-1.3677947663381929e-15 -6.106226635438361e-16 1.4210854715202004e-16" rpy="0 0 0"/>
-    <mass value="1.178790491238132"/>
-    <inertia ixx="0.009661" iyy="0.018749" izz="0.009661" ixy="-0.0" iyz="-0.0" ixz="-0.0"/>
-  </inertial>
-  <visual>
-    <origin xyz="0.0 -0.257 0.0" rpy="0 0 0"/>
-    <geometry>
-      <mesh filename="package://roomac_description/meshes/wheel_tire_left_1.stl" scale="0.001 0.001 0.001"/>
-    </geometry>
-    <material name="black"/>
-  </visual>
-  <collision>
-    <origin xyz="0.0 -0.257 0.0" rpy="0 0 0"/>
-    <geometry>
-      <mesh filename="package://roomac_description/meshes/wheel_tire_left_1.stl" scale="0.001 0.001 0.001"/>
-    </geometry>
-  </collision>
-</link>
-<link name="base_link_frames_1">
-  <inertial>
-    <origin xyz="0.05219682070735798 0.09908927488444497 0.4776891193965433" rpy="0 0 0"/>
-    <mass value="2.6725201136516104"/>
-    <inertia ixx="0.264075" iyy="0.253077" izz="0.065833" ixy="1e-06" iyz="-8e-06" ixz="-0.022361"/>
-  </inertial>
-  <visual>
-    <origin xyz="0.223282 0.099058 0.0075" rpy="0 0 0"/>
-    <geometry>
-      <mesh filename="package://roomac_description/meshes/base_link_frames_1.stl" scale="0.001 0.001 0.001"/>
-    </geometry>
-    <material name="white"/>
-  </visual>
-  <collision>
-    <origin xyz="0.223282 0.099058 0.0075" rpy="0 0 0"/>
-    <geometry>
-      <mesh filename="package://roomac_description/meshes/base_link_frames_1.stl" scale="0.001 0.001 0.001"/>
-    </geometry>
-  </collision>
-</link>
-<link name="shoulder_elbow_gear_right_1">
-  <inertial>
-    <origin xyz="4.458388786428291e-05 -3.227258993376836e-08 0.001208993450583895" rpy="0 0 0"/>
-    <mass value="0.48507719135410154"/>
-    <inertia ixx="0.000258" iyy="0.000141" izz="0.000153" ixy="-0.0" iyz="0.0" ixz="0.0"/>
-  </inertial>
-  <visual>
-    <origin xyz="0.113 0.243979 -0.9345" rpy="0 0 0"/>
-    <geometry>
-      <mesh filename="package://roomac_description/meshes/shoulder_elbow_gear_right_1.stl" scale="0.001 0.001 0.001"/>
-    </geometry>
-    <material name="black"/>
-  </visual>
-  <collision>
-    <origin xyz="0.113 0.243979 -0.9345" rpy="0 0 0"/>
-    <geometry>
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
Commit message: Fix shoulder pitch rotate direction

File: roomac_description/urdf/roomac_body.xacro (robot description, xacro)
@@ -679,5 +679,5 @@
   <parent link="shoulder_base_right_1"/>
   <child link="shoulder_right_1"/>
-  <axis xyz="0.0 -1.0 0.0"/>
+  <axis xyz="0.0 1.0 0.0"/>
   <limit effort="30" velocity="1.0" lower="-2.390" upper="0.489" />
 </joint>

Commit message: Update kinect's position

File: roomac_description/urdf/roomac_body.xacro (robot description, xacro)
@@ -82,6 +82,6 @@
 <link name="camera_link" />
 <joint name="kinect_joint" type="fixed">
-  <!-- todo: update kinect position -->
-  <origin rpy="0 ${(31.513/180.)*pi} 0" xyz="-0.108561 0.039543 0.479024"/>
+  <!-- 0.03 comes from calibration - ground was slightly tilted and I calibrated it in rviz to be parallel  -->
+  <origin rpy="0 ${(31.513/180.)*pi - 0.03} 0" xyz="-0.108561 0.039543 0.467024"/>
   <parent link="base_link"/>
   <child link="camera_link"/>

Commit message: Add base footprint and publish maps in this frame
it is base link projected on the ground, maps visualization in rviz looks better when they are on the actual ground

File: roomac_description/urdf/roomac_body.xacro (robot description, xacro)
@@ -3,4 +3,5 @@
 <!-- BODY -->
 <link name="base_link" />
+<link name="base_footprint" />
 <!-- Additional link needed to solve moveit warning (as far as I know it shouldn't cause any issue as I'm not using KDL, but still better to solve it): -->
 <!-- The root link base_link has an inertia specified in the URDF, but KDL does not support a root link with an inertia.  As a workaround, you can add an extra dummy link to your URDF. -->
@@ -65,4 +66,9 @@
   </collision>
 </link>
+<joint name="base_joint" type="fixed">
+  <origin rpy="0 0 0" xyz="0 0 0.145"/>
+  <parent link="base_footprint"/>
+  <child link="base_link"/>
+</joint>
 <joint name="robot_base" type="fixed">
   <parent link="base_link"/>
