Commit message: Update urdf to use model with fewer parts (some of them converted to dae)

File: roomac_description/urdf/roomac_body.xacro (robot description, xacro)
@@ -1,4 +1,6 @@
 <?xml version="1.0" ?>
 <robot name="roomac" xmlns:xacro="http://www.ros.org/wiki/xacro">
+<!-- todo cleanup axis in urdf -->
+<!-- todo remove material from dae -->
 <!-- BODY -->
 <link name="base_link" />
@@ -8,7 +10,7 @@
 <link name="robot_base_1">
   <inertial>
-    <origin xyz="-0.18736789633381332 0.0015304678388801296 0.2632175316600572" rpy="0 0 0"/>
-    <mass value="31.013883468506926"/>
-    <inertia ixx="2.674027" iyy="2.737864" izz="0.665771" ixy="-0.003283" iyz="-0.013126" ixz="-0.310987"/>
+    <origin xyz="-0.14414593948878596 0.007272292388517288 0.4790557350675238" rpy="0 0 0"/>
+    <mass value="7.356876734373038"/>
+    <inertia ixx="0.055113" iyy="0.026097" izz="0.045184" ixy="-0.000286" iyz="-0.000998" ixz="0.003045"/>
   </inertial>
   <visual>
@@ -28,7 +30,7 @@
 <link name="base_link_frames_1">
   <inertial>
-    <origin xyz="0.05219682070735798 0.09908927488444497 0.4776891193965433" rpy="0 0 0"/>
-    <mass value="2.6725201136516104"/>
-    <inertia ixx="0.264075" iyy="0.253077" izz="0.065833" ixy="1e-06" iyz="-8e-06" ixz="-0.022361"/>
+    <origin xyz="0.09299736209064594 0.09816853953024438 0.7758797564332383" rpy="0 0 0"/>
+    <mass value="0.7337661134722138"/>
+    <inertia ixx="0.014481" iyy="0.016578" izz="0.009497" ixy="2.8e-05" iyz="-0.000106" ixz="-5.3e-05"/>
   </inertial>
   <visual>
@@ -135,79 +137,37 @@
 <link name="caster_right_1">
   <inertial>
-    <origin xyz="0.0037004833856989494 -0.027923972873388603 -0.08822047192631874" rpy="0 0 0"/>
-    <mass value="0.9867038593578229"/>
-    <inertia ixx="0.000947" iyy="0.001166" izz="0.000456" ixy="-2e-06" iyz="-5e-06" ixz="-0.000231"/>
-  </inertial>
-  <visual>
+    <origin xyz="0.00355868425330208 -0.0279262663780577 -0.08858638249680677" rpy="0 0 0"/>
+    <mass value="1.0173955553418546"/>
+    <inertia ixx="0.000972" iyy="0.001208" izz="0.000477" ixy="-2e-06" iyz="-5e-06" ixz="-0.000233"/>
+  </inertial>
+  <visual>
+    <origin xyz="0.324 -0.187 0.00465" rpy="0 0 0"/>
+    <geometry>
+      <mesh filename="package://roomac_description/meshes/caster.dae" scale="0.001 0.001 0.001"/>
+    </geometry>
+  </visual>
+  <collision>
     <origin xyz="0.324 0.133 0.00465" rpy="0 0 0"/>
     <geometry>
       <mesh filename="package://roomac_description/meshes/caster_right_1.stl" scale="0.001 0.001 0.001"/>
     </geometry>
-    <material name="silver"/>
-  </visual>
-  <collision>
-    <origin xyz="0.324 0.133 0.00465" rpy="0 0 0"/>
-    <geometry>
-      <mesh filename="package://roomac_description/meshes/caster_right_1.stl" scale="0.001 0.001 0.001"/>
-    </geometry>
   </collision>
 </link>
 <link name="caster_left_1">
   <inertial>
-    <origin xyz="0.0037004833856989494 0.021923972873387293 -0.0882204719263213" rpy="0 0 0"/>
-    <mass value="0.9867038593578229"/>
-    <inertia ixx="0.000947" iyy="0.001166" izz="0.000456" ixy="2e-06" iyz="5e-06" ixz="-0.000231"/>
+    <origin xyz="0.0035586842533020246 0.02192626637805642 -0.0885863824968092" rpy="0 0 0"/>
+    <mass value="1.0173955553418546"/>
+    <inertia ixx="0.000972" iyy="0.001208" izz="0.000477" ixy="2e-06" iyz="5e-06" ixz="-0.000233"/>
   </inertial>
   <visual>
     <origin xyz="0.324 -0.139 0.00465" rpy="0 0 0"/>
     <geometry>
+      <mesh filename="package://roomac_description/meshes/caster.dae" scale="0.001 0.001 0.001"/>
+    </geometry>
+  </visual>
+  <collision>
+    <origin xyz="0.324 -0.139 0.00465" rpy="0 0 0"/>
+    <geometry>
       <mesh filename="package://roomac_description/meshes/caster_left_1.stl" scale="0.001 0.001 0.001"/>
-    </geometry>
-    <material name="silver"/>
-  </visual>
-  <collision>
-    <origin xyz="0.324 -0.139 0.00465" rpy="0 0 0"/>
-    <geometry>
-      <mesh filename="package://roomac_description/meshes/caster_left_1.stl" scale="0.001 0.001 0.001"/>
-    </geometry>
-  </collision>
-</link>
-<link name="caster_tire_right_1">
-  <inertial>
-    <origin xyz="-2.3869795029440866e-15 -2.498001805406602e-16 5.398459457239824e-15" rpy="0 0 0"/>
-    <mass value="0.030691695984031726"/>
-    <inertia ixx="2.1e-05" iyy="3.7e-05" izz="2.1e-05" ixy="-0.0" iyz="-0.0" ixz="-0.0"/>
-  </inertial>
-  <visual>
-    <origin xyz="0.325 0.161 0.105" rpy="0 0 0"/>
-    <geometry>
-      <mesh filename="package://roomac_description/meshes/caster_tire_right_1.stl" scale="0.001 0.001 0.001"/>
-    </geometry>
-    <material name="black"/>
-  </visual>
-  <collision>
-    <origin xyz="0.325 0.161 0.105" rpy="0 0 0"/>
-    <geometry>
-      <mesh filename="package://roomac_description/meshes/caster_tire_right_1.stl" scale="0.001 0.001 0.001"/>
-    </geometry>
-  </collision>
-</link>
-<link name="caster_tire_left_1">
-  <inertial>
-    <origin xyz="-2.55351295663786e-15 -7.494005416219807e-16 3.969047313034935e-15" rpy="0 0 0"/>
-    <mass value="0.03069169598403176"/>
-    <inertia ixx="2.1e-05" iyy="3.7e-05" izz="2.1e-05" ixy="-0.0" iyz="-0.0" ixz="-0.0"/>
-  </inertial>
-  <visual>
-    <origin xyz="0.325 -0.161 0.105" rpy="0 0 0"/>
-    <geometry>
-      <mesh filename="package://roomac_description/meshes/caster_tire_left_1.stl" scale="0.001 0.001 0.001"/>
-    </geometry>
-    <material name="black"/>
-  </visual>
-  <collision>
-    <origin xyz="0.325 -0.161 0.105" rpy="0 0 0"/>
-    <geometry>
-      <mesh filename="package://roomac_description/meshes/caster_tire_left_1.stl" scale="0.001 0.001 0.001"/>
     </geometry>
   </collision>
@@ -223,150 +183,48 @@
   <child link="caster_left_1"/>
 </joint>
-<joint name="caster_tire_right" type="fixed">
-  <origin xyz="-0.001 -0.028 -0.10035" rpy="0 0 0"/>
-  <parent link="caster_right_1"/>
-  <child link="caster_tire_right_1"/>
-</joint>
-<joint name="caster_tire_left" type="fixed">
-  <origin xyz="-0.001 0.022 -0.10035" rpy="0 0 0"/>
-  <parent link="caster_left_1"/>
-  <child link="caster_tire_left_1"/>
-</joint>
 <!-- WHEELS -->
-<link name="hub_right_1">
-  <inertial>
-    <origin xyz="-1.789765220804318e-06 0.012712108125801869 3.1361035183559637e-06" rpy="0 0 0"/>
-    <mass value="0.09451094240372103"/>
-    <inertia ixx="5e-05" iyy="8.5e-05" izz="5e-05" ixy="0.0" iyz="-0.0" ixz="0.0"/>
-  </inertial>
-  <visual>
-    <origin xyz="0.0 0.246 0.0" rpy="0 0 0"/>
-    <geometry>
-      <mesh filename="package://roomac_description/meshes/hub_right_1.stl" scale="0.001 0.001 0.001"/>
-    </geometry>
-    <material name="black"/>
-  </visual>
-  <collision>
-    <origin xyz="0.0 0.246 0.0" rpy="0 0 0"/>
-    <geometry>
-      <mesh filename="package://roomac_description/meshes/hub_right_1.stl" scale="0.001 0.001 0.001"/>
-    </geometry>
-  </collision>
-</link>
-<link name="hub_left_1">
-  <inertial>
-    <origin xyz="-1.7897652210308038e-06 -0.012712108125801591 3.1361035183086937e-06" rpy="0 0 0"/>
-    <mass value="0.09451094240372113"/>
-    <inertia ixx="5e-05" iyy="8.5e-05" izz="5e-05" ixy="-0.0" iyz="0.0" ixz="0.0"/>
-  </inertial>
-  <visual>
-    <origin xyz="0.0 -0.246 0.0" rpy="0 0 0"/>
-    <geometry>
-      <mesh filename="package://roomac_description/meshes/hub_left_1.stl" scale="0.001 0.001 0.001"/>
-    </geometry>
-    <material name="black"/>
-  </visual>
-  <collision>
-    <origin xyz="0.0 -0.246 0.0" rpy="0 0 0"/>
-    <geometry>
-      <mesh filename="package://roomac_description/meshes/hub_left_1.stl" scale="0.001 0.001 0.001"/>
-    </geometry>
-  </collision>
-</link>
 <link name="wheel_right_1">
   <inertial>
-    <origin xyz="-4.446890699227879e-08 -0.046359989716390604 2.8955374773431687e-08" rpy="0 0 0"/>
-    <mass value="1.4792126361607076"/>
-    <inertia ixx="0.006728" iyy="0.012762" izz="0.006728" ixy="0.0" iyz="-0.0" ixz="0.0"/>
-  </inertial>
-  <visual>
+    <origin xyz="-8.535155939829862e-08 -0.045545810193822645 1.2324269625501287e-07" rpy="0 0 0"/>
+    <mass value="2.752514069802561"/>
+    <inertia ixx="0.01649" iyy="0.031597" izz="0.01649" ixy="0.0" iyz="-0.0" ixz="0.0"/>
+  </inertial>
+  <visual>
+    <origin xyz="-0.0 0.21064 0.0" rpy="${pi} 0 0"/>
+    <geometry>
+      <mesh filename="package://roomac_description/meshes/wheel.dae" scale="0.001 0.001 0.001"/>
+    </geometry>
+  </visual>
+  <collision>
     <origin xyz="-0.0 0.21064 0.0" rpy="0 0 0"/>
     <geometry>
       <mesh filename="package://roomac_description/meshes/wheel_right_1.stl" scale="0.001 0.001 0.001"/>
     </geometry>
-    <material name="silver"/>
-  </visual>
-  <collision>
-    <origin xyz="-0.0 0.21064 0.0" rpy="0 0 0"/>
-    <geometry>
-      <mesh filename="package://roomac_description/meshes/wheel_right_1.stl" scale="0.001 0.001 0.001"/>
-    </geometry>
   </collision>
 </link>
 <link name="wheel_left_1">
   <inertial>
-    <origin xyz="-3.1796540813644466e-08 0.04035998903806015 1.6110734861740638e-08" rpy="0 0 0"/>
-    <mass value="1.4792124768984427"/>
-    <inertia ixx="0.006728" iyy="0.012762" izz="0.006728" ixy="0.0" iyz="0.0" ixz="0.0"/>
+    <origin xyz="-7.854137935392783e-08 0.039545809782175645 1.1633993854093376e-07" rpy="0 0 0"/>
+    <mass value="2.7525139105402956"/>
+    <inertia ixx="0.01649" iyy="0.031597" izz="0.01649" ixy="-0.0" iyz="0.0" ixz="0.0"/>
   </inertial>
   <visual>
     <origin xyz="0.0 -0.21664 0.0" rpy="0 0 0"/>
     <geometry>
+      <mesh filename="package://roomac_description/meshes/wheel.dae" scale="0.001 0.001 0.001"/>
+    </geometry>
+  </visual>
+  <collision>
+    <origin xyz="0.0 -0.21664 0.0" rpy="0 0 0"/>
+    <geometry>
       <mesh filename="package://roomac_description/meshes/wheel_left_1.stl" scale="0.001 0.001 0.001"/>
     </geometry>
-    <material name="silver"/>
-  </visual>
-  <collision>
-    <origin xyz="0.0 -0.21664 0.0" rpy="0 0 0"/>
-    <geometry>
-      <mesh filename="package://roomac_description/meshes/wheel_left_1.stl" scale="0.001 0.001 0.001"/>
-    </geometry>
-  </collision>
-</link>
-<link name="wheel_tire_right_1">
-  <inertial>
-    <origin xyz="-1.0835776720341528e-15 -2.220446049250313e-16 1.4210854715202004e-16" rpy="0 0 0"/>
-    <mass value="1.1787904912381322"/>
-    <inertia ixx="0.009661" iyy="0.018749" izz="0.009661" ixy="-0.0" iyz="-0.0" ixz="-0.0"/>
-  </inertial>
-  <visual>
-    <origin xyz="0.0 0.257 -0.0" rpy="0 0 0"/>
-    <geometry>
-      <mesh filename="package://roomac_description/meshes/wheel_tire_right_1.stl" scale="0.001 0.001 0.001"/>
-    </geometry>
-    <material name="black"/>
-  </visual>
-  <collision>
-    <origin xyz="0.0 0.257 -0.0" rpy="0 0 0"/>
-    <geometry>
-      <mesh filename="package://roomac_description/meshes/wheel_tire_right_1.stl" scale="0.001 0.001 0.001"/>
-    </geometry>
-  </collision>
-</link>
-<link name="wheel_tire_left_1">
-  <inertial>
-    <origin xyz="-1.3677947663381929e-15 -6.106226635438361e-16 1.4210854715202004e-16" rpy="0 0 0"/>
-    <mass value="1.178790491238132"/>
-    <inertia ixx="0.009661" iyy="0.018749" izz="0.009661" ixy="-0.0" iyz="-0.0" ixz="-0.0"/>
-  </inertial>
-  <visual>
-    <origin xyz="0.0 -0.257 0.0" rpy="0 0 0"/>
-    <geometry>
-      <mesh filename="package://roomac_description/meshes/wheel_tire_left_1.stl" scale="0.001 0.001 0.001"/>
-    </geometry>
-    <material name="black"/>
-  </visual>
-  <collision>
-    <origin xyz="0.0 -0.257 0.0" rpy="0 0 0"/>
-    <geometry>
-      <mesh filename="package://roomac_description/meshes/wheel_tire_left_1.stl" scale="0.001 0.001 0.001"/>
-    </geometry>
-  </collision>
-</link>
-<joint name="hub_right" type="fixed">
-  <origin xyz="-0.0 -0.03536 0.0" rpy="0 0 0"/>
-  <parent link="wheel_right_1"/>
-  <child link="hub_right_1"/>
-</joint>
-<joint name="hub_left" type="fixed">
-  <origin xyz="0.0 0.02936 0.0" rpy="0 0 0"/>
-  <parent link="wheel_left_1"/>
-  <child link="hub_left_1"/>
-</joint>
+  </collision>
+</link>
 <joint name="wheel_right" type="continuous">
   <origin xyz="0.0 -0.21064 0.0" rpy="0 0 0"/>
   <parent link="base_link"/>
   <child link="wheel_right_1"/>
-  <axis xyz="0.0 1.0 -0.0"/>
+  <axis xyz="0.0 1.0 0.0"/>
 </joint>
 <joint name="wheel_left" type="continuous">
@@ -374,15 +232,5 @@
   <parent link="base_link"/>
   <child link="wheel_left_1"/>
-  <axis xyz="-0.0 1.0 -0.0"/>
-</joint>
-<joint name="wheel_tire_right" type="fixed">
-  <origin xyz="-0.0 -0.04636 0.0" rpy="0 0 0"/>
-  <parent link="wheel_right_1"/>
-  <child link="wheel_tire_right_1"/>
-</joint>
-<joint name="wheel_tire_left" type="fixed">
-  <origin xyz="0.0 0.04036 0.0" rpy="0 0 0"/>
-  <parent link="wheel_left_1"/>
-  <child link="wheel_tire_left_1"/>
+  <axis xyz="0.0 1.0 0.0"/>
 </joint>
 <!-- HEAD -->
@@ -463,24 +311,4 @@
 </joint>
 <!-- RIGHT ARM -->
-<link name="shoulder_base_right_1">
-  <inertial>
-    <origin xyz="-0.07808936770346069 -0.00579384989233192 -0.015842800732696283" rpy="0 0 0"/>
-    <mass value="1.58045814183351"/>
-    <inertia ixx="0.000698" iyy="0.003262" izz="0.003259" ixy="-0.000283" iyz="-4.1e-05" ixz="-0.000224"/>
-  </inertial>
-  <visual>
-    <origin xyz="0.0725 0.134829 -0.961645" rpy="0 0 0"/>
-    <geometry>
-      <mesh filename="package://roomac_description/meshes/shoulder_base_right_1.stl" scale="0.001 0.001 0.001"/>
-    </geometry>
-    <material name="black"/>
-  </visual>
-  <collision>
-    <origin xyz="0.0725 0.134829 -0.961645" rpy="0 0 0"/>
-    <geometry>
-      <mesh filename="package://roomac_description/meshes/shoulder_base_right_1.stl" scale="0.001 0.001 0.001"/>
-    </geometry>
-  </collision>
-</link>
 <link name="shoulder_right_1">
   <inertial>
@@ -503,72 +331,31 @@
   </collision>
 </link>
-<link name="shoulder_elbow_gear_right_1">
-  <inertial>
-    <origin xyz="4.458388786428291e-05 -3.227258993376836e-08 0.001208993450583895" rpy="0 0 0"/>
-    <mass value="0.48507719135410154"/>
-    <inertia ixx="0.000258" iyy="0.000141" izz="0.000153" ixy="-0.0" iyz="0.0" ixz="0.0"/>
+<link name="shoulder_elbow_right_1">
+  <inertial>
+    <origin xyz="-1.8144588477334023e-05 1.4016989058340812e-07 -0.08491558495824947" rpy="0 0 0"/>
+    <mass value="1.0007451414955084"/>
+    <inertia ixx="0.008299" iyy="0.0082" izz="0.000235" ixy="-0.0" iyz="0.0" ixz="3e-06"/>
   </inertial>
   <visual>
     <origin xyz="0.113 0.243979 -0.9345" rpy="0 0 0"/>
     <geometry>
-      <mesh filename="package://roomac_description/meshes/shoulder_elbow_gear_right_1.stl" scale="0.001 0.001 0.001"/>
-    </geometry>
-    <material name="black"/>
+      <mesh filename="package://roomac_description/meshes/shoulder_elbow_right_1.dae" scale="0.001 0.001 0.001"/>
+    </geometry>
   </visual>
   <collision>
     <origin xyz="0.113 0.243979 -0.9345" rpy="0 0 0"/>
     <geometry>
-      <mesh filename="package://roomac_description/meshes/shoulder_elbow_gear_right_1.stl" scale="0.001 0.001 0.001"/>
-    </geometry>
-  </collision>
-</link>
-<link name="shoulder_elbow_right_1">
-  <inertial>
-    <origin xyz="4.232586503505331e-12 3.0408664961067977e-07 -0.07500000000256124" rpy="0 0 0"/>
-    <mass value="0.09112500000022286"/>
-    <inertia ixx="0.000173" iyy="0.000173" izz="3e-06" ixy="0.0" iyz="-0.0" ixz="-0.0"/>
-  </inertial>
-  <visual>
-    <origin xyz="0.1135 0.243979 -0.924925" rpy="0 0 0"/>
-    <geometry>
       <mesh filename="package://roomac_description/meshes/shoulder_elbow_right_1.stl" scale="0.001 0.001 0.001"/>
     </geometry>
-    <material name="silver"/>
-  </visual>
-  <collision>
-    <origin xyz="0.1135 0.243979 -0.924925" rpy="0 0 0"/>
-    <geometry>
-      <mesh filename="package://roomac_description/meshes/shoulder_elbow_right_1.stl" scale="0.001 0.001 0.001"/>
-    </geometry>
-  </collision>
-</link>
-<link name="elbow_right_1">
-  <inertial>
-    <origin xyz="0.0005136115276251074 3.101290486640096e-07 -0.023818498356463658" rpy="0 0 0"/>
-    <mass value="0.4245429501284504"/>
-    <inertia ixx="0.000153" iyy="0.00017" izz="7.8e-05" ixy="0.0" iyz="-0.0" ixz="4e-06"/>
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
Commit message: Cleanup axis components in urdf

File: roomac_description/urdf/roomac_body.xacro (robot description, xacro)
@@ -1,6 +1,4 @@
 <?xml version="1.0" ?>
 <robot name="roomac" xmlns:xacro="http://www.ros.org/wiki/xacro">
-<!-- todo cleanup axis in urdf -->
-<!-- todo remove material from dae -->
 <!-- BODY -->
 <link name="base_link" />
@@ -115,5 +113,4 @@
       <mesh filename="package://roomac_description/materials/artag_bundle.dae" scale="3.142857143 1.2 0.001"/>
     </geometry>
-    <material name="artag"/>
   </visual>
   <collision>
@@ -130,5 +127,5 @@
 </joint>
 <joint name="artag_joint_bundle_visual" type="fixed">
-  <origin rpy="0 0 0" xyz="0.01 0.0 0"/>
+  <origin rpy="0 0 0" xyz="0.01 0.0 0.0"/>
   <parent link="artag_link"/>
   <child link="artag_link_bundle_visual"/>
@@ -226,5 +223,5 @@
   <parent link="base_link"/>
   <child link="wheel_right_1"/>
-  <axis xyz="0.0 1.0 0.0"/>
+  <axis xyz="0 1 0"/>
 </joint>
 <joint name="wheel_left" type="continuous">
@@ -232,5 +229,5 @@
   <parent link="base_link"/>
   <child link="wheel_left_1"/>
-  <axis xyz="0.0 1.0 0.0"/>
+  <axis xyz="0 1 0"/>
 </joint>
 <!-- HEAD -->
@@ -457,5 +454,5 @@
   <parent link="base_link"/>
   <child link="shoulder_right_1"/>
-  <axis xyz="0.0 1.0 0.0"/>
+  <axis xyz="0 1 0"/>
   <limit effort="30" velocity="1.0" lower="-2.390" upper="0.489" />
 </joint>
@@ -464,5 +461,5 @@
   <parent link="shoulder_right_1"/>
   <child link="shoulder_elbow_right_1"/>
-  <axis xyz="-1.0 -0.0 0.0"/>
+  <axis xyz="-1 0 0"/>
   <!-- Calculated lower: -0.899, adjusted it due to colision with gear-->
   <limit effort="30" velocity="1.0" lower="-0.800" upper="1.979" />
@@ -472,5 +469,5 @@
   <parent link="shoulder_elbow_right_1"/>
   <child link="elbow_wrist_right_1"/>
-  <axis xyz="1.0 0.0 -0.0"/>
+  <axis xyz="1 0 0"/>
   <!-- Calculated lower: -2.879 upper: 2.879, adjusted due to collisions-->
   <!-- Safe values, might be some room for increase -->
@@ -481,5 +478,5 @@
   <parent link="elbow_wrist_right_1"/>
   <child link="wrist_right_1"/>
-  <axis xyz="-1.0 -0.0 0.0"/>
+  <axis xyz="-1 0 0"/>
   <limit effort="30" velocity="1.0" lower="-1.994" upper="1.146" />
 </joint>
@@ -488,5 +485,5 @@
   <parent link="wrist_right_1"/>
   <child link="gripper_right_1"/>
-  <axis xyz="0.0 0.0 -1.0"/>
+  <axis xyz="0 0 -1"/>
   <limit effort="30" velocity="1.0" lower="-1.570" upper="1.570" />
 </joint>
@@ -654,5 +651,5 @@
   <parent link="base_link"/>
   <child link="shoulder_left_1"/>
-  <axis xyz="0.0 1.0 -0.0"/>
+  <axis xyz="0 1 0"/>
 </joint>
 <joint name="shoulder_roll_left" type="continuous">
@@ -660,5 +657,5 @@
   <parent link="shoulder_left_1"/>
   <child link="shoulder_elbow_left_1"/>
-  <axis xyz="1.0 -0.0 -0.0"/>
+  <axis xyz="1 0 0"/>
 </joint>
 <joint name="elbow_left" type="continuous">
@@ -666,5 +663,5 @@
   <parent link="shoulder_elbow_left_1"/>
   <child link="elbow_wrist_left_1"/>
-  <axis xyz="1.0 -0.0 -0.0"/>
+  <axis xyz="1 0 0"/>
 </joint>
 <joint name="wrist_left" type="continuous">
@@ -672,5 +669,5 @@
   <parent link="elbow_wrist_left_1"/>
   <child link="wrist_left_1"/>
-  <axis xyz="1.0 -0.0 -0.0"/>
+  <axis xyz="1 0 0"/>
 </joint>
 <joint name="gripper_twist_left" type="continuous">
@@ -678,5 +675,5 @@
   <parent link="wrist_left_1"/>
   <child link="gripper_left_1"/>
-  <axis xyz="-0.0 -0.0 -1.0"/>
+  <axis xyz="0 0 -1"/>
 </joint>
 <joint name="gripper_finger_r_left" type="fixed">

Commit message: Rename robot_base to robot_body link

File: roomac_description/urdf/roomac_body.xacro (robot description, xacro)
@@ -6,5 +6,5 @@
 <!-- Additional link needed to solve moveit warning (as far as I know it shouldn't cause any issue as I'm not using KDL, but still better to solve it): -->
 <!-- The root link base_link has an inertia specified in the URDF, but KDL does not support a root link with an inertia.  As a workaround, you can add an extra dummy link to your URDF. -->
-<link name="robot_base_1">
+<link name="robot_body_1">
   <inertial>
     <origin xyz="-0.14414593948878596 0.007272292388517288 0.4790557350675238" rpy="0 0 0"/>
@@ -71,7 +71,7 @@
   <child link="base_link"/>
 </joint>
-<joint name="robot_base" type="fixed">
-  <parent link="base_link"/>
-  <child link="robot_base_1"/>
+<joint name="robot_body" type="fixed">
+  <parent link="base_link"/>
+  <child link="robot_body_1"/>
 </joint>
 <joint name="base_link_frames" type="fixed">
