Commit message: Fix mesh file names

File: roomac_description/urdf/roomac_body.xacro (robot description, xacro)
@@ -16,5 +16,5 @@
     <origin xyz="0 0 0" rpy="0 0 0"/>
     <geometry>
-      <mesh filename="package://roomac_description/meshes/base_link.stl" scale="0.001 0.001 0.001"/>
+      <mesh filename="package://roomac_description/meshes/robot_body.stl" scale="0.001 0.001 0.001"/>
     </geometry>
     <material name="black"/>
@@ -23,5 +23,5 @@
     <origin xyz="0 0 0" rpy="0 0 0"/>
     <geometry>
-      <mesh filename="package://roomac_description/meshes/base_link.stl" scale="0.001 0.001 0.001"/>
+      <mesh filename="package://roomac_description/meshes/robot_body.stl" scale="0.001 0.001 0.001"/>
     </geometry>
   </collision>
@@ -36,5 +36,5 @@
     <origin xyz="0.223282 0.099058 0.0075" rpy="0 0 0"/>
     <geometry>
-      <mesh filename="package://roomac_description/meshes/robot_body_frames_link.stl" scale="0.001 0.001 0.001"/>
+      <mesh filename="package://roomac_description/meshes/robot_body_frames.stl" scale="0.001 0.001 0.001"/>
     </geometry>
     <material name="white"/>
@@ -43,5 +43,5 @@
     <origin xyz="0.223282 0.099058 0.0075" rpy="0 0 0"/>
     <geometry>
-      <mesh filename="package://roomac_description/meshes/robot_body_frames_link.stl" scale="0.001 0.001 0.001"/>
+      <mesh filename="package://roomac_description/meshes/robot_body_frames.stl" scale="0.001 0.001 0.001"/>
     </geometry>
   </collision>
@@ -56,5 +56,5 @@
     <origin xyz="0.06485 -0.10315 -0.52765" rpy="0 0 0"/>
     <geometry>
-      <mesh filename="package://roomac_description/meshes/frame_link.stl" scale="0.001 0.001 0.001"/>
+      <mesh filename="package://roomac_description/meshes/frame.dae" scale="0.001 0.001 0.001"/>
     </geometry>
     <material name="silver"/>
@@ -63,5 +63,5 @@
     <origin xyz="0.06485 -0.10315 -0.52765" rpy="0 0 0"/>
     <geometry>
-      <mesh filename="package://roomac_description/meshes/frame_link.stl" scale="0.001 0.001 0.001"/>
+      <mesh filename="package://roomac_description/meshes/frame.stl" scale="0.001 0.001 0.001"/>
     </geometry>
   </collision>
@@ -103,4 +103,5 @@
 <!-- ARTAG -->
 <link name="artag_link" />
+<!-- todo: move artag bundle file to meshes -->
 <link name="artag_bundle_visual_link">
   <inertial>
@@ -148,5 +149,5 @@
     <origin xyz="0.324 0.133 0.00465" rpy="0 0 0"/>
     <geometry>
-      <mesh filename="package://roomac_description/meshes/caster_right_link.stl" scale="0.001 0.001 0.001"/>
+      <mesh filename="package://roomac_description/meshes/caster_right.stl" scale="0.001 0.001 0.001"/>
     </geometry>
   </collision>
@@ -167,5 +168,5 @@
     <origin xyz="0.324 -0.139 0.00465" rpy="0 0 0"/>
     <geometry>
-      <mesh filename="package://roomac_description/meshes/caster_left_link.stl" scale="0.001 0.001 0.001"/>
+      <mesh filename="package://roomac_description/meshes/caster_left.stl" scale="0.001 0.001 0.001"/>
     </geometry>
   </collision>
@@ -197,5 +198,5 @@
     <origin xyz="-0.0 0.21064 0.0" rpy="0 0 0"/>
     <geometry>
-      <mesh filename="package://roomac_description/meshes/wheel_right_link.stl" scale="0.001 0.001 0.001"/>
+      <mesh filename="package://roomac_description/meshes/wheel_right.stl" scale="0.001 0.001 0.001"/>
     </geometry>
   </collision>
@@ -216,5 +217,5 @@
     <origin xyz="0.0 -0.21664 0.0" rpy="0 0 0"/>
     <geometry>
-      <mesh filename="package://roomac_description/meshes/wheel_left_link.stl" scale="0.001 0.001 0.001"/>
+      <mesh filename="package://roomac_description/meshes/wheel_left.stl" scale="0.001 0.001 0.001"/>
     </geometry>
   </collision>
@@ -242,5 +243,5 @@
     <origin xyz="0.08 -2.1e-05 -0.969145" rpy="0 0 0"/>
     <geometry>
-      <mesh filename="package://roomac_description/meshes/head_link.stl" scale="0.001 0.001 0.001"/>
+      <mesh filename="package://roomac_description/meshes/head.stl" scale="0.001 0.001 0.001"/>
     </geometry>
     <material name="black"/>
@@ -249,5 +250,5 @@
     <origin xyz="0.08 -2.1e-05 -0.969145" rpy="0 0 0"/>
     <geometry>
-      <mesh filename="package://roomac_description/meshes/head_link.stl" scale="0.001 0.001 0.001"/>
+      <mesh filename="package://roomac_description/meshes/head.stl" scale="0.001 0.001 0.001"/>
     </geometry>
   </collision>
@@ -262,5 +263,5 @@
     <origin xyz="0.0825 0.055979 -1.083347" rpy="0 0 0"/>
     <geometry>
-      <mesh filename="package://roomac_description/meshes/eye_right_link.stl" scale="0.001 0.001 0.001"/>
+      <mesh filename="package://roomac_description/meshes/eye_right.stl" scale="0.001 0.001 0.001"/>
     </geometry>
     <material name="white"/>
@@ -269,5 +270,5 @@
     <origin xyz="0.0825 0.055979 -1.083347" rpy="0 0 0"/>
     <geometry>
-      <mesh filename="package://roomac_description/meshes/eye_right_link.stl" scale="0.001 0.001 0.001"/>
+      <mesh filename="package://roomac_description/meshes/eye_right.stl" scale="0.001 0.001 0.001"/>
     </geometry>
   </collision>
@@ -282,5 +283,5 @@
     <origin xyz="0.0825 -0.056021 -1.083347" rpy="0 0 0"/>
     <geometry>
-      <mesh filename="package://roomac_description/meshes/eye_left_link.stl" scale="0.001 0.001 0.001"/>
+      <mesh filename="package://roomac_description/meshes/eye_left.stl" scale="0.001 0.001 0.001"/>
     </geometry>
     <material name="white"/>
@@ -289,5 +290,5 @@
     <origin xyz="0.0825 -0.056021 -1.083347" rpy="0 0 0"/>
     <geometry>
-      <mesh filename="package://roomac_description/meshes/eye_left_link.stl" scale="0.001 0.001 0.001"/>
+      <mesh filename="package://roomac_description/meshes/eye_left.stl" scale="0.001 0.001 0.001"/>
     </geometry>
   </collision>
@@ -318,5 +319,5 @@
     <origin xyz="0.1135 0.174979 -0.9345" rpy="0 0 0"/>
     <geometry>
-      <mesh filename="package://roomac_description/meshes/shoulder_right_link.stl" scale="0.001 0.001 0.001"/>
+      <mesh filename="package://roomac_description/meshes/shoulder_right.stl" scale="0.001 0.001 0.001"/>
     </geometry>
     <material name="black"/>
@@ -325,5 +326,5 @@
     <origin xyz="0.1135 0.174979 -0.9345" rpy="0 0 0"/>
     <geometry>
-      <mesh filename="package://roomac_description/meshes/shoulder_right_link.stl" scale="0.001 0.001 0.001"/>
+      <mesh filename="package://roomac_description/meshes/shoulder_right.stl" scale="0.001 0.001 0.001"/>
     </geometry>
   </collision>
@@ -338,5 +339,5 @@
     <origin xyz="0.113 0.243979 -0.9345" rpy="0 0 0"/>
     <geometry>
-      <mesh filename="package://roomac_description/meshes/shoulder_elbow_right_link.dae" scale="0.001 0.001 0.001"/>
+      <mesh filename="package://roomac_description/meshes/shoulder_elbow_right.dae" scale="0.001 0.001 0.001"/>
     </geometry>
   </visual>
@@ -344,5 +345,5 @@
     <origin xyz="0.113 0.243979 -0.9345" rpy="0 0 0"/>
     <geometry>
-      <mesh filename="package://roomac_description/meshes/shoulder_elbow_right_link.stl" scale="0.001 0.001 0.001"/>
+      <mesh filename="package://roomac_description/meshes/shoulder_elbow_right.stl" scale="0.001 0.001 0.001"/>
     </geometry>
   </collision>
@@ -357,5 +358,5 @@
     <origin xyz="0.0925 0.243979 -0.733425" rpy="0 0 0"/>
     <geometry>
-      <mesh filename="package://roomac_description/meshes/elbow_wrist_right_link.stl" scale="0.001 0.001 0.001"/>
+      <mesh filename="package://roomac_description/meshes/elbow_wrist_right.stl" scale="0.001 0.001 0.001"/>
     </geometry>
     <material name="black"/>
@@ -364,5 +365,5 @@
     <origin xyz="0.0925 0.243979 -0.733425" rpy="0 0 0"/>
     <geometry>
-      <mesh filename="package://roomac_description/meshes/elbow_wrist_right_link.stl" scale="0.001 0.001 0.001"/>
+      <mesh filename="package://roomac_description/meshes/elbow_wrist_right.stl" scale="0.001 0.001 0.001"/>
     </geometry>
   </collision>
@@ -377,5 +378,5 @@
     <origin xyz="0.139354 0.243979 -0.603583" rpy="0 0 0"/>
     <geometry>
-      <mesh filename="package://roomac_description/meshes/wrist_right_link.stl" scale="0.001 0.001 0.001"/>
+      <mesh filename="package://roomac_description/meshes/wrist_right.stl" scale="0.001 0.001 0.001"/>
     </geometry>
     <material name="black"/>
@@ -384,5 +385,5 @@
     <origin xyz="0.139354 0.243979 -0.603583" rpy="0 0 0"/>
     <geometry>
-      <mesh filename="package://roomac_description/meshes/wrist_right_link.stl" scale="0.001 0.001 0.001"/>
+      <mesh filename="package://roomac_description/meshes/wrist_right.stl" scale="0.001 0.001 0.001"/>
     </geometry>
   </collision>
@@ -397,5 +398,5 @@
     <origin xyz="0.114635 0.244052 -0.544791" rpy="0 0 0"/>
     <geometry>
-      <mesh filename="package://roomac_description/meshes/gripper_right_link.stl" scale="0.001 0.001 0.001"/>
+      <mesh filename="package://roomac_description/meshes/gripper_right.stl" scale="0.001 0.001 0.001"/>
     </geometry>
     <material name="black"/>
@@ -404,5 +405,5 @@
     <origin xyz="0.114635 0.244052 -0.544791" rpy="0 0 0"/>
     <geometry>
-      <mesh filename="package://roomac_description/meshes/gripper_right_link.stl" scale="0.001 0.001 0.001"/>
+      <mesh filename="package://roomac_description/meshes/gripper_right.stl" scale="0.001 0.001 0.001"/>
     </geometry>
   </collision>
@@ -420,5 +421,5 @@
     <origin xyz="0.117385 0.274314 -0.487684" rpy="0 0 0"/>
     <geometry>
-      <mesh filename="package://roomac_description/meshes/gripper_finger_r_right_link.stl" scale="0.001 0.001 0.001"/>
+      <mesh filename="package://roomac_description/meshes/gripper_finger_r_right.stl" scale="0.001 0.001 0.001"/>
     </geometry>
     <material name="black"/>
@@ -427,5 +428,5 @@
     <origin xyz="0.117385 0.274314 -0.487684" rpy="0 0 0"/>
     <geometry>
-      <mesh filename="package://roomac_description/meshes/gripper_finger_r_right_link.stl" scale="0.001 0.001 0.001"/>
+      <mesh filename="package://roomac_description/meshes/gripper_finger_r_right.stl" scale="0.001 0.001 0.001"/>
     </geometry>
   </collision>
@@ -440,5 +441,5 @@
     <origin xyz="0.117385 0.214585 -0.487684" rpy="0 0 0"/>
     <geometry>
-      <mesh filename="package://roomac_description/meshes/gripper_finger_l_right_link.stl" scale="0.001 0.001 0.001"/>
+      <mesh filename="package://roomac_description/meshes/gripper_finger_l_right.stl" scale="0.001 0.001 0.001"/>
     </geometry>
     <material name="black"/>
@@ -447,5 +448,5 @@
     <origin xyz="0.117385 0.214585 -0.487684" rpy="0 0 0"/>
     <geometry>
-      <mesh filename="package://roomac_description/meshes/gripper_finger_l_right_link.stl" scale="0.001 0.001 0.001"/>
+      <mesh filename="package://roomac_description/meshes/gripper_finger_l_right.stl" scale="0.001 0.001 0.001"/>
     </geometry>
   </collision>
@@ -520,5 +521,5 @@
     <origin xyz="0.1135 -0.175021 -0.9345" rpy="0 0 0"/>
     <geometry>
-      <mesh filename="package://roomac_description/meshes/shoulder_left_link.stl" scale="0.001 0.001 0.001"/>
+      <mesh filename="package://roomac_description/meshes/shoulder_left.stl" scale="0.001 0.001 0.001"/>
     </geometry>
     <material name="black"/>
@@ -527,5 +528,5 @@
     <origin xyz="0.1135 -0.175021 -0.9345" rpy="0 0 0"/>
     <geometry>
-      <mesh filename="package://roomac_description/meshes/shoulder_left_link.stl" scale="0.001 0.001 0.001"/>
+      <mesh filename="package://roomac_description/meshes/shoulder_left.stl" scale="0.001 0.001 0.001"/>
     </geometry>
   </collision>
@@ -540,5 +541,5 @@
     <origin xyz="0.113 -0.244021 -0.9345" rpy="0 0 0"/>
     <geometry>
-      <mesh filename="package://roomac_description/meshes/shoulder_elbow_left_link.dae" scale="0.001 0.001 0.001"/>
+      <mesh filename="package://roomac_description/meshes/shoulder_elbow_left.dae" scale="0.001 0.001 0.001"/>
     </geometry>
   </visual>
@@ -546,5 +547,5 @@
     <origin xyz="0.113 -0.244021 -0.9345" rpy="0 0 0"/>
     <geometry>
-      <mesh filename="package://roomac_description/meshes/shoulder_elbow_left_link.stl" scale="0.001 0.001 0.001"/>
+      <mesh filename="package://roomac_description/meshes/shoulder_elbow_left.stl" scale="0.001 0.001 0.001"/>
     </geometry>
   </collision>
@@ -559,5 +560,5 @@
     <origin xyz="0.0925 -0.244021 -0.733443" rpy="0 0 0"/>
     <geometry>
-      <mesh filename="package://roomac_description/meshes/elbow_wrist_left_link.stl" scale="0.001 0.001 0.001"/>
+      <mesh filename="package://roomac_description/meshes/elbow_wrist_left.stl" scale="0.001 0.001 0.001"/>
     </geometry>
     <material name="black"/>
@@ -566,5 +567,5 @@
     <origin xyz="0.0925 -0.244021 -0.733443" rpy="0 0 0"/>
     <geometry>
-      <mesh filename="package://roomac_description/meshes/elbow_wrist_left_link.stl" scale="0.001 0.001 0.001"/>
+      <mesh filename="package://roomac_description/meshes/elbow_wrist_left.stl" scale="0.001 0.001 0.001"/>
     </geometry>
   </collision>
@@ -579,5 +580,5 @@
     <origin xyz="0.139354 -0.244021 -0.603601" rpy="0 0 0"/>
     <geometry>
-      <mesh filename="package://roomac_description/meshes/wrist_left_link.stl" scale="0.001 0.001 0.001"/>
+      <mesh filename="package://roomac_description/meshes/wrist_left.stl" scale="0.001 0.001 0.001"/>
     </geometry>
     <material name="black"/>
@@ -586,5 +587,5 @@
     <origin xyz="0.139354 -0.244021 -0.603601" rpy="0 0 0"/>
     <geometry>
-      <mesh filename="package://roomac_description/meshes/wrist_left_link.stl" scale="0.001 0.001 0.001"/>
+      <mesh filename="package://roomac_description/meshes/wrist_left.stl" scale="0.001 0.001 0.001"/>
     </geometry>
   </collision>
@@ -599,5 +600,5 @@
     <origin xyz="0.114635 -0.244094 -0.544809" rpy="0 0 0"/>
     <geometry>
-      <mesh filename="package://roomac_description/meshes/gripper_left_link.stl" scale="0.001 0.001 0.001"/>
+      <mesh filename="package://roomac_description/meshes/gripper_left.stl" scale="0.001 0.001 0.001"/>
     </geometry>
     <material name="black"/>
@@ -606,5 +607,5 @@
     <origin xyz="0.114635 -0.244094 -0.544809" rpy="0 0 0"/>
     <geometry>
-      <mesh filename="package://roomac_description/meshes/gripper_left_link.stl" scale="0.001 0.001 0.001"/>
+      <mesh filename="package://roomac_description/meshes/gripper_left.stl" scale="0.001 0.001 0.001"/>
     </geometry>
   </collision>
@@ -619,5 +620,5 @@
     <origin xyz="0.117385 -0.274357 -0.487702" rpy="0 0 0"/>
     <geometry>
-      <mesh filename="package://roomac_description/meshes/gripper_finger_l_left_link.stl" scale="0.001 0.001 0.001"/>
+      <mesh filename="package://roomac_description/meshes/gripper_finger_l_left.stl" scale="0.001 0.001 0.001"/>
     </geometry>
     <material name="black"/>
@@ -626,5 +627,5 @@
     <origin xyz="0.117385 -0.274357 -0.487702" rpy="0 0 0"/>
     <geometry>
-      <mesh filename="package://roomac_description/meshes/gripper_finger_l_left_link.stl" scale="0.001 0.001 0.001"/>
+      <mesh filename="package://roomac_description/meshes/gripper_finger_l_left.stl" scale="0.001 0.001 0.001"/>
     </geometry>
   </collision>
@@ -639,5 +640,5 @@
     <origin xyz="0.117385 -0.214627 -0.487702" rpy="0 0 0"/>
     <geometry>
-      <mesh filename="package://roomac_description/meshes/gripper_finger_r_left_link.stl" scale="0.001 0.001 0.001"/>
+      <mesh filename="package://roomac_description/meshes/gripper_finger_r_left.stl" scale="0.001 0.001 0.001"/>
     </geometry>
     <material name="black"/>
@@ -646,5 +647,5 @@
     <origin xyz="0.117385 -0.214627 -0.487702" rpy="0 0 0"/>
     <geometry>
-      <mesh filename="package://roomac_description/meshes/gripper_finger_r_left_link.stl" scale="0.001 0.001 0.001"/>
+      <mesh filename="package://roomac_description/meshes/gripper_finger_r_left.stl" scale="0.001 0.001 0.001"/>
     </geometry>
   </collision>

Commit message: Remove unnecessary collision and inertial attributes

File: roomac_description/urdf/roomac_body.xacro (robot description, xacro)
@@ -2,4 +2,7 @@
 <robot name="roomac" xmlns:xacro="http://www.ros.org/wiki/xacro">
 <!-- todo: standardize joint names -->
+<!-- Some links are used only for visuals:
+  - robot_body_frames_link, frame_link and artag_bundle_visual_link - collision model in robot_body_link takes them into account, and also there is no point in inertial attribute for them (again robot_body_link should be enough)
+  - eye_right_link and eye_left_link - similar to previous example collision model in head is enough -->
 <!-- BODY -->
 <link name="base_link" />
@@ -28,9 +31,4 @@
 </link>
 <link name="robot_body_frames_link">
-  <inertial>
-    <origin xyz="0.09299736209064594 0.09816853953024438 0.7758797564332383" rpy="0 0 0"/>
-    <mass value="0.7337661134722138"/>
-    <inertia ixx="0.014481" iyy="0.016578" izz="0.009497" ixy="2.8e-05" iyz="-0.000106" ixz="-5.3e-05"/>
-  </inertial>
   <visual>
     <origin xyz="0.223282 0.099058 0.0075" rpy="0 0 0"/>
@@ -40,17 +38,6 @@
     <material name="white"/>
   </visual>
-  <collision>
-    <origin xyz="0.223282 0.099058 0.0075" rpy="0 0 0"/>
-    <geometry>
-      <mesh filename="package://roomac_description/meshes/robot_body_frames.stl" scale="0.001 0.001 0.001"/>
-    </geometry>
-  </collision>
 </link>
 <link name="frame_link">
-  <inertial>
-    <origin xyz="-0.06363233755923882 -0.10316506754069626 -0.18305645699853168" rpy="0 0 0"/>
-    <mass value="4.866480003493675"/>
-    <inertia ixx="0.611797" iyy="0.597598" izz="0.154569" ixy="-7e-06" iyz="5e-06" ixz="0.016258"/>
-  </inertial>
   <visual>
     <origin xyz="0.06485 -0.10315 -0.52765" rpy="0 0 0"/>
@@ -60,10 +47,4 @@
     <material name="silver"/>
   </visual>
-  <collision>
-    <origin xyz="0.06485 -0.10315 -0.52765" rpy="0 0 0"/>
-    <geometry>
-      <mesh filename="package://roomac_description/meshes/frame.stl" scale="0.001 0.001 0.001"/>
-    </geometry>
-  </collision>
 </link>
 <joint name="base_joint" type="fixed">
@@ -105,21 +86,10 @@
 <!-- todo: move artag bundle file to meshes -->
 <link name="artag_bundle_visual_link">
-  <inertial>
+  <visual>
     <origin rpy="0 0 0" xyz="0 0 0"/>
-    <mass value="0.1"/>
-    <inertia ixx="0" ixy="-0.0" ixz="0.0" iyy="0" iyz="0.0" izz="0"/>
-  </inertial>
-  <visual name="visual">
-    <origin rpy="0 0 0" xyz="0.0 0.0 0.0"/>
     <geometry>
       <mesh filename="package://roomac_description/materials/artag_bundle.dae" scale="3.142857143 1.2 0.001"/>
     </geometry>
   </visual>
-  <collision>
-    <origin rpy="0 0 0" xyz="0.0 0.0 0.0"/>
-    <geometry>
-      <mesh filename="package://roomac_description/materials/artag_bundle.dae" scale="3.142857143 1.2 0.001"/>
-    </geometry>
-  </collision>
 </link>
 <joint name="artag_joint" type="fixed">
@@ -255,9 +225,4 @@
 </link>
 <link name="eye_right_link">
-  <inertial>
-    <origin xyz="0.00626024105824001 3.517735655544918e-08 -3.559806300845736e-07" rpy="0 0 0"/>
-    <mass value="0.12003246414388505"/>
-    <inertia ixx="0.000115" iyy="5.8e-05" izz="5.8e-05" ixy="-0.0" iyz="0.0" ixz="-0.0"/>
-  </inertial>
   <visual>
     <origin xyz="0.0825 0.055979 -1.083347" rpy="0 0 0"/>
@@ -267,17 +232,6 @@
     <material name="white"/>
   </visual>
-  <collision>
-    <origin xyz="0.0825 0.055979 -1.083347" rpy="0 0 0"/>
-    <geometry>
-      <mesh filename="package://roomac_description/meshes/eye_right.stl" scale="0.001 0.001 0.001"/>
-    </geometry>
-  </collision>
 </link>
 <link name="eye_left_link">
-  <inertial>
-    <origin xyz="0.006260241058239718 3.517735615299333e-08 -3.5598063252706424e-07" rpy="0 0 0"/>
-    <mass value="0.12003246414388502"/>
-    <inertia ixx="0.000115" iyy="5.8e-05" izz="5.8e-05" ixy="-0.0" iyz="0.0" ixz="-0.0"/>
-  </inertial>
   <visual>
     <origin xyz="0.0825 -0.056021 -1.083347" rpy="0 0 0"/>
@@ -287,10 +241,4 @@
     <material name="white"/>
   </visual>
-  <collision>
-    <origin xyz="0.0825 -0.056021 -1.083347" rpy="0 0 0"/>
-    <geometry>
-      <mesh filename="package://roomac_description/meshes/eye_left.stl" scale="0.001 0.001 0.001"/>
-    </geometry>
-  </collision>
 </link>
 <joint name="head" type="fixed">
