Commit message: Change collisions in urdf to new meshes
(simplified versions of visuals)

File: roomac_description/urdf/roomac_body.xacro (robot description, xacro)
@@ -26,5 +26,5 @@
     <origin xyz="0 0 0" rpy="0 0 0"/>
     <geometry>
-      <mesh filename="package://roomac_description/meshes/robot_body.stl" scale="0.001 0.001 0.001"/>
+      <mesh filename="package://roomac_description/meshes/robot_body_collision.stl" scale="0.001 0.001 0.001"/>
     </geometry>
   </collision>
@@ -104,4 +104,6 @@
 </joint>
 <!-- CASTERS -->
+<xacro:property name="caster_wheel_width" value="0.034" />
+<xacro:property name="caster_wheel_radius" value="0.0375" />
 <link name="caster_right_link">
   <inertial>
@@ -115,9 +117,10 @@
       <mesh filename="package://roomac_description/meshes/caster.dae" scale="0.001 0.001 0.001"/>
     </geometry>
-  </visual>
-  <collision>
-    <origin xyz="0.324 0.133 0.00465" rpy="0 0 0"/>
-    <geometry>
-      <mesh filename="package://roomac_description/meshes/caster_right.stl" scale="0.001 0.001 0.001"/>
+    <material name="black"/>
+  </visual>
+  <collision>
+    <origin xyz="-0.001 -0.026 -0.10035" rpy="${pi/2.} 0 0"/>
+    <geometry>
+      <cylinder length="${caster_wheel_width}" radius="${caster_wheel_radius}"/>
     </geometry>
   </collision>
@@ -134,9 +137,10 @@
       <mesh filename="package://roomac_description/meshes/caster.dae" scale="0.001 0.001 0.001"/>
     </geometry>
-  </visual>
-  <collision>
-    <origin xyz="0.324 -0.139 0.00465" rpy="0 0 0"/>
-    <geometry>
-      <mesh filename="package://roomac_description/meshes/caster_left.stl" scale="0.001 0.001 0.001"/>
+    <material name="black"/>
+  </visual>
+  <collision>
+    <origin xyz="-0.001 0.022 -0.10035" rpy="${pi/2.} 0 0"/>
+    <geometry>
+      <cylinder length="${caster_wheel_width}" radius="${caster_wheel_radius}"/>
     </geometry>
   </collision>
@@ -153,4 +157,7 @@
 </joint>
 <!-- WHEELS -->
+<xacro:property name="wheel_width" value="0.062" />
+<xacro:property name="wheel_radius" value="0.145" />
+<xacro:property name="wheel_body_separation" value="0.01536" />
 <link name="wheel_right_link">
   <inertial>
@@ -164,9 +171,10 @@
       <mesh filename="package://roomac_description/meshes/wheel.dae" scale="0.001 0.001 0.001"/>
     </geometry>
-  </visual>
-  <collision>
-    <origin xyz="-0.0 0.21064 0.0" rpy="0 0 0"/>
-    <geometry>
-      <mesh filename="package://roomac_description/meshes/wheel_right.stl" scale="0.001 0.001 0.001"/>
+    <material name="black"/>
+  </visual>
+  <collision>
+    <origin xyz="0 ${-wheel_width/2. - wheel_body_separation} 0" rpy="${pi/2.} 0 0"/>
+    <geometry>
+      <cylinder length="${wheel_width}" radius="${wheel_radius}"/>
     </geometry>
   </collision>
@@ -183,9 +191,10 @@
       <mesh filename="package://roomac_description/meshes/wheel.dae" scale="0.001 0.001 0.001"/>
     </geometry>
-  </visual>
-  <collision>
-    <origin xyz="0.0 -0.21664 0.0" rpy="0 0 0"/>
-    <geometry>
-      <mesh filename="package://roomac_description/meshes/wheel_left.stl" scale="0.001 0.001 0.001"/>
+    <material name="black"/>
+  </visual>
+  <collision>
+    <origin xyz="0 ${wheel_width/2. + wheel_body_separation} 0" rpy="${pi/2.} 0 0"/>
+    <geometry>
+      <cylinder length="${wheel_width}" radius="${wheel_radius}"/>
     </geometry>
   </collision>
@@ -220,5 +229,5 @@
     <origin xyz="0.08 -2.1e-05 -0.969145" rpy="0 0 0"/>
     <geometry>
-      <mesh filename="package://roomac_description/meshes/head.stl" scale="0.001 0.001 0.001"/>
+      <mesh filename="package://roomac_description/meshes/head_collision.stl" scale="0.001 0.001 0.001"/>
     </geometry>
   </collision>
@@ -274,5 +283,5 @@
     <origin xyz="0.1135 0.174979 -0.9345" rpy="0 0 0"/>
     <geometry>
-      <mesh filename="package://roomac_description/meshes/shoulder_right.stl" scale="0.001 0.001 0.001"/>
+      <mesh filename="package://roomac_description/meshes/shoulder_right_collision.stl" scale="0.001 0.001 0.001"/>
     </geometry>
   </collision>
@@ -289,9 +298,10 @@
       <mesh filename="package://roomac_description/meshes/shoulder_elbow_right.dae" scale="0.001 0.001 0.001"/>
     </geometry>
+    <material name="black"/>
   </visual>
   <collision>
     <origin xyz="0.113 0.243979 -0.9345" rpy="0 0 0"/>
     <geometry>
-      <mesh filename="package://roomac_description/meshes/shoulder_elbow_right.stl" scale="0.001 0.001 0.001"/>
+      <mesh filename="package://roomac_description/meshes/shoulder_elbow_right_collision.stl" scale="0.001 0.001 0.001"/>
     </geometry>
   </collision>
@@ -313,5 +323,5 @@
     <origin xyz="0.0925 0.243979 -0.733425" rpy="0 0 0"/>
     <geometry>
-      <mesh filename="package://roomac_description/meshes/elbow_wrist_right.stl" scale="0.001 0.001 0.001"/>
+      <mesh filename="package://roomac_description/meshes/elbow_wrist_right_collision.stl" scale="0.001 0.001 0.001"/>
     </geometry>
   </collision>
@@ -333,5 +343,5 @@
     <origin xyz="0.139354 0.243979 -0.603583" rpy="0 0 0"/>
     <geometry>
-      <mesh filename="package://roomac_description/meshes/wrist_right.stl" scale="0.001 0.001 0.001"/>
+      <mesh filename="package://roomac_description/meshes/wrist_right_collision.stl" scale="0.001 0.001 0.001"/>
     </geometry>
   </collision>
@@ -353,5 +363,5 @@
     <origin xyz="0.114635 0.244052 -0.544791" rpy="0 0 0"/>
     <geometry>
-      <mesh filename="package://roomac_description/meshes/gripper_right.stl" scale="0.001 0.001 0.001"/>
+      <mesh filename="package://roomac_description/meshes/gripper_right_collision.stl" scale="0.001 0.001 0.001"/>
     </geometry>
   </collision>
@@ -376,5 +386,5 @@
     <origin xyz="0.117385 0.274314 -0.487684" rpy="0 0 0"/>
     <geometry>
-      <mesh filename="package://roomac_description/meshes/gripper_finger_r_right.stl" scale="0.001 0.001 0.001"/>
+      <mesh filename="package://roomac_description/meshes/gripper_finger_r_right_collision.stl" scale="0.001 0.001 0.001"/>
     </geometry>
   </collision>
@@ -396,5 +406,5 @@
     <origin xyz="0.117385 0.214585 -0.487684" rpy="0 0 0"/>
     <geometry>
-      <mesh filename="package://roomac_description/meshes/gripper_finger_l_right.stl" scale="0.001 0.001 0.001"/>
+      <mesh filename="package://roomac_description/meshes/gripper_finger_l_right_collision.stl" scale="0.001 0.001 0.001"/>
     </geometry>
   </collision>
@@ -476,5 +486,5 @@
     <origin xyz="0.1135 -0.175021 -0.9345" rpy="0 0 0"/>
     <geometry>
-      <mesh filename="package://roomac_description/meshes/shoulder_left.stl" scale="0.001 0.001 0.001"/>
+      <mesh filename="package://roomac_description/meshes/shoulder_left_collision.stl" scale="0.001 0.001 0.001"/>
     </geometry>
   </collision>
@@ -491,9 +501,10 @@
       <mesh filename="package://roomac_description/meshes/shoulder_elbow_left.dae" scale="0.001 0.001 0.001"/>
     </geometry>
+    <material name="black"/>
   </visual>
   <collision>
     <origin xyz="0.113 -0.244021 -0.9345" rpy="0 0 0"/>
     <geometry>
-      <mesh filename="package://roomac_description/meshes/shoulder_elbow_left.stl" scale="0.001 0.001 0.001"/>
+      <mesh filename="package://roomac_description/meshes/shoulder_elbow_left_collision.stl" scale="0.001 0.001 0.001"/>
     </geometry>
   </collision>
@@ -515,5 +526,5 @@
     <origin xyz="0.0925 -0.244021 -0.733443" rpy="0 0 0"/>
     <geometry>
-      <mesh filename="package://roomac_description/meshes/elbow_wrist_left.stl" scale="0.001 0.001 0.001"/>
+      <mesh filename="package://roomac_description/meshes/elbow_wrist_left_collision.stl" scale="0.001 0.001 0.001"/>
     </geometry>
   </collision>
@@ -535,5 +546,5 @@
     <origin xyz="0.139354 -0.244021 -0.603601" rpy="0 0 0"/>
     <geometry>
-      <mesh filename="package://roomac_description/meshes/wrist_left.stl" scale="0.001 0.001 0.001"/>
+      <mesh filename="package://roomac_description/meshes/wrist_left_collision.stl" scale="0.001 0.001 0.001"/>
     </geometry>
   </collision>
@@ -555,5 +566,5 @@
     <origin xyz="0.114635 -0.244094 -0.544809" rpy="0 0 0"/>
     <geometry>
-      <mesh filename="package://roomac_description/meshes/gripper_left.stl" scale="0.001 0.001 0.001"/>
+      <mesh filename="package://roomac_description/meshes/gripper_left_collision.stl" scale="0.001 0.001 0.001"/>
     </geometry>
   </collision>
@@ -575,5 +586,5 @@
     <origin xyz="0.117385 -0.274357 -0.487702" rpy="0 0 0"/>
     <geometry>
-      <mesh filename="package://roomac_description/meshes/gripper_finger_l_left.stl" scale="0.001 0.001 0.001"/>
+      <mesh filename="package://roomac_description/meshes/gripper_finger_l_left_collision.stl" scale="0.001 0.001 0.001"/>
     </geometry>
   </collision>
@@ -595,5 +606,5 @@
     <origin xyz="0.117385 -0.214627 -0.487702" rpy="0 0 0"/>
     <geometry>
-      <mesh filename="package://roomac_description/meshes/gripper_finger_r_left.stl" scale="0.001 0.001 0.001"/>
+      <mesh filename="package://roomac_description/meshes/gripper_finger_r_left_collision.stl" scale="0.001 0.001 0.001"/>
     </geometry>
   </collision>

Commit message: Fix left wheel

File: roomac_description/urdf/roomac_body.xacro (robot description, xacro)
@@ -187,5 +187,5 @@
   </inertial>
   <visual>
-    <origin xyz="0.0 -0.21664 0.0" rpy="0 0 0"/>
+    <origin xyz="0.0 -0.21064 0.0" rpy="0 0 0"/>
     <geometry>
       <mesh filename="package://roomac_description/meshes/wheel.dae" scale="0.001 0.001 0.001"/>
@@ -207,5 +207,5 @@
 </joint>
 <joint name="wheel_left" type="continuous">
-  <origin xyz="0.0 0.21664 0.0" rpy="0 0 0"/>
+  <origin xyz="0.0 0.21064 0.0" rpy="0 0 0"/>
   <parent link="base_link"/>
   <child link="wheel_left_link"/>

Commit message: Move frames into robot body

File: roomac_description/urdf/roomac_body.xacro (robot description, xacro)
@@ -12,12 +12,12 @@
 <link name="robot_body_link">
   <inertial>
-    <origin xyz="-0.14414593948878596 0.007272292388517288 0.4790557350675238" rpy="0 0 0"/>
-    <mass value="7.356876734373038"/>
-    <inertia ixx="0.055113" iyy="0.026097" izz="0.045184" ixy="-0.000286" iyz="-0.000998" ixz="0.003045"/>
+    <origin xyz="-0.13821660856078213 0.0043835143674895525 0.42578889973861744" rpy="0 0 0"/>
+    <mass value="12.267858710704742"/>
+    <inertia ixx="0.720301" iyy="0.677932" izz="0.200987" ixy="4.5e-05" iyz="-0.003874" ixz="0.025748"/>
   </inertial>
   <visual>
     <origin xyz="0 0 0" rpy="0 0 0"/>
     <geometry>
-      <mesh filename="package://roomac_description/meshes/robot_body.stl" scale="0.001 0.001 0.001"/>
+      <mesh filename="package://roomac_description/meshes/robot_body.dae" scale="0.001 0.001 0.001"/>
     </geometry>
     <material name="black"/>
@@ -37,13 +37,4 @@
     </geometry>
     <material name="white"/>
-  </visual>
-</link>
-<link name="frame_link">
-  <visual>
-    <origin xyz="0.06485 -0.10315 -0.52765" rpy="0 0 0"/>
-    <geometry>
-      <mesh filename="package://roomac_description/meshes/frame.dae" scale="0.001 0.001 0.001"/>
-    </geometry>
-    <material name="silver"/>
   </visual>
 </link>
@@ -61,9 +52,4 @@
   <parent link="base_link"/>
   <child link="robot_body_frames_link"/>
-</joint>
-<joint name="frame" type="fixed">
-  <origin xyz="-0.06485 0.10315 0.52765" rpy="0 0 0"/>
-  <parent link="base_link"/>
-  <child link="frame_link"/>
 </joint>
 <!-- KINECT -->
@@ -252,6 +238,6 @@
 </link>
 <joint name="head" type="fixed">
-  <origin xyz="-0.01515 -0.103129 0.441495" rpy="0 0 0"/>
-  <parent link="frame_link"/>
+  <origin xyz="-0.08 2.1e-05 0.969145" rpy="0 0 0"/>
+  <parent link="base_link"/>
   <child link="head_link"/>
 </joint>

Commit message: Change all visual meshes to dae

File: roomac_description/urdf/roomac_body.xacro (robot description, xacro)
@@ -34,5 +34,5 @@
     <origin xyz="0.223282 0.099058 0.0075" rpy="0 0 0"/>
     <geometry>
-      <mesh filename="package://roomac_description/meshes/robot_body_frames.stl" scale="0.001 0.001 0.001"/>
+      <mesh filename="package://roomac_description/meshes/robot_body_frames.dae" scale="0.001 0.001 0.001"/>
     </geometry>
     <material name="white"/>
@@ -208,5 +208,5 @@
     <origin xyz="0.08 -2.1e-05 -0.969145" rpy="0 0 0"/>
     <geometry>
-      <mesh filename="package://roomac_description/meshes/head.stl" scale="0.001 0.001 0.001"/>
+      <mesh filename="package://roomac_description/meshes/head.dae" scale="0.001 0.001 0.001"/>
     </geometry>
     <material name="black"/>
@@ -223,5 +223,5 @@
     <origin xyz="0.0825 0.055979 -1.083347" rpy="0 0 0"/>
     <geometry>
-      <mesh filename="package://roomac_description/meshes/eye_right.stl" scale="0.001 0.001 0.001"/>
+      <mesh filename="package://roomac_description/meshes/eye_right.dae" scale="0.001 0.001 0.001"/>
     </geometry>
     <material name="white"/>
@@ -232,5 +232,5 @@
     <origin xyz="0.0825 -0.056021 -1.083347" rpy="0 0 0"/>
     <geometry>
-      <mesh filename="package://roomac_description/meshes/eye_left.stl" scale="0.001 0.001 0.001"/>
+      <mesh filename="package://roomac_description/meshes/eye_left.dae" scale="0.001 0.001 0.001"/>
     </geometry>
     <material name="white"/>
@@ -262,5 +262,5 @@
     <origin xyz="0.1135 0.174979 -0.9345" rpy="0 0 0"/>
     <geometry>
-      <mesh filename="package://roomac_description/meshes/shoulder_right.stl" scale="0.001 0.001 0.001"/>
+      <mesh filename="package://roomac_description/meshes/shoulder_right.dae" scale="0.001 0.001 0.001"/>
     </geometry>
     <material name="black"/>
@@ -302,5 +302,5 @@
     <origin xyz="0.0925 0.243979 -0.733425" rpy="0 0 0"/>
     <geometry>
-      <mesh filename="package://roomac_description/meshes/elbow_wrist_right.stl" scale="0.001 0.001 0.001"/>
+      <mesh filename="package://roomac_description/meshes/elbow_wrist_right.dae" scale="0.001 0.001 0.001"/>
     </geometry>
     <material name="black"/>
@@ -322,5 +322,5 @@
     <origin xyz="0.139354 0.243979 -0.603583" rpy="0 0 0"/>
     <geometry>
-      <mesh filename="package://roomac_description/meshes/wrist_right.stl" scale="0.001 0.001 0.001"/>
+      <mesh filename="package://roomac_description/meshes/wrist_right.dae" scale="0.001 0.001 0.001"/>
     </geometry>
     <material name="black"/>
@@ -342,5 +342,5 @@
     <origin xyz="0.114635 0.244052 -0.544791" rpy="0 0 0"/>
     <geometry>
-      <mesh filename="package://roomac_description/meshes/gripper_right.stl" scale="0.001 0.001 0.001"/>
+      <mesh filename="package://roomac_description/meshes/gripper_right.dae" scale="0.001 0.001 0.001"/>
     </geometry>
     <material name="black"/>
@@ -365,5 +365,5 @@
     <origin xyz="0.117385 0.274314 -0.487684" rpy="0 0 0"/>
     <geometry>
-      <mesh filename="package://roomac_description/meshes/gripper_finger_r_right.stl" scale="0.001 0.001 0.001"/>
+      <mesh filename="package://roomac_description/meshes/gripper_finger_r_right.dae" scale="0.001 0.001 0.001"/>
     </geometry>
     <material name="black"/>
@@ -385,5 +385,5 @@
     <origin xyz="0.117385 0.214585 -0.487684" rpy="0 0 0"/>
     <geometry>
-      <mesh filename="package://roomac_description/meshes/gripper_finger_l_right.stl" scale="0.001 0.001 0.001"/>
+      <mesh filename="package://roomac_description/meshes/gripper_finger_l_right.dae" scale="0.001 0.001 0.001"/>
     </geometry>
     <material name="black"/>
@@ -465,5 +465,5 @@
     <origin xyz="0.1135 -0.175021 -0.9345" rpy="0 0 0"/>
     <geometry>
-      <mesh filename="package://roomac_description/meshes/shoulder_left.stl" scale="0.001 0.001 0.001"/>
+      <mesh filename="package://roomac_description/meshes/shoulder_left.dae" scale="0.001 0.001 0.001"/>
     </geometry>
     <material name="black"/>
@@ -505,5 +505,5 @@
     <origin xyz="0.0925 -0.244021 -0.733443" rpy="0 0 0"/>
     <geometry>
-      <mesh filename="package://roomac_description/meshes/elbow_wrist_left.stl" scale="0.001 0.001 0.001"/>
+      <mesh filename="package://roomac_description/meshes/elbow_wrist_left.dae" scale="0.001 0.001 0.001"/>
     </geometry>
     <material name="black"/>
@@ -525,5 +525,5 @@
     <origin xyz="0.139354 -0.244021 -0.603601" rpy="0 0 0"/>
     <geometry>
-      <mesh filename="package://roomac_description/meshes/wrist_left.stl" scale="0.001 0.001 0.001"/>
+      <mesh filename="package://roomac_description/meshes/wrist_left.dae" scale="0.001 0.001 0.001"/>
     </geometry>
     <material name="black"/>
@@ -545,5 +545,5 @@
     <origin xyz="0.114635 -0.244094 -0.544809" rpy="0 0 0"/>
     <geometry>
-      <mesh filename="package://roomac_description/meshes/gripper_left.stl" scale="0.001 0.001 0.001"/>
+      <mesh filename="package://roomac_description/meshes/gripper_left.dae" scale="0.001 0.001 0.001"/>
     </geometry>
     <material name="black"/>
@@ -565,5 +565,5 @@
     <origin xyz="0.117385 -0.274357 -0.487702" rpy="0 0 0"/>
     <geometry>
-      <mesh filename="package://roomac_description/meshes/gripper_finger_l_left.stl" scale="0.001 0.001 0.001"/>
+      <mesh filename="package://roomac_description/meshes/gripper_finger_l_left.dae" scale="0.001 0.001 0.001"/>
     </geometry>
     <material name="black"/>
@@ -585,5 +585,5 @@
     <origin xyz="0.117385 -0.214627 -0.487702" rpy="0 0 0"/>
     <geometry>
-      <mesh filename="package://roomac_description/meshes/gripper_finger_r_left.stl" scale="0.001 0.001 0.001"/>
+      <mesh filename="package://roomac_description/meshes/gripper_finger_r_left.dae" scale="0.001 0.001 0.001"/>
     </geometry>
     <material name="black"/>

Commit message: Combine frames with main body and eyes with head
moveit collision checking used visual only links, so I don't want to use them

File: roomac_description/urdf/roomac_body.xacro (robot description, xacro)
@@ -5,7 +5,4 @@
   <color rgba="0.15 0.15 0.15 1.0"/>
 </material>
-<!-- Some links are used only for visuals:
-  - robot_body_frames_link and artag_bundle_visual_link - collision model in robot_body_link takes them into account, and also there is no point in inertial attribute for them (again robot_body_link should be enough)
-  - eye_right_link and eye_left_link - similar to previous example collision model in head is enough -->
 <!-- BODY -->
 <link name="base_link" />
@@ -33,11 +30,23 @@
   </collision>
 </link>
-<link name="robot_body_frames_link">
-  <visual>
-    <origin xyz="0.223282 0.099058 0.0075" rpy="0 0 0"/>
-    <geometry>
-      <mesh filename="package://roomac_description/meshes/robot_body_frames.dae" scale="0.001 0.001 0.001"/>
-    </geometry>
-  </visual>
+<link name="head_link">
+  <inertial>
+    <origin xyz="-0.057525587412925475 -6.228687900878637e-07 0.06845033639955778" rpy="0 0 0"/>
+    <mass value="4.300223439076428"/>
+    <inertia ixx="0.025424" iyy="0.022772" izz="0.013755" ixy="0.0" iyz="-0.0" ixz="-0.001476"/>
+  </inertial>
+  <visual>
+    <origin xyz="0.08 -2.1e-05 -0.969145" rpy="0 0 0"/>
+    <geometry>
+      <mesh filename="package://roomac_description/meshes/head.dae" scale="0.001 0.001 0.001"/>
+    </geometry>
+    <material name="black"/>
+  </visual>
+  <collision>
+    <origin xyz="0.08 -2.1e-05 -0.969145" rpy="0 0 0"/>
+    <geometry>
+      <mesh filename="package://roomac_description/meshes/head_collision.stl" scale="0.001 0.001 0.001"/>
+    </geometry>
+  </collision>
 </link>
 <joint name="base_joint" type="fixed">
@@ -50,8 +59,8 @@
   <child link="robot_body_link"/>
 </joint>
-<joint name="robot_body_frames" type="fixed">
-  <origin xyz="-0.223282 -0.099058 -0.0075" rpy="0 0 0"/>
-  <parent link="base_link"/>
-  <child link="robot_body_frames_link"/>
+<joint name="head" type="fixed">
+  <origin xyz="-0.08 2.1e-05 0.969145" rpy="0 0 0"/>
+  <parent link="base_link"/>
+  <child link="head_link"/>
 </joint>
 <!-- KINECT -->
@@ -80,4 +89,7 @@
     </geometry>
   </visual>
+  <!-- No collision, visual mesh will be used for collision in moveit in melodic
+  (important, in noetic behaviour changed and it will be ignored, either case is alright, this collision is not important)
+  in gazebo collision will be ignored without collision tag -->
 </link>
 <joint name="artag_joint" type="fixed">
@@ -199,56 +211,4 @@
   <child link="wheel_left_link"/>
   <axis xyz="0 1 0"/>
-</joint>
-<!-- HEAD -->
-<link name="head_link">
-  <inertial>
-    <origin xyz="-0.057525587412925475 -6.228687900878637e-07 0.06845033639955778" rpy="0 0 0"/>
-    <mass value="4.300223439076428"/>
-    <inertia ixx="0.025424" iyy="0.022772" izz="0.013755" ixy="0.0" iyz="-0.0" ixz="-0.001476"/>
-  </inertial>
-  <visual>
-    <origin xyz="0.08 -2.1e-05 -0.969145" rpy="0 0 0"/>
-    <geometry>
-      <mesh filename="package://roomac_description/meshes/head.dae" scale="0.001 0.001 0.001"/>
-    </geometry>
-    <material name="black"/>
-  </visual>
-  <collision>
-    <origin xyz="0.08 -2.1e-05 -0.969145" rpy="0 0 0"/>
-    <geometry>
-      <mesh filename="package://roomac_description/meshes/head_collision.stl" scale="0.001 0.001 0.001"/>
-    </geometry>
-  </collision>
-</link>
-<link name="eye_right_link">
-  <visual>
-    <origin xyz="0.0825 0.055979 -1.083347" rpy="0 0 0"/>
-    <geometry>
-      <mesh filename="package://roomac_description/meshes/eye_right.dae" scale="0.001 0.001 0.001"/>
-    </geometry>
-  </visual>
-</link>
-<link name="eye_left_link">
-  <visual>
-    <origin xyz="0.0825 -0.056021 -1.083347" rpy="0 0 0"/>
-    <geometry>
-      <mesh filename="package://roomac_description/meshes/eye_left.dae" scale="0.001 0.001 0.001"/>
-    </geometry>
-  </visual>
-</link>
-<joint name="head" type="fixed">
-  <origin xyz="-0.08 2.1e-05 0.969145" rpy="0 0 0"/>
-  <parent link="base_link"/>
-  <child link="head_link"/>
-</joint>
-<joint name="eye_right" type="fixed">
-  <origin xyz="-0.0025 -0.056 0.114202" rpy="0 0 0"/>
-  <parent link="head_link"/>
-  <child link="eye_right_link"/>
-</joint>
-<joint name="eye_left" type="fixed">
-  <origin xyz="-0.0025 0.056 0.114202" rpy="0 0 0"/>
-  <parent link="head_link"/>
-  <child link="eye_left_link"/>
 </joint>
 <!-- RIGHT ARM -->

Commit message: Edit artag bundle dae
rename texture file
add scale into dae
remove camera and light

File: roomac_description/urdf/roomac_body.xacro (robot description, xacro)
@@ -86,5 +86,5 @@
     <origin rpy="0 0 0" xyz="0 0 0"/>
     <geometry>
-      <mesh filename="package://roomac_description/materials/artag_bundle.dae" scale="3.142857143 1.2 0.001"/>
+      <mesh filename="package://roomac_description/materials/artag_bundle.dae" scale="1 1 1"/>
     </geometry>
   </visual>

Commit message: Remove materials directory

File: roomac_description/urdf/roomac_body.xacro (robot description, xacro)
@@ -81,10 +81,9 @@
 <!-- ARTAG -->
 <link name="artag_link" />
-<!-- todo: move artag bundle file to meshes -->
 <link name="artag_bundle_visual_link">
   <visual>
     <origin rpy="0 0 0" xyz="0 0 0"/>
     <geometry>
-      <mesh filename="package://roomac_description/materials/artag_bundle.dae" scale="1 1 1"/>
+      <mesh filename="package://roomac_description/meshes/artag_bundle.dae" scale="1 1 1"/>
     </geometry>
   </visual>
