Commit message: Change joint names to include _joint postfix

File: roomac_description/urdf/roomac_body.xacro (robot description, xacro)
@@ -55,9 +55,9 @@
   <child link="base_link"/>
 </joint>
-<joint name="robot_body" type="fixed">
+<joint name="robot_body_joint" type="fixed">
   <parent link="base_link"/>
   <child link="robot_body_link"/>
 </joint>
-<joint name="head" type="fixed">
+<joint name="head_joint" type="fixed">
   <origin xyz="-0.08 2.1e-05 0.969145" rpy="0 0 0"/>
   <parent link="base_link"/>
@@ -97,5 +97,5 @@
   <child link="artag_link"/>
 </joint>
-<joint name="artag_joint_bundle_visual" type="fixed">
+<joint name="artag_bundle_visual_joint" type="fixed">
   <origin rpy="0 0 0" xyz="0.01 0.0 0.0"/>
   <parent link="artag_link"/>
@@ -145,10 +145,10 @@
   </collision>
 </link>
-<joint name="caster_right" type="fixed">
+<joint name="caster_right_joint" type="fixed">
   <origin xyz="-0.324 -0.133 -0.00465" rpy="0 0 0"/>
   <parent link="base_link"/>
   <child link="caster_right_link"/>
 </joint>
-<joint name="caster_left" type="fixed">
+<joint name="caster_left_joint" type="fixed">
   <origin xyz="-0.324 0.139 -0.00465" rpy="0 0 0"/>
   <parent link="base_link"/>
@@ -199,5 +199,5 @@
   </collision>
 </link>
-<joint name="wheel_right" type="continuous">
+<joint name="wheel_right_joint" type="continuous">
   <origin xyz="0.0 -0.21064 0.0" rpy="0 0 0"/>
   <parent link="base_link"/>
@@ -205,5 +205,5 @@
   <axis xyz="0 1 0"/>
 </joint>
-<joint name="wheel_left" type="continuous">
+<joint name="wheel_left_joint" type="continuous">
   <origin xyz="0.0 0.21064 0.0" rpy="0 0 0"/>
   <parent link="base_link"/>
@@ -357,5 +357,5 @@
 <!-- Values for effort and velocity are from example (they are required)
   not sure if correct, may need to change them -->
-<joint name="shoulder_pitch_right" type="revolute">
+<joint name="shoulder_pitch_right_joint" type="revolute">
   <origin xyz="-0.1135 -0.174979 0.9345" rpy="0 0 0"/>
   <parent link="base_link"/>
@@ -364,5 +364,5 @@
   <limit effort="30" velocity="1.0" lower="-2.390" upper="0.489" />
 </joint>
-<joint name="shoulder_roll_right" type="revolute">
+<joint name="shoulder_roll_right_joint" type="revolute">
   <origin xyz="0.0005 -0.069 0.0" rpy="0 0 0"/>
   <parent link="shoulder_right_link"/>
@@ -372,5 +372,5 @@
   <limit effort="30" velocity="1.0" lower="-0.800" upper="1.979" />
 </joint>
-<joint name="elbow_right" type="revolute">
+<joint name="elbow_right_joint" type="revolute">
   <origin xyz="0.0205 0.0 -0.201075" rpy="0 0 0"/>
   <parent link="shoulder_elbow_right_link"/>
@@ -381,5 +381,5 @@
   <limit effort="30" velocity="1.0" lower="-2.1" upper="2.1" />
 </joint>
-<joint name="wrist_right" type="revolute">
+<joint name="wrist_right_joint" type="revolute">
   <origin xyz="-0.046854 0.0 -0.129842" rpy="0 0 0"/>
   <parent link="elbow_wrist_right_link"/>
@@ -388,5 +388,5 @@
   <limit effort="30" velocity="1.0" lower="-1.994" upper="1.146" />
 </joint>
-<joint name="gripper_twist_right" type="revolute">
+<joint name="gripper_twist_right_joint" type="revolute">
   <origin xyz="0.024719 -7.3e-05 -0.058792" rpy="0 0 0"/>
   <parent link="wrist_right_link"/>
@@ -395,5 +395,5 @@
   <limit effort="30" velocity="1.0" lower="-1.570" upper="1.570" />
 </joint>
-<joint name="gripper_finger_r_right" type="prismatic">
+<joint name="gripper_finger_r_right_joint" type="prismatic">
   <origin xyz="-0.00275 -0.030262 -0.057107" rpy="0 0 0"/>
   <parent link="gripper_right_link"/>
@@ -402,5 +402,5 @@
   <limit effort="100" velocity="100" lower="-0.0045" upper="0.015"/>
 </joint>
-<joint name="gripper_finger_l_right" type="prismatic">
+<joint name="gripper_finger_l_right_joint" type="prismatic">
   <origin xyz="-0.00275 0.029467 -0.057107" rpy="0 0 0"/>
   <parent link="gripper_right_link"/>
@@ -409,5 +409,6 @@
   <limit effort="100" velocity="100" lower="-0.015" upper="0.0045"/>
 </joint>
-<joint name="right_grip" type="fixed">
+<!-- todo: change it -->
+<joint name="right_grip_joint" type="fixed">
   <origin rpy="0 0 0" xyz="0.0 0.0 -0.085"/>
   <parent link="gripper_right_link"/>
@@ -555,5 +556,5 @@
   </collision>
 </link>
-<joint name="shoulder_pitch_left" type="continuous">
+<joint name="shoulder_pitch_left_joint" type="continuous">
   <origin xyz="-0.1135 0.175021 0.9345" rpy="0 0 0"/>
   <parent link="base_link"/>
@@ -561,5 +562,5 @@
   <axis xyz="0 1 0"/>
 </joint>
-<joint name="shoulder_roll_left" type="continuous">
+<joint name="shoulder_roll_left_joint" type="continuous">
   <origin xyz="0.0005 0.069 0.0" rpy="0 0 0"/>
   <parent link="shoulder_left_link"/>
@@ -567,5 +568,5 @@
   <axis xyz="1 0 0"/>
 </joint>
-<joint name="elbow_left" type="continuous">
+<joint name="elbow_left_joint" type="continuous">
   <origin xyz="0.0205 0.0 -0.201057" rpy="0 0 0"/>
   <parent link="shoulder_elbow_left_link"/>
@@ -573,5 +574,5 @@
   <axis xyz="1 0 0"/>
 </joint>
-<joint name="wrist_left" type="continuous">
+<joint name="wrist_left_joint" type="continuous">
   <origin xyz="-0.046854 0.0 -0.129842" rpy="0 0 0"/>
   <parent link="elbow_wrist_left_link"/>
@@ -579,5 +580,5 @@
   <axis xyz="1 0 0"/>
 </joint>
-<joint name="gripper_twist_left" type="continuous">
+<joint name="gripper_twist_left_joint" type="continuous">
   <origin xyz="0.024719 7.3e-05 -0.058792" rpy="0 0 0"/>
   <parent link="wrist_left_link"/>
@@ -585,10 +586,10 @@
   <axis xyz="0 0 -1"/>
 </joint>
-<joint name="gripper_finger_r_left" type="fixed">
+<joint name="gripper_finger_r_left_joint" type="fixed">
   <origin xyz="-0.00275 -0.029467 -0.057107" rpy="0 0 0"/>
   <parent link="gripper_left_link"/>
   <child link="gripper_finger_r_left_link"/>
 </joint>
-<joint name="gripper_finger_l_left" type="fixed">
+<joint name="gripper_finger_l_left_joint" type="fixed">
   <origin xyz="-0.00275 0.030263 -0.057107" rpy="0 0 0"/>
   <parent link="gripper_left_link"/>
