Commit message: Add gripping link to urdf

File: roomac_description/urdf/roomac.xacro (robot description, xacro)
@@ -4,4 +4,10 @@
 <xacro:include filename="$(find roomac_description)/urdf/roomac.trans" />
 <xacro:include filename="$(find roomac_description)/urdf/roomac.gazebo" />
+<link name="gripper_right_grip"/>
+<joint name="right_grip" type="fixed">
+  <origin rpy="0 0 0" xyz="0.0 0.0 -0.085"/>
+  <parent link="gripper_right_1"/>
+  <child link="gripper_right_grip"/>
+</joint>
 <link name="base_link">
   <inertial>

Commit message: Fix caster joints

File: roomac_description/urdf/roomac.xacro (robot description, xacro)
@@ -52,10 +52,10 @@
 <link name="right_caster_1">
   <inertial>
-    <origin rpy="0 0 0" xyz="0.35270689508123315 -0.10093900679315995 -0.2719583755549746"/>
+    <origin rpy="0 0 0" xyz="-0.020793104918766903 -0.0009180067931599534 -0.11995837555497461"/>
     <mass value="1.2807118618501256"/>
     <inertia ixx="0.001622" ixy="-2e-06" ixz="-0.000322" iyy="0.002002" iyz="-8e-06" izz="0.000685"/>
   </inertial>
   <visual>
-    <origin rpy="0 0 0" xyz="0.672 0.059979 -0.1795"/>
+    <origin rpy="0 0 0" xyz="0.2985 0.16 -0.0275"/>
     <geometry>
       <mesh filename="package://roomac_description/meshes/right_caster_1.stl" scale="0.001 0.001 0.001"/>
@@ -64,5 +64,5 @@
   </visual>
   <collision>
-    <origin rpy="0 0 0" xyz="0.672 0.059979 -0.1795"/>
+    <origin rpy="0 0 0" xyz="0.2985 0.16 -0.0275"/>
     <geometry>
       <mesh filename="package://roomac_description/meshes/right_caster_1.stl" scale="0.001 0.001 0.001"/>
@@ -232,10 +232,10 @@
 <link name="left_caster_1">
   <inertial>
-    <origin rpy="0 0 0" xyz="0.35270689508120884 0.4928970067931112 -0.27195837555497454"/>
-    <mass value="1.2807118618501248"/>
-    <inertia ixx="0.001622" ixy="2e-06" ixz="-0.000322" iyy="0.002002" iyz="8e-06" izz="0.000685"/>
-  </inertial>
-  <visual>
-    <origin rpy="0 0 0" xyz="0.672 0.331979 -0.1795"/>
+    <origin rpy="0 0 0" xyz="-0.020793104918766903 -0.0009180067931599534 -0.11995837555497461"/>
+    <mass value="1.2807118618501256"/>
+    <inertia ixx="0.001622" ixy="-2e-06" ixz="-0.000322" iyy="0.002002" iyz="-8e-06" izz="0.000685"/>
+  </inertial>
+  <visual>
+    <origin rpy="0 0 0" xyz="0.2985 -0.16 -0.0275"/>
     <geometry>
       <mesh filename="package://roomac_description/meshes/left_caster_1.stl" scale="0.001 0.001 0.001"/>
@@ -244,5 +244,5 @@
   </visual>
   <collision>
-    <origin rpy="0 0 0" xyz="0.672 0.331979 -0.1795"/>
+    <origin rpy="0 0 0" xyz="0.2985 -0.16 -0.0275"/>
     <geometry>
       <mesh filename="package://roomac_description/meshes/left_caster_1.stl" scale="0.001 0.001 0.001"/>
@@ -396,5 +396,5 @@
 </joint>
 <joint name="right_caster" type="fixed">
-  <origin rpy="0 0 0" xyz="-0.672 -0.059979 0.1795"/>
+  <origin rpy="0 0 0" xyz="-0.2985 -0.16 0.0275"/>
   <parent link="base_link"/>
   <child link="right_caster_1"/>
@@ -446,5 +446,5 @@
 </joint>
 <joint name="left_caster" type="fixed">
-  <origin rpy="0 0 0" xyz="-0.672 -0.331979 0.1795"/>
+  <origin rpy="0 0 0" xyz="-0.2985 0.16 0.0275"/>
   <parent link="base_link"/>
   <child link="left_caster_1"/>

Commit message: Add kinect joint

File: roomac_description/urdf/roomac.xacro (robot description, xacro)
@@ -492,3 +492,9 @@
   <axis xyz="-0.0 1.0 0.0"/>
 </joint>
+<joint name="kinect_joint" type="fixed">
+		<origin rpy="0 ${(31.513/180.)*pi} 0" xyz="-0.108561 0.039543 0.479024"/>
+		<parent link="base_link"/>
+		<child link="camera_link"/>
+</joint>
+<link name="camera_link" />
 </robot>

Commit message: Add simulating diff drive in gazebo

File: roomac_description/urdf/roomac.xacro (robot description, xacro)
@@ -484,5 +484,5 @@
   <parent link="base_link"/>
   <child link="right_wheel_1"/>
-  <axis xyz="0.0 -1.0 -0.0"/>
+  <axis xyz="0.0 1.0 -0.0"/>
 </joint>
 <joint name="left_wheel" type="continuous">

Commit message: Add imu joint

File: roomac_description/urdf/roomac.xacro (robot description, xacro)
@@ -498,3 +498,9 @@
 </joint>
 <link name="camera_link" />
+<joint name="imu_joint" type="fixed">
+		<origin rpy="0 0 0" xyz="0 0 0"/>
+		<parent link="base_link"/>
+		<child link="imu"/>
+</joint>
+<link name="imu" />
 </robot>

Commit message: Fix pan and lift joints rotation direction

File: roomac_description/urdf/roomac.xacro (robot description, xacro)
@@ -404,5 +404,5 @@
   <parent link="base_up_1"/>
   <child link="shoulder_right_1"/>
-  <axis xyz="0.0 -1.0 -0.0"/>
+  <axis xyz="0.0 1.0 -0.0"/>
 </joint>
 <joint name="right_shoulder_lift" type="continuous">
@@ -410,5 +410,5 @@
   <parent link="shoulder_right_1"/>
   <child link="shoulder_elbow_right_1"/>
-  <axis xyz="1.0 0.0 -0.0"/>
+  <axis xyz="-1.0 0.0 -0.0"/>
 </joint>
 <joint name="right_elbow" type="continuous">

Commit message: Add artag to roomac model

File: roomac_description/urdf/roomac.xacro (robot description, xacro)
@@ -504,3 +504,28 @@
 </joint>
 <link name="imu" />
+<link name="artag_link">
+    <inertial>
+        <origin rpy="0 0 0" xyz="0 0 0"/>
+        <mass value="0.1"/>
+        <inertia ixx="0" ixy="-0.0" ixz="0.0" iyy="0" iyz="0.0" izz="0"/>
+    </inertial>
+    <visual name="visual">
+        <origin rpy="0 0 1.57" xyz="0.0 0.0 0.0"/>
+        <geometry>
+            <mesh filename="package://roomac_description/materials/aruco_cube_5cm.dae" scale="1 1 0.001"/>
+        </geometry>
+        <material name="artag"/>
+    </visual>
+    <collision>
+        <origin rpy="0 0 0" xyz="0.0 0.0 0.0"/>
+        <geometry>
+            <mesh filename="package://roomac_description/materials/aruco_cube_5cm.dae" scale="1 1 0.001"/>
+        </geometry>
+    </collision>
+</link>
+  <joint name="artag_joint" type="fixed">
+    <origin rpy="0 0 0" xyz="-0.1 -0.17 1"/>
+    <parent link="base_link"/>
+    <child link="artag_link"/>
+</joint>
 </robot>

Commit message: Add publishing tfs based on artag detection

File: roomac_description/urdf/roomac.xacro (robot description, xacro)
@@ -511,5 +511,5 @@
     </inertial>
     <visual name="visual">
-        <origin rpy="0 0 1.57" xyz="0.0 0.0 0.0"/>
+        <origin rpy="0 0 0" xyz="0.0 0.0 0.0"/>
         <geometry>
             <mesh filename="package://roomac_description/materials/aruco_cube_5cm.dae" scale="1 1 0.001"/>
@@ -529,3 +529,9 @@
     <child link="artag_link"/>
 </joint>
+<joint name="artag_joint_2" type="fixed">
+    <origin rpy="0 0 ${pi/2}" xyz="0 0 0"/>
+    <parent link="artag_link"/>
+    <child link="artag_link_2"/>
+</joint>
+<link name="artag_link_2"/>
 </robot>

Commit message: Add test gripper with moving fingers

File: roomac_description/urdf/roomac.xacro (robot description, xacro)
@@ -151,5 +151,5 @@
 </link>
 <link name="gripper_right_1">
-  <inertial>
+  <!-- <inertial>
     <origin rpy="0 0 0" xyz="0.0003095175801113986 0.0006959817920443867 -0.037223762933811466"/>
     <mass value="0.2826112434389509"/>
@@ -168,5 +168,83 @@
       <mesh filename="package://roomac_description/meshes/gripper_right_1.stl" scale="0.001 0.001 0.001"/>
     </geometry>
-  </collision>
+  </collision> -->
+  <collision>
+		<origin xyz="0 0 0" rpy="1.5708 0 0"/>
+		<geometry>
+			<cylinder length="0.1" radius="0.01"/>
+		</geometry>
+	</collision>
+	<visual>
+		<origin xyz="0 0 0" rpy="1.5708 0 0"/>
+		<geometry>
+			<cylinder length="0.1" radius="0.01"/>
+		</geometry>
+	</visual>
+	<inertial>
+		<origin xyz="0 0 0" rpy="1.5708 0 0"/>
+		<mass value="0.4"/>
+		<inertia
+			ixx="0.05" ixy="0.0" ixz="0.0"
+			iyy="0.002" iyz="0.0"
+			izz="0.05"/>
+	</inertial>
+</link>
+<joint name="finger1_joint" type="prismatic">
+	<parent link="gripper_right_1"/>
+	<child link="finger1"/>
+	<origin xyz="0 0.05 0" rpy="0 0 0"/>
+	<axis xyz="0 1 0"/>
+	<limit effort="100" velocity="100" lower="-0.05" upper="0.0"/>
+</joint>
+<link name="finger1">
+	<collision>
+		<origin xyz="0 0 -0.05" rpy="0 0 0"/>
+		<geometry>
+			<cylinder length="0.1" radius="0.01"/>
+		</geometry>
+	</collision>
+	<visual>
+		<origin xyz="0 0 -0.05" rpy="0 0 0"/>
+		<geometry>
+			<cylinder length="0.1" radius="0.01"/>
+		</geometry>
+	</visual>
+	<inertial>
+		<origin xyz="0 0 -0.05" rpy="0 0 0"/>
+		<mass value="0.2"/>
+		<inertia
+			ixx="0.02" ixy="0.0" ixz="0.0"
+			iyy="0.02" iyz="0.0"
+			izz="0.001"/>
+	</inertial>
+</link>
+<joint name="finger2_joint" type="prismatic">
+	<parent link="gripper_right_1"/>
+	<child link="finger2"/>
+	<origin xyz="0 -0.05 0" rpy="0 0 0"/>
+	<axis xyz="0 1 0"/>
+	<limit effort="100" velocity="100" lower="0.0" upper="0.05"/>
+</joint>
+<link name="finger2">
+	<collision>
+		<origin xyz="0 0 -0.05" rpy="0 0 0"/>
+		<geometry>
+			<cylinder length="0.1" radius="0.01"/>
+		</geometry>
+	</collision>
+	<visual>
+		<origin xyz="0 0 -0.05" rpy="0 0 0"/>
+		<geometry>
+			<cylinder length="0.1" radius="0.01"/>
+		</geometry>
+	</visual>
+	<inertial>
+		<origin xyz="0 0 -0.05" rpy="0 0 0"/>
+		<mass value="0.2"/>
+		<inertia
+			ixx="0.02" ixy="0.0" ixz="0.0"
+			iyy="0.02" iyz="0.0"
+			izz="0.001"/>
+	</inertial>
 </link>
 <link name="base_up_1">
@@ -425,5 +503,5 @@
 </joint>
 <joint name="right_gripper_twist" type="continuous">
-  <origin rpy="0 0 0" xyz="-0.025772 -7.3e-05 -0.057042"/>
+  <origin rpy="0 0 0" xyz="-0.025772 -7.3e-05 -0.097042"/>
   <parent link="wrist_right_1"/>
   <child link="gripper_right_1"/>

Commit message: Add limits to right arm urdf

File: roomac_description/urdf/roomac.xacro (robot description, xacro)
@@ -400,33 +400,43 @@
   <child link="right_caster_1"/>
 </joint>
-<joint name="right_shoulder_pan" type="continuous">
+<!-- Values for effort and velocity are from example (they are required)
+  not sure if correct, may need to change them -->
+<joint name="right_shoulder_pan" type="revolute">
   <origin rpy="0 0 0" xyz="-0.0505 -0.042479 0.405"/>
   <parent link="base_up_1"/>
   <child link="shoulder_right_1"/>
   <axis xyz="0.0 1.0 -0.0"/>
-</joint>
-<joint name="right_shoulder_lift" type="continuous">
+  <limit effort="30" velocity="1.0" lower="-2.390" upper="0.489" />
+</joint>
+<joint name="right_shoulder_lift" type="revolute">
   <origin rpy="0 0 0" xyz="-0.0265 -0.0995 0.0"/>
   <parent link="shoulder_right_1"/>
   <child link="shoulder_elbow_right_1"/>
   <axis xyz="-1.0 0.0 -0.0"/>
-</joint>
-<joint name="right_elbow" type="continuous">
+  <!-- Calculated lower: -0.899, adjusted it due to colision with gear-->
+  <limit effort="30" velocity="1.0" lower="-0.800" upper="1.979" />
+</joint>
+<joint name="right_elbow" type="revolute">
   <origin rpy="0 0 0" xyz="0.0425 0.0 -0.201075"/>
   <parent link="shoulder_elbow_right_1"/>
   <child link="elbow_wrist_right_1"/>
   <axis xyz="1.0 0.0 -0.0"/>
-</joint>
-<joint name="right_wrist" type="continuous">
+  <!-- Calculated lower: -2.879 upper: 2.879, adjusted due to collisions-->
+  <!-- Safe values, might be some room for increase -->
+  <limit effort="30" velocity="1.0" lower="-2.1" upper="2.1" />
+</joint>
+<joint name="right_wrist" type="revolute">
   <origin rpy="0 0 0" xyz="0.008637 0.0 -0.129818"/>
   <parent link="elbow_wrist_right_1"/>
   <child link="wrist_right_1"/>
   <axis xyz="-1.0 -0.0 0.0"/>
-</joint>
-<joint name="right_gripper_twist" type="continuous">
+  <limit effort="30" velocity="1.0" lower="-1.994" upper="1.146" />
+</joint>
+<joint name="right_gripper_twist" type="revolute">
   <origin rpy="0 0 0" xyz="-0.025772 -7.3e-05 -0.057042"/>
   <parent link="wrist_right_1"/>
   <child link="gripper_right_1"/>
   <axis xyz="-0.0 0.0 -1.0"/>
+  <limit effort="30" velocity="1.0" lower="-1.570" upper="1.570" />
 </joint>
 <joint name="up_base" type="fixed">

Commit message: Change fingers to cubes

File: roomac_description/urdf/roomac.xacro (robot description, xacro)
@@ -199,17 +199,17 @@
 <link name="finger1">
 	<collision>
-		<origin xyz="0 0 -0.05" rpy="0 0 0"/>
+		<origin xyz="0 0 -0.03" rpy="0 0 0"/>
 		<geometry>
-			<cylinder length="0.1" radius="0.01"/>
+      <box size="0.02 0.02 0.06" />
 		</geometry>
 	</collision>
 	<visual>
-		<origin xyz="0 0 -0.05" rpy="0 0 0"/>
+		<origin xyz="0 0 -0.03" rpy="0 0 0"/>
 		<geometry>
-			<cylinder length="0.1" radius="0.01"/>
+      <box size="0.02 0.02 0.06" />
 		</geometry>
 	</visual>
 	<inertial>
-		<origin xyz="0 0 -0.05" rpy="0 0 0"/>
+		<origin xyz="0 0 -0.03" rpy="0 0 0"/>
 		<mass value="0.2"/>
 		<inertia
@@ -228,17 +228,17 @@
 <link name="finger2">
 	<collision>
-		<origin xyz="0 0 -0.05" rpy="0 0 0"/>
+		<origin xyz="0 0 -0.03" rpy="0 0 0"/>
 		<geometry>
-			<cylinder length="0.1" radius="0.01"/>
+      <box size="0.02 0.02 0.06" />
 		</geometry>
 	</collision>
 	<visual>
-		<origin xyz="0 0 -0.05" rpy="0 0 0"/>
+		<origin xyz="0 0 -0.03" rpy="0 0 0"/>
 		<geometry>
-			<cylinder length="0.1" radius="0.01"/>
+      <box size="0.02 0.02 0.06" />
 		</geometry>
 	</visual>
 	<inertial>
-		<origin xyz="0 0 -0.05" rpy="0 0 0"/>
+		<origin xyz="0 0 -0.03" rpy="0 0 0"/>
 		<mass value="0.2"/>
 		<inertia

Commit message: Update ar tag position on robot

File: roomac_description/urdf/roomac.xacro (robot description, xacro)
@@ -613,5 +613,6 @@
 </link>
   <joint name="artag_joint" type="fixed">
-    <origin rpy="0 0 0" xyz="-0.1 -0.17 1"/>
+    <!-- Real z position is 0.972, but I had to add 12mm (height of plywood) - this urdf is older - pre base rework -->
+    <origin rpy="0 0 0" xyz="-0.149 -0.125 0.984"/>
     <parent link="base_link"/>
     <child link="artag_link"/>

Commit message: Comment out fingers, get back to previous gripper

File: roomac_description/urdf/roomac.xacro (robot description, xacro)
@@ -151,5 +151,5 @@
 </link>
 <link name="gripper_right_1">
-  <!-- <inertial>
+  <inertial>
     <origin rpy="0 0 0" xyz="0.0003095175801113986 0.0006959817920443867 -0.037223762933811466"/>
     <mass value="0.2826112434389509"/>
@@ -168,6 +168,6 @@
       <mesh filename="package://roomac_description/meshes/gripper_right_1.stl" scale="0.001 0.001 0.001"/>
     </geometry>
-  </collision> -->
-  <collision>
+  </collision>
+  <!-- <collision>
 		<origin xyz="0 0 0" rpy="1.5708 0 0"/>
 		<geometry>
@@ -188,7 +188,7 @@
 			iyy="0.002" iyz="0.0"
 			izz="0.05"/>
-	</inertial>
-</link>
-<joint name="finger1_joint" type="prismatic">
+	</inertial> -->
+</link>
+<!-- <joint name="finger1_joint" type="prismatic">
 	<parent link="gripper_right_1"/>
 	<child link="finger1"/>
@@ -247,5 +247,5 @@
 			izz="0.001"/>
 	</inertial>
-</link>
+</link> -->
 <link name="base_up_1">
   <inertial>

Commit message: Update IMU position in urdf

File: roomac_description/urdf/roomac.xacro (robot description, xacro)
@@ -509,5 +509,5 @@
 <link name="camera_link" />
 <joint name="imu_joint" type="fixed">
-		<origin rpy="0 0 0" xyz="0 0 0"/>
+		<origin rpy="0 0 0" xyz="-0.09873 -0.0375 0.0305"/>
 		<parent link="base_link"/>
 		<child link="imu"/>

Commit message: Add artag bundle to robot model

File: roomac_description/urdf/roomac.xacro (robot description, xacro)
@@ -7,3 +7,9 @@
 <xacro:include filename="$(find roomac_description)/urdf/roomac_gripper_real.xacro" />
 <xacro:include filename="$(find roomac_description)/urdf/roomac_arm_precision_test.xacro" />
+<joint name="artag_joint_2" type="fixed">
+    <origin rpy="0 0 ${pi/2}" xyz="0.0595 -0.004 0"/>
+    <parent link="artag_link"/>
+    <child link="artag_link_2"/>
+</joint>
+<link name="artag_link_2"/>
 </robot>

File: roomac_description/urdf/roomac_body.xacro (robot description, xacro)
@@ -493,4 +493,12 @@
 <link name="imu" />
 <link name="artag_link">
+</link>
+<joint name="artag_joint" type="fixed">
+    <!-- Real z position is 0.972, but I had to add 12mm (height of plywood) - this urdf is older - pre base rework -->
+    <origin rpy="0 0 0" xyz="-0.149 -0.125 0.984"/>
+    <parent link="base_link"/>
+    <child link="artag_link"/>
+</joint>
+<link name="artag_link_bundle_visual">
     <inertial>
         <origin rpy="0 0 0" xyz="0 0 0"/>
@@ -501,5 +509,5 @@
         <origin rpy="0 0 0" xyz="0.0 0.0 0.0"/>
         <geometry>
-            <mesh filename="package://roomac_description/materials/aruco_cube_5cm.dae" scale="1.2 1.2 0.001"/>
+            <mesh filename="package://roomac_description/materials/artag_bundle.dae" scale="3.142857143 1.2 0.001"/>
         </geometry>
         <material name="artag"/>
@@ -508,19 +516,12 @@
         <origin rpy="0 0 0" xyz="0.0 0.0 0.0"/>
         <geometry>
-            <mesh filename="package://roomac_description/materials/aruco_cube_5cm.dae" scale="1.2 1.2 0.001"/>
+            <mesh filename="package://roomac_description/materials/artag_bundle.dae" scale="3.142857143 1.2 0.001"/>
         </geometry>
     </collision>
 </link>
-  <joint name="artag_joint" type="fixed">
-    <!-- Real z position is 0.972, but I had to add 12mm (height of plywood) - this urdf is older - pre base rework -->
-    <origin rpy="0 0 0" xyz="-0.149 -0.125 0.984"/>
-    <parent link="base_link"/>
-    <child link="artag_link"/>
-</joint>
-<joint name="artag_joint_2" type="fixed">
-    <origin rpy="0 0 ${pi/2}" xyz="0.0595 -0.004 0"/>
+<joint name="artag_joint_bundle_visual" type="fixed">
+    <origin rpy="0 0 0" xyz="0.01 0.0 0"/>
     <parent link="artag_link"/>
-    <child link="artag_link_2"/>
-</joint>
-<link name="artag_link_2"/>
+    <child link="artag_link_bundle_visual"/>
+</joint>
 </robot>

File: roomac_description/urdf/roomac_simulation_picking.xacro (robot description, xacro)
@@ -9,3 +9,9 @@
 <xacro:include filename="$(find roomac_description)/urdf/roomac_gripper_simulation.trans" />
 <xacro:include filename="$(find roomac_description)/urdf/roomac_arm_precision_test.xacro" />
+<joint name="artag_joint_2" type="fixed">
+    <origin rpy="${-pi/2} 0 0" xyz="0.04857 0 0"/>
+    <parent link="artag_link_bundle_visual"/>
+    <child link="artag_link_2"/>
+</joint>
+<link name="artag_link_2"/>
 </robot>

Commit message: Rename artag link 2 to artag link bundle

File: roomac_description/urdf/roomac.xacro (robot description, xacro)
@@ -7,9 +7,9 @@
 <xacro:include filename="$(find roomac_description)/urdf/roomac_gripper_real.xacro" />
 <xacro:include filename="$(find roomac_description)/urdf/roomac_arm_precision_test.xacro" />
-<joint name="artag_joint_2" type="fixed">
+<joint name="artag_joint_bundle" type="fixed">
     <origin rpy="0 0 ${pi/2}" xyz="0.0595 -0.004 0"/>
     <parent link="artag_link"/>
-    <child link="artag_link_2"/>
+    <child link="artag_link_bundle"/>
 </joint>
-<link name="artag_link_2"/>
+<link name="artag_link_bundle"/>
 </robot>

File: roomac_description/urdf/roomac_simulation_picking.xacro (robot description, xacro)
@@ -9,9 +9,9 @@
 <xacro:include filename="$(find roomac_description)/urdf/roomac_gripper_simulation.trans" />
 <xacro:include filename="$(find roomac_description)/urdf/roomac_arm_precision_test.xacro" />
-<joint name="artag_joint_2" type="fixed">
+<joint name="artag_joint_bundle" type="fixed">
     <origin rpy="${-pi/2} 0 0" xyz="0.04857 0 0"/>
     <parent link="artag_link_bundle_visual"/>
-    <child link="artag_link_2"/>
+    <child link="artag_link_bundle"/>
 </joint>
-<link name="artag_link_2"/>
+<link name="artag_link_bundle"/>
 </robot>
