Commit message: Change fingers in simulation to real gripper's ones

File: roomac_description/urdf/roomac.xacro (robot description, xacro)
@@ -5,5 +5,4 @@
 <xacro:include filename="$(find roomac_description)/urdf/roomac.gazebo" />
 <xacro:include filename="$(find roomac_description)/urdf/roomac_body.xacro" />
-<xacro:include filename="$(find roomac_description)/urdf/roomac_gripper_real.xacro" />
 <xacro:include filename="$(find roomac_description)/urdf/roomac_arm_precision_test.xacro" />
 <joint name="artag_joint_bundle" type="fixed">

File: roomac_description/urdf/roomac_body.xacro (robot description, xacro)
@@ -594,4 +594,65 @@
     <geometry>
       <mesh filename="package://roomac_description/meshes/wrist_right_1.stl" scale="0.001 0.001 0.001"/>
+    </geometry>
+  </collision>
+</link>
+<link name="gripper_right_grip"/>
+<link name="gripper_right_1">
+  <inertial>
+    <origin xyz="-0.00024163561260628907 0.001034172528649041 -0.024005885240587554" rpy="0 0 0"/>
+    <mass value="0.20788263258389922"/>
+    <inertia ixx="8.7e-05" iyy="5.3e-05" izz="5.8e-05" ixy="4e-06" iyz="-1e-06" ixz="3e-06"/>
+  </inertial>
+  <visual>
+    <origin xyz="0.114635 0.244052 -0.544809" rpy="0 0 0"/>
+    <geometry>
+      <mesh filename="package://roomac_description/meshes/gripper_right_1.stl" scale="0.001 0.001 0.001"/>
+    </geometry>
+    <material name="black"/>
+  </visual>
+  <collision>
+    <origin xyz="0.114635 0.244052 -0.544809" rpy="0 0 0"/>
+    <geometry>
+      <mesh filename="package://roomac_description/meshes/gripper_right_1.stl" scale="0.001 0.001 0.001"/>
+    </geometry>
+  </collision>
+</link>
+<link name="gripper_finger_1_right_1">
+  <inertial>
+    <origin xyz="0.004500248654849631 0.005686730533079498 -0.01101605906930514" rpy="0 0 0"/>
+    <mass value="0.03746064390067365"/>
+    <inertia ixx="1.2e-05" iyy="1e-05" izz="2e-06" ixy="-0.0" iyz="4e-06" ixz="-0.0"/>
+  </inertial>
+  <visual>
+    <origin xyz="0.117385 0.274314 -0.487702" rpy="0 0 0"/>
+    <geometry>
+      <mesh filename="package://roomac_description/meshes/gripper_finger_1_right_1.stl" scale="0.001 0.001 0.001"/>
+    </geometry>
+    <material name="black"/>
+  </visual>
+  <collision>
+    <origin xyz="0.117385 0.274314 -0.487702" rpy="0 0 0"/>
+    <geometry>
+      <mesh filename="package://roomac_description/meshes/gripper_finger_1_right_1.stl" scale="0.001 0.001 0.001"/>
+    </geometry>
+  </collision>
+</link>
+<link name="gripper_finger_2_right_1">
+  <inertial>
+    <origin xyz="0.00450024860853869 -0.005494466336699089 -0.011113636952014339" rpy="0 0 0"/>
+    <mass value="0.037460643900623564"/>
+    <inertia ixx="1.2e-05" iyy="1e-05" izz="2e-06" ixy="-0.0" iyz="-4e-06" ixz="-0.0"/>
+  </inertial>
+  <visual>
+    <origin xyz="0.117385 0.214585 -0.487702" rpy="0 0 0"/>
+    <geometry>
+      <mesh filename="package://roomac_description/meshes/gripper_finger_2_right_1.stl" scale="0.001 0.001 0.001"/>
+    </geometry>
+    <material name="black"/>
+  </visual>
+  <collision>
+    <origin xyz="0.117385 0.214585 -0.487702" rpy="0 0 0"/>
+    <geometry>
+      <mesh filename="package://roomac_description/meshes/gripper_finger_2_right_1.stl" scale="0.001 0.001 0.001"/>
     </geometry>
   </collision>
@@ -652,4 +713,23 @@
   <limit effort="30" velocity="1.0" lower="-1.570" upper="1.570" />
 </joint>
+<joint name="gripper_finger_r_right" type="prismatic">
+  <origin xyz="-0.00275 -0.030262 -0.057107" rpy="0 0 0"/>
+  <parent link="gripper_right_1"/>
+  <child link="gripper_finger_1_right_1"/>
+  <axis xyz="0 1 0"/>
+  <limit effort="100" velocity="100" lower="-0.0045" upper="0.015"/>
+</joint>
+<joint name="gripper_finger_l_right" type="prismatic">
+  <origin xyz="-0.00275 0.029467 -0.057107" rpy="0 0 0"/>
+  <parent link="gripper_right_1"/>
+  <child link="gripper_finger_2_right_1"/>
+  <axis xyz="0 1 0"/>
+  <limit effort="100" velocity="100" lower="-0.015" upper="0.0045"/>
+</joint>
+<joint name="right_grip" type="fixed">
+  <origin rpy="0 0 0" xyz="0.0 0.0 -0.085"/>
+  <parent link="gripper_right_1"/>
+  <child link="gripper_right_grip"/>
+</joint>
 <!-- LEFT ARM -->
 <link name="shoulder_base_left_1">

File: roomac_description/urdf/roomac_simulation_picking.xacro (robot description, xacro)
@@ -5,7 +5,4 @@
 <xacro:include filename="$(find roomac_description)/urdf/roomac.gazebo" />
 <xacro:include filename="$(find roomac_description)/urdf/roomac_body.xacro" />
-<xacro:include filename="$(find roomac_description)/urdf/roomac_gripper_simulation.xacro" />
-<xacro:include filename="$(find roomac_description)/urdf/roomac_gripper_simulation.gazebo" />
-<xacro:include filename="$(find roomac_description)/urdf/roomac_gripper_simulation.trans" />
 <xacro:include filename="$(find roomac_description)/urdf/roomac_arm_precision_test.xacro" />
 <joint name="artag_joint_bundle" type="fixed">
