Commit message: Change link names to name with _link suffix

File: roomac_description/urdf/roomac.xacro (robot description, xacro)
@@ -6,9 +6,9 @@
 <xacro:include filename="$(find roomac_description)/urdf/roomac_body.xacro" />
 <xacro:include filename="$(find roomac_description)/urdf/roomac_arm_precision_test.xacro" />
+<link name="artag_bundle_link"/>
 <joint name="artag_joint_bundle" type="fixed">
     <origin rpy="0 0 ${pi/2}" xyz="0.0595 -0.004 0"/>
     <parent link="artag_link"/>
-    <child link="artag_link_bundle"/>
+    <child link="artag_bundle_link"/>
 </joint>
-<link name="artag_link_bundle"/>
 </robot>

File: roomac_description/urdf/roomac_arm_precision_test.xacro (robot description, xacro)
@@ -1,15 +1,15 @@
 <?xml version="1.0" ?>
 <robot name="roomac" xmlns:xacro="http://www.ros.org/wiki/xacro">
-  <link name="gripper_right_precision_test_tip"/>
+  <link name="gripper_right_precision_test_tip_link"/>
   <joint name="gripper_right_precision_test_tip_joint" type="fixed">
     <origin rpy="0 0 0" xyz="0.005894 0.0 -0.109041"/>
-    <parent link="gripper_right_1"/>
-    <child link="gripper_right_precision_test_tip"/>
+    <parent link="gripper_right_link"/>
+    <child link="gripper_right_precision_test_tip_link"/>
   </joint>
-  <link name="body_precision_test_tip"/>
+  <link name="body_precision_test_tip_link"/>
   <joint name="body_precision_test_tip_joint" type="fixed">
     <origin rpy="0 0 0" xyz="0.01115 0.0 0.9474945"/>
     <parent link="base_link"/>
-    <child link="body_precision_test_tip"/>
+    <child link="body_precision_test_tip_link"/>
   </joint>
 </robot>

File: roomac_description/urdf/roomac_body.xacro (robot description, xacro)
@@ -1,4 +1,5 @@
 <?xml version="1.0" ?>
 <robot name="roomac" xmlns:xacro="http://www.ros.org/wiki/xacro">
+<!-- todo: standardize joint names -->
 <!-- BODY -->
 <link name="base_link" />
@@ -6,5 +7,5 @@
 <!-- Additional link needed to solve moveit warning (as far as I know it shouldn't cause any issue as I'm not using KDL, but still better to solve it): -->
 <!-- The root link base_link has an inertia specified in the URDF, but KDL does not support a root link with an inertia.  As a workaround, you can add an extra dummy link to your URDF. -->
-<link name="robot_body_1">
+<link name="robot_body_link">
   <inertial>
     <origin xyz="-0.14414593948878596 0.007272292388517288 0.4790557350675238" rpy="0 0 0"/>
@@ -26,5 +27,5 @@
   </collision>
 </link>
-<link name="base_link_frames_1">
+<link name="robot_body_frames_link">
   <inertial>
     <origin xyz="0.09299736209064594 0.09816853953024438 0.7758797564332383" rpy="0 0 0"/>
@@ -35,5 +36,5 @@
     <origin xyz="0.223282 0.099058 0.0075" rpy="0 0 0"/>
     <geometry>
-      <mesh filename="package://roomac_description/meshes/base_link_frames_1.stl" scale="0.001 0.001 0.001"/>
+      <mesh filename="package://roomac_description/meshes/robot_body_frames_link.stl" scale="0.001 0.001 0.001"/>
     </geometry>
     <material name="white"/>
@@ -42,9 +43,9 @@
     <origin xyz="0.223282 0.099058 0.0075" rpy="0 0 0"/>
     <geometry>
-      <mesh filename="package://roomac_description/meshes/base_link_frames_1.stl" scale="0.001 0.001 0.001"/>
-    </geometry>
-  </collision>
-</link>
-<link name="frame_1">
+      <mesh filename="package://roomac_description/meshes/robot_body_frames_link.stl" scale="0.001 0.001 0.001"/>
+    </geometry>
+  </collision>
+</link>
+<link name="frame_link">
   <inertial>
     <origin xyz="-0.06363233755923882 -0.10316506754069626 -0.18305645699853168" rpy="0 0 0"/>
@@ -55,5 +56,5 @@
     <origin xyz="0.06485 -0.10315 -0.52765" rpy="0 0 0"/>
     <geometry>
-      <mesh filename="package://roomac_description/meshes/frame_1.stl" scale="0.001 0.001 0.001"/>
+      <mesh filename="package://roomac_description/meshes/frame_link.stl" scale="0.001 0.001 0.001"/>
     </geometry>
     <material name="silver"/>
@@ -62,5 +63,5 @@
     <origin xyz="0.06485 -0.10315 -0.52765" rpy="0 0 0"/>
     <geometry>
-      <mesh filename="package://roomac_description/meshes/frame_1.stl" scale="0.001 0.001 0.001"/>
+      <mesh filename="package://roomac_description/meshes/frame_link.stl" scale="0.001 0.001 0.001"/>
     </geometry>
   </collision>
@@ -73,15 +74,15 @@
 <joint name="robot_body" type="fixed">
   <parent link="base_link"/>
-  <child link="robot_body_1"/>
-</joint>
-<joint name="base_link_frames" type="fixed">
+  <child link="robot_body_link"/>
+</joint>
+<joint name="robot_body_frames" type="fixed">
   <origin xyz="-0.223282 -0.099058 -0.0075" rpy="0 0 0"/>
   <parent link="base_link"/>
-  <child link="base_link_frames_1"/>
+  <child link="robot_body_frames_link"/>
 </joint>
 <joint name="frame" type="fixed">
   <origin xyz="-0.06485 0.10315 0.52765" rpy="0 0 0"/>
   <parent link="base_link"/>
-  <child link="frame_1"/>
+  <child link="frame_link"/>
 </joint>
 <!-- KINECT -->
@@ -94,13 +95,13 @@
 </joint>
 <!-- IMU -->
-<link name="imu" />
+<link name="imu_link" />
 <joint name="imu_joint" type="fixed">
   <origin rpy="0 0 0" xyz="-0.09873 -0.0375 0.0305"/>
   <parent link="base_link"/>
-  <child link="imu"/>
+  <child link="imu_link"/>
 </joint>
 <!-- ARTAG -->
 <link name="artag_link" />
-<link name="artag_link_bundle_visual">
+<link name="artag_bundle_visual_link">
   <inertial>
     <origin rpy="0 0 0" xyz="0 0 0"/>
@@ -129,8 +130,8 @@
   <origin rpy="0 0 0" xyz="0.01 0.0 0.0"/>
   <parent link="artag_link"/>
-  <child link="artag_link_bundle_visual"/>
+  <child link="artag_bundle_visual_link"/>
 </joint>
 <!-- CASTERS -->
-<link name="caster_right_1">
+<link name="caster_right_link">
   <inertial>
     <origin xyz="0.00355868425330208 -0.0279262663780577 -0.08858638249680677" rpy="0 0 0"/>
@@ -147,9 +148,9 @@
     <origin xyz="0.324 0.133 0.00465" rpy="0 0 0"/>
     <geometry>
-      <mesh filename="package://roomac_description/meshes/caster_right_1.stl" scale="0.001 0.001 0.001"/>
-    </geometry>
-  </collision>
-</link>
-<link name="caster_left_1">
+      <mesh filename="package://roomac_description/meshes/caster_right_link.stl" scale="0.001 0.001 0.001"/>
+    </geometry>
+  </collision>
+</link>
+<link name="caster_left_link">
   <inertial>
     <origin xyz="0.0035586842533020246 0.02192626637805642 -0.0885863824968092" rpy="0 0 0"/>
@@ -166,5 +167,5 @@
     <origin xyz="0.324 -0.139 0.00465" rpy="0 0 0"/>
     <geometry>
-      <mesh filename="package://roomac_description/meshes/caster_left_1.stl" scale="0.001 0.001 0.001"/>
+      <mesh filename="package://roomac_description/meshes/caster_left_link.stl" scale="0.001 0.001 0.001"/>
     </geometry>
   </collision>
@@ -173,13 +174,13 @@
   <origin xyz="-0.324 -0.133 -0.00465" rpy="0 0 0"/>
   <parent link="base_link"/>
-  <child link="caster_right_1"/>
+  <child link="caster_right_link"/>
 </joint>
 <joint name="caster_left" type="fixed">
   <origin xyz="-0.324 0.139 -0.00465" rpy="0 0 0"/>
   <parent link="base_link"/>
-  <child link="caster_left_1"/>
+  <child link="caster_left_link"/>
 </joint>
 <!-- WHEELS -->
-<link name="wheel_right_1">
+<link name="wheel_right_link">
   <inertial>
     <origin xyz="-8.535155939829862e-08 -0.045545810193822645 1.2324269625501287e-07" rpy="0 0 0"/>
@@ -196,9 +197,9 @@
     <origin xyz="-0.0 0.21064 0.0" rpy="0 0 0"/>
     <geometry>
-      <mesh filename="package://roomac_description/meshes/wheel_right_1.stl" scale="0.001 0.001 0.001"/>
-    </geometry>
-  </collision>
-</link>
-<link name="wheel_left_1">
+      <mesh filename="package://roomac_description/meshes/wheel_right_link.stl" scale="0.001 0.001 0.001"/>
+    </geometry>
+  </collision>
+</link>
+<link name="wheel_left_link">
   <inertial>
     <origin xyz="-7.854137935392783e-08 0.039545809782175645 1.1633993854093376e-07" rpy="0 0 0"/>
@@ -215,5 +216,5 @@
     <origin xyz="0.0 -0.21664 0.0" rpy="0 0 0"/>
     <geometry>
-      <mesh filename="package://roomac_description/meshes/wheel_left_1.stl" scale="0.001 0.001 0.001"/>
+      <mesh filename="package://roomac_description/meshes/wheel_left_link.stl" scale="0.001 0.001 0.001"/>
     </geometry>
   </collision>
@@ -222,5 +223,5 @@
   <origin xyz="0.0 -0.21064 0.0" rpy="0 0 0"/>
   <parent link="base_link"/>
-  <child link="wheel_right_1"/>
+  <child link="wheel_right_link"/>
   <axis xyz="0 1 0"/>
 </joint>
@@ -228,9 +229,9 @@
   <origin xyz="0.0 0.21664 0.0" rpy="0 0 0"/>
   <parent link="base_link"/>
-  <child link="wheel_left_1"/>
+  <child link="wheel_left_link"/>
   <axis xyz="0 1 0"/>
 </joint>
 <!-- HEAD -->
-<link name="head_1">
+<link name="head_link">
   <inertial>
     <origin xyz="-0.057525587412925475 -6.228687900878637e-07 0.06845033639955778" rpy="0 0 0"/>
@@ -241,5 +242,5 @@
     <origin xyz="0.08 -2.1e-05 -0.969145" rpy="0 0 0"/>
     <geometry>
-      <mesh filename="package://roomac_description/meshes/head_1.stl" scale="0.001 0.001 0.001"/>
+      <mesh filename="package://roomac_description/meshes/head_link.stl" scale="0.001 0.001 0.001"/>
     </geometry>
     <material name="black"/>
@@ -248,9 +249,9 @@
     <origin xyz="0.08 -2.1e-05 -0.969145" rpy="0 0 0"/>
     <geometry>
-      <mesh filename="package://roomac_description/meshes/head_1.stl" scale="0.001 0.001 0.001"/>
-    </geometry>
-  </collision>
-</link>
-<link name="eye_right_1">
+      <mesh filename="package://roomac_description/meshes/head_link.stl" scale="0.001 0.001 0.001"/>
+    </geometry>
+  </collision>
+</link>
+<link name="eye_right_link">
   <inertial>
     <origin xyz="0.00626024105824001 3.517735655544918e-08 -3.559806300845736e-07" rpy="0 0 0"/>
@@ -261,5 +262,5 @@
     <origin xyz="0.0825 0.055979 -1.083347" rpy="0 0 0"/>
     <geometry>
-      <mesh filename="package://roomac_description/meshes/eye_right_1.stl" scale="0.001 0.001 0.001"/>
+      <mesh filename="package://roomac_description/meshes/eye_right_link.stl" scale="0.001 0.001 0.001"/>
     </geometry>
     <material name="white"/>
@@ -268,9 +269,9 @@
     <origin xyz="0.0825 0.055979 -1.083347" rpy="0 0 0"/>
     <geometry>
-      <mesh filename="package://roomac_description/meshes/eye_right_1.stl" scale="0.001 0.001 0.001"/>
-    </geometry>
-  </collision>
-</link>
-<link name="eye_left_1">
+      <mesh filename="package://roomac_description/meshes/eye_right_link.stl" scale="0.001 0.001 0.001"/>
+    </geometry>
+  </collision>
+</link>
+<link name="eye_left_link">
   <inertial>
     <origin xyz="0.006260241058239718 3.517735615299333e-08 -3.5598063252706424e-07" rpy="0 0 0"/>
@@ -281,5 +282,5 @@
     <origin xyz="0.0825 -0.056021 -1.083347" rpy="0 0 0"/>
     <geometry>
-      <mesh filename="package://roomac_description/meshes/eye_left_1.stl" scale="0.001 0.001 0.001"/>
+      <mesh filename="package://roomac_description/meshes/eye_left_link.stl" scale="0.001 0.001 0.001"/>
     </geometry>
     <material name="white"/>
@@ -288,5 +289,5 @@
     <origin xyz="0.0825 -0.056021 -1.083347" rpy="0 0 0"/>
     <geometry>
-      <mesh filename="package://roomac_description/meshes/eye_left_1.stl" scale="0.001 0.001 0.001"/>
+      <mesh filename="package://roomac_description/meshes/eye_left_link.stl" scale="0.001 0.001 0.001"/>
     </geometry>
   </collision>
@@ -294,19 +295,19 @@
 <joint name="head" type="fixed">
   <origin xyz="-0.01515 -0.103129 0.441495" rpy="0 0 0"/>
-  <parent link="frame_1"/>
-  <child link="head_1"/>
+  <parent link="frame_link"/>
+  <child link="head_link"/>
 </joint>
 <joint name="eye_right" type="fixed">
   <origin xyz="-0.0025 -0.056 0.114202" rpy="0 0 0"/>
-  <parent link="head_1"/>
-  <child link="eye_right_1"/>
+  <parent link="head_link"/>
+  <child link="eye_right_link"/>
 </joint>
 <joint name="eye_left" type="fixed">
   <origin xyz="-0.0025 0.056 0.114202" rpy="0 0 0"/>
-  <parent link="head_1"/>
-  <child link="eye_left_1"/>
+  <parent link="head_link"/>
+  <child link="eye_left_link"/>
 </joint>
 <!-- RIGHT ARM -->
-<link name="shoulder_right_1">
+<link name="shoulder_right_link">
   <inertial>
     <origin xyz="-0.00456057320555428 -0.012787272244286635 0.0077144845604640855" rpy="0 0 0"/>
@@ -317,5 +318,5 @@
     <origin xyz="0.1135 0.174979 -0.9345" rpy="0 0 0"/>
     <geometry>
-      <mesh filename="package://roomac_description/meshes/shoulder_right_1.stl" scale="0.001 0.001 0.001"/>
+      <mesh filename="package://roomac_description/meshes/shoulder_right_link.stl" scale="0.001 0.001 0.001"/>
     </geometry>
     <material name="black"/>
@@ -324,9 +325,9 @@
     <origin xyz="0.1135 0.174979 -0.9345" rpy="0 0 0"/>
     <geometry>
-      <mesh filename="package://roomac_description/meshes/shoulder_right_1.stl" scale="0.001 0.001 0.001"/>
-    </geometry>
-  </collision>
-</link>
-<link name="shoulder_elbow_right_1">
+      <mesh filename="package://roomac_description/meshes/shoulder_right_link.stl" scale="0.001 0.001 0.001"/>
+    </geometry>
+  </collision>
+</link>
+<link name="shoulder_elbow_right_link">
   <inertial>
     <origin xyz="-1.8144588477334023e-05 1.4016989058340812e-07 -0.08491558495824947" rpy="0 0 0"/>
@@ -337,5 +338,5 @@
     <origin xyz="0.113 0.243979 -0.9345" rpy="0 0 0"/>
     <geometry>
-      <mesh filename="package://roomac_description/meshes/shoulder_elbow_right_1.dae" scale="0.001 0.001 0.001"/>
+      <mesh filename="package://roomac_description/meshes/shoulder_elbow_right_link.dae" scale="0.001 0.001 0.001"/>
     </geometry>
   </visual>
@@ -343,9 +344,9 @@
     <origin xyz="0.113 0.243979 -0.9345" rpy="0 0 0"/>
     <geometry>
-      <mesh filename="package://roomac_description/meshes/shoulder_elbow_right_1.stl" scale="0.001 0.001 0.001"/>
-    </geometry>
-  </collision>
-</link>
-<link name="elbow_wrist_right_1">
+      <mesh filename="package://roomac_description/meshes/shoulder_elbow_right_link.stl" scale="0.001 0.001 0.001"/>
+    </geometry>
+  </collision>
+</link>
+<link name="elbow_wrist_right_link">
   <inertial>
     <origin xyz="-0.019371175261057735 -0.001202599027629786 -0.0924289033208664" rpy="0 0 0"/>
@@ -356,5 +357,5 @@
     <origin xyz="0.0925 0.243979 -0.733425" rpy="0 0 0"/>
     <geometry>
-      <mesh filename="package://roomac_description/meshes/elbow_wrist_right_1.stl" scale="0.001 0.001 0.001"/>
+      <mesh filename="package://roomac_description/meshes/elbow_wrist_right_link.stl" scale="0.001 0.001 0.001"/>
     </geometry>
     <material name="black"/>
@@ -363,9 +364,9 @@
     <origin xyz="0.0925 0.243979 -0.733425" rpy="0 0 0"/>
     <geometry>
-      <mesh filename="package://roomac_description/meshes/elbow_wrist_right_1.stl" scale="0.001 0.001 0.001"/>
-    </geometry>
-  </collision>
-</link>
-<link name="wrist_right_1">
+      <mesh filename="package://roomac_description/meshes/elbow_wrist_right_link.stl" scale="0.001 0.001 0.001"/>
+    </geometry>
+  </collision>
+</link>
+<link name="wrist_right_link">
   <inertial>
     <origin xyz="0.02427263159088841 -0.0008946909470901598 -0.023520404043236964" rpy="0 0 0"/>
@@ -376,5 +377,5 @@
     <origin xyz="0.139354 0.243979 -0.603583" rpy="0 0 0"/>
     <geometry>
-      <mesh filename="package://roomac_description/meshes/wrist_right_1.stl" scale="0.001 0.001 0.001"/>
+      <mesh filename="package://roomac_description/meshes/wrist_right_link.stl" scale="0.001 0.001 0.001"/>
     </geometry>
     <material name="black"/>
@@ -383,10 +384,9 @@
     <origin xyz="0.139354 0.243979 -0.603583" rpy="0 0 0"/>
     <geometry>
-      <mesh filename="package://roomac_description/meshes/wrist_right_1.stl" scale="0.001 0.001 0.001"/>
-    </geometry>
-  </collision>
-</link>
-<link name="gripper_right_grip"/>
-<link name="gripper_right_1">
+      <mesh filename="package://roomac_description/meshes/wrist_right_link.stl" scale="0.001 0.001 0.001"/>
+    </geometry>
+  </collision>
+</link>
+<link name="gripper_right_link">
   <inertial>
     <origin xyz="-0.00024163561260406863 0.0010341725235240573 -0.024005848417666398" rpy="0 0 0"/>
@@ -397,5 +397,5 @@
     <origin xyz="0.114635 0.244052 -0.544791" rpy="0 0 0"/>
     <geometry>
-      <mesh filename="package://roomac_description/meshes/gripper_right_1.stl" scale="0.001 0.001 0.001"/>
+      <mesh filename="package://roomac_description/meshes/gripper_right_link.stl" scale="0.001 0.001 0.001"/>
     </geometry>
     <material name="black"/>
@@ -404,9 +404,12 @@
     <origin xyz="0.114635 0.244052 -0.544791" rpy="0 0 0"/>
     <geometry>
-      <mesh filename="package://roomac_description/meshes/gripper_right_1.stl" scale="0.001 0.001 0.001"/>
-    </geometry>
-  </collision>
-</link>
-<link name="gripper_finger_1_right_1">
+      <mesh filename="package://roomac_description/meshes/gripper_right_link.stl" scale="0.001 0.001 0.001"/>
+    </geometry>
+  </collision>
+</link>
+<!-- Point approximately in the middle between fingers, used as a position for gripping objects
+  (in inverse kinematics this point should match objects position) -->
+<link name="gripping_right_link"/>
+<link name="gripper_finger_r_right_link">
   <inertial>
     <origin xyz="0.004500248654851852 0.005686730528388695 -0.011016022246636392" rpy="0 0 0"/>
@@ -417,5 +420,5 @@
     <origin xyz="0.117385 0.274314 -0.487684" rpy="0 0 0"/>
     <geometry>
-      <mesh filename="package://roomac_description/meshes/gripper_finger_1_right_1.stl" scale="0.001 0.001 0.001"/>
+      <mesh filename="package://roomac_description/meshes/gripper_finger_r_right_link.stl" scale="0.001 0.001 0.001"/>
     </geometry>
     <material name="black"/>
@@ -424,9 +427,9 @@
     <origin xyz="0.117385 0.274314 -0.487684" rpy="0 0 0"/>
     <geometry>
-      <mesh filename="package://roomac_description/meshes/gripper_finger_1_right_1.stl" scale="0.001 0.001 0.001"/>
-    </geometry>
-  </collision>
-</link>
-<link name="gripper_finger_2_right_1">
+      <mesh filename="package://roomac_description/meshes/gripper_finger_r_right_link.stl" scale="0.001 0.001 0.001"/>
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
File: roomac_description/urdf/roomac_simulation_picking.xacro (robot description, xacro)
@@ -6,9 +6,9 @@
 <xacro:include filename="$(find roomac_description)/urdf/roomac_body.xacro" />
 <xacro:include filename="$(find roomac_description)/urdf/roomac_arm_precision_test.xacro" />
+<link name="artag_bundle_link"/>
 <joint name="artag_joint_bundle" type="fixed">
     <origin rpy="${-pi/2} 0 0" xyz="0.04857 0 0"/>
-    <parent link="artag_link_bundle_visual"/>
-    <child link="artag_link_bundle"/>
+    <parent link="artag_bundle_visual_link"/>
+    <child link="artag_bundle_link"/>
 </joint>
-<link name="artag_link_bundle"/>
 </robot>

Commit message: Remove materials.xacro file
only black definition is used, no point in keeping it in a separate file

File: roomac_description/urdf/roomac.xacro (robot description, xacro)
@@ -1,5 +1,4 @@
 <?xml version="1.0" ?>
 <robot name="roomac" xmlns:xacro="http://www.ros.org/wiki/xacro">
-<xacro:include filename="$(find roomac_description)/urdf/materials.xacro" />
 <xacro:include filename="$(find roomac_description)/urdf/roomac.trans" />
 <xacro:include filename="$(find roomac_description)/urdf/roomac.gazebo" />

File: roomac_description/urdf/roomac_body.xacro (robot description, xacro)
@@ -2,6 +2,9 @@
 <robot name="roomac" xmlns:xacro="http://www.ros.org/wiki/xacro">
 <!-- todo: standardize joint names -->
+<material name="black">
+  <color rgba="0.15 0.15 0.15 1.0"/>
+</material>
 <!-- Some links are used only for visuals:
-  - robot_body_frames_link, frame_link and artag_bundle_visual_link - collision model in robot_body_link takes them into account, and also there is no point in inertial attribute for them (again robot_body_link should be enough)
+  - robot_body_frames_link and artag_bundle_visual_link - collision model in robot_body_link takes them into account, and also there is no point in inertial attribute for them (again robot_body_link should be enough)
   - eye_right_link and eye_left_link - similar to previous example collision model in head is enough -->
 <!-- BODY -->
@@ -36,5 +39,4 @@
       <mesh filename="package://roomac_description/meshes/robot_body_frames.dae" scale="0.001 0.001 0.001"/>
     </geometry>
-    <material name="white"/>
   </visual>
 </link>
@@ -225,5 +227,4 @@
       <mesh filename="package://roomac_description/meshes/eye_right.dae" scale="0.001 0.001 0.001"/>
     </geometry>
-    <material name="white"/>
   </visual>
 </link>
@@ -234,5 +235,4 @@
       <mesh filename="package://roomac_description/meshes/eye_left.dae" scale="0.001 0.001 0.001"/>
     </geometry>
-    <material name="white"/>
   </visual>
 </link>

File: roomac_description/urdf/roomac_simulation.xacro (robot description, xacro)
@@ -1,5 +1,4 @@
 <?xml version="1.0" ?>
 <robot name="roomac" xmlns:xacro="http://www.ros.org/wiki/xacro">
-<xacro:include filename="$(find roomac_description)/urdf/materials.xacro" />
 <xacro:include filename="$(find roomac_description)/urdf/roomac.trans" />
 <xacro:include filename="$(find roomac_description)/urdf/roomac.gazebo" />
