Commit message: Change gripper rotation joint limits

File: roomac_description/urdf/roomac.xacro (robot description, xacro)
@@ -28,5 +28,5 @@
     <origin xyz="0 0 0" rpy="0 0 0"/>
     <geometry>
-      <mesh filename="package://roomac_description/meshes/robot_body_collision.stl" scale="0.001 0.00105 0.001"/>
+      <mesh filename="package://roomac_description/meshes/robot_body_collision.stl" scale="0.001 0.0011 0.001"/>
     </geometry>
   </collision>
@@ -411,5 +411,5 @@
   <child link="gripper_right_link"/>
   <axis xyz="0 0 -1"/>
-  <limit effort="30" velocity="1.0" lower="-1.570" upper="1.570"/>
+  <limit effort="30" velocity="1.0" lower="-3.14" upper="0.1"/>
 </joint>
 <joint name="gripper_finger_r_right_joint" type="prismatic">
